File: DSN/PowerDomains.kicad_sch (KiCad schematic)
At the start: 0 parts

Commit message: Added Footprints
Other:
- title: (none) -> Power Strategy
Changed lines of the file:
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@@
 (kicad_sch (version 20211123) (generator eeschema)
   (paper "A4")
+  (title_block
+    (title "Power Strategy")
+    (date "2023-03-07")
+    (rev "A")
+    (comment 1 "Designed by DragonEnjoyer :3")
+  )
   (image (at 135.89 88.9) (scale 0.892189)
     (data
