File: DSN/PSRAM.kicad_sch (KiCad schematic)
At the start: 6 parts

Commit message: Added Footprints
Parts:
- U?: footprint (none) -> Package_BGA:24-BGA_6x8mm_5x5mm_ball_1.0mm_pitch; MFR PN (none) -> S80KS5122GABHM020
Other:
- title: (none) -> PSRAM
Changed lines of the file:
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@@
 (kicad_sch (version 20211123) (generator eeschema)
   (paper "A4")
+  (title_block
+    (title "PSRAM")
+    (date "2023-03-07")
+    (rev "A")
+    (comment 1 "Designed by DragonEnjoyer :3")
+  )
   (junction (at 93.98 72.39) (diameter 0) (color 0 0 0 0)
   )
@@
     (property "Reference" "U?" (id 0) (at 148.59 71.12 0))
     (property "Value" "S80KS5122GABHM020" (id 1) (at 148.59 73.66 0))
-    (property "Footprint" "" (id 2) (at 102.87 153.67 0)
-      (effects (font (size 1.27 1.27)) hide)
-    )
-    (property "Datasheet" "" (id 3) (at 102.87 153.67 0)
-      (effects (font (size 1.27 1.27)) hide)
-    )
+    (property "Footprint" "Package_BGA:24-BGA_6x8mm_5x5mm_ball_1.0mm_pitch" (id 2) (at 102.87 153.67 0)
+      (effects (font (size 1.27 1.27)) hide)
+    )
+    (property "Datasheet" "https://www.infineon.com/dgdl/Infineon-S80KS5122_1.8_V_512-Mbit_HyperBus_Interface_HyperRAM_(Self-Refresh_DRAM)-DataSheet-v01_00-EN.pdf?fileId=8ac78c8c7dc4255f017dd81b77c1088f" (id 3) (at 102.87 153.67 0)
+      (effects (font (size 1.27 1.27)) hide)
+    )
+    (property "MFR PN" "S80KS5122GABHM020" (id 4) (at 139.7 123.19 0)
+      (effects (font (size 1.27 1.27)) hide)
+    )

Commit message: Added component ref des
Parts:
- gave numbers to parts that had none: 6
Changed lines of the file:
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@@
   (symbol (lib_id "power:GND") (at 116.84 80.01 0) (mirror y) (unit 1)
     (in_bom yes) (on_board yes)
-    (property "Reference" "#PWR?" (id 0) (at 116.84 86.36 0)
+    (property "Reference" "#PWR0114" (id 0) (at 116.84 86.36 0)
       (effects (font (size 1.27 1.27)) hide)
     )
@@
   (symbol (lib_id "power:GND") (at 134.62 133.35 0) (mirror y) (unit 1)
     (in_bom yes) (on_board yes)
-    (property "Reference" "#PWR?" (id 0) (at 134.62 139.7 0)
+    (property "Reference" "#PWR0117" (id 0) (at 134.62 139.7 0)
       (effects (font (size 1.27 1.27)) hide)
     )
@@
   (symbol (lib_id "Device:C_Small") (at 116.84 76.2 0) (mirror y) (unit 1)
     (in_bom yes) (on_board yes) (fields_autoplaced)
-    (property "Reference" "C?" (id 0) (at 114.3 74.9362 0)
+    (property "Reference" "C63" (id 0) (at 114.3 74.9362 0)
       (effects (font (size 1.27 1.27)) (justify left))
     )
@@
   (symbol (lib_id "Device:C_Small") (at 93.98 76.2 0) (mirror y) (unit 1)
     (in_bom yes) (on_board yes) (fields_autoplaced)
-    (property "Reference" "C?" (id 0) (at 91.44 74.9362 0)
+    (property "Reference" "C61" (id 0) (at 91.44 74.9362 0)
       (effects (font (size 1.27 1.27)) (justify left))
     )
@@
   (symbol (lib_id "power:GND") (at 105.41 80.01 0) (mirror y) (unit 1)
     (in_bom yes) (on_board yes)
-    (property "Reference" "#PWR?" (id 0) (at 105.41 86.36 0)
+    (property "Reference" "#PWR0113" (id 0) (at 105.41 86.36 0)
       (effects (font (size 1.27 1.27)) hide)
     )
@@
   (symbol (lib_id "power:+1V8") (at 119.38 111.76 0) (unit 1)
     (in_bom yes) (on_board yes)
-    (property "Reference" "#PWR?" (id 0) (at 119.38 115.57 0)
+    (property "Reference" "#PWR0115" (id 0) (at 119.38 115.57 0)
       (effects (font (size 1.27 1.27)) hide)
     )
@@
   (symbol (lib_id "Memory_RAM:S80KS5122GABHM020") (at 139.7 123.19 0) (unit 1)
     (in_bom yes) (on_board yes) (fields_autoplaced)
-    (property "Reference" "U?" (id 0) (at 148.59 71.12 0))
+    (property "Reference" "U9" (id 0) (at 148.59 71.12 0))
     (property "Value" "S80KS5122GABHM020" (id 1) (at 148.59 73.66 0))
     (property "Footprint" "Package_BGA:24-BGA_6x8mm_5x5mm_ball_1.0mm_pitch" (id 2) (at 102.87 153.67 0)
@@
   (symbol (lib_id "Device:C_Small") (at 128.27 76.2 0) (mirror y) (unit 1)
     (in_bom yes) (on_board yes) (fields_autoplaced)
-    (property "Reference" "C?" (id 0) (at 125.73 74.9362 0)
+    (property "Reference" "C64" (id 0) (at 125.73 74.9362 0)
       (effects (font (size 1.27 1.27)) (justify left))
     )
@@
   (symbol (lib_id "Device:R_US") (at 124.46 109.22 0) (mirror x) (unit 1)
     (in_bom yes) (on_board yes)
-    (property "Reference" "R?" (id 0) (at 127 111.76 0))
+    (property "Reference" "R49" (id 0) (at 127 111.76 0))
     (property "Value" "100K" (id 1) (at 128.27 109.22 0))
     (property "Footprint" "Resistor_SMD:R_0402_1005Metric" (id 2) (at 125.476 108.966 90)
@@
   (symbol (lib_id "power:+1V8") (at 93.98 71.12 0) (unit 1)
     (in_bom yes) (on_board yes)
-    (property "Reference" "#PWR?" (id 0) (at 93.98 74.93 0)
+    (property "Reference" "#PWR0111" (id 0) (at 93.98 74.93 0)
       (effects (font (size 1.27 1.27)) hide)
     )
@@
   (symbol (lib_id "power:GND") (at 128.27 80.01 0) (mirror y) (unit 1)
     (in_bom yes) (on_board yes)
-    (property "Reference" "#PWR?" (id 0) (at 128.27 86.36 0)
+    (property "Reference" "#PWR0116" (id 0) (at 128.27 86.36 0)
       (effects (font (size 1.27 1.27)) hide)
     )
@@
   (symbol (lib_id "power:GND") (at 93.98 80.01 0) (mirror y) (unit 1)
     (in_bom yes) (on_board yes)
-    (property "Reference" "#PWR?" (id 0) (at 93.98 86.36 0)
+    (property "Reference" "#PWR0112" (id 0) (at 93.98 86.36 0)
       (effects (font (size 1.27 1.27)) hide)
     )
@@
   (symbol (lib_id "Device:C_Small") (at 105.41 76.2 0) (mirror y) (unit 1)
     (in_bom yes) (on_board yes) (fields_autoplaced)
-    (property "Reference" "C?" (id 0) (at 102.87 74.9362 0)
-      (effects (font (size 1.27 1.27)) (justify left))
-    )
+    (property "Reference" "C62" (id 0) (at 102.87 74.9362 0)
+      (effects (font (size 1.27 1.27)) (justify left))
+    )
