File: DSN/FPGA_0.kicad_sch (KiCad schematic)
At the start: 134 parts

Commit message: Added PSRAM, Finished Schematic
Footprint assignment required, some minor changes to be made to schematic. Sheet naming and commenting to be done.
Parts:
- added C? (x8): 100nF, Capacitor_SMD:C_0402_1005Metric, symbol Device:C_Small
- added U? (x4): TXB0108PWR, digikey-footprints:TSSOP-20_W4.4mm, symbol dk_Logic-Translators-Level-Shifters:TXB0108PWR
Connections:
- net +1V8: now also C?.1, C?.1, C?.1, C?.1, C?.1, C?.1, C?.1, U?.C1 (VCCO_35), U?.F2 (VCCO_35), U?.H6 (VCCO_35), U?.J3 (VCCO_35), U?.M4 (VCCO_35), U?.N1 (VCCO_35), C?.1, C?.1, C?.1, C?.1, U?.10 (OE), U?.10 (OE), U?.10 (OE), U?.10 (OE), U?.2 (VCCA), U?.2 (VCCA), U?.2 (VCCA), U?.2 (VCCA)
- net +3V3: now also C?.1, C?.1, C?.1, C?.1, U?.19 (VCCB), U?.19 (VCCB), U?.19 (VCCB), U?.19 (VCCB); no longer C?.1, C?.1, C?.1, C?.1, C?.1, C?.1, C?.1, U?.C1 (VCCO_35), U?.F2 (VCCO_35), U?.H6 (VCCO_35), U?.J3 (VCCO_35), U?.M4 (VCCO_35), U?.N1 (VCCO_35)
- net GND: now also C?.2, C?.2, C?.2, C?.2, C?.2, C?.2, C?.2, C?.2, U?.11 (GND), U?.11 (GND), U?.11 (GND), U?.11 (GND)
- net FPGA_0_GTP_CLK1_N: now reaches U?.E10 (MGTREFCLK1N_216)
- net FPGA_0_GTP_CLK1_P: now reaches U?.F10 (MGTREFCLK1P_216)
- net FPGA_0_DP_RXL0_N renamed FPGA_0_RXL0_N
- net FPGA_0_DP_RXL0_P renamed FPGA_0_RXL0_P
- net FPGA_0_DP_RXL1_N renamed FPGA_0_RXL1_N
- net FPGA_0_DP_RXL1_P renamed FPGA_0_RXL1_P
- net FPGA_0_DP_RXL2_N renamed FPGA_0_RXL2_N
- net FPGA_0_DP_RXL2_P renamed FPGA_0_RXL2_P
- net FPGA_0_DP_RXL3_N renamed FPGA_0_RXL3_N
- net FPGA_0_DP_RXL3_P renamed FPGA_0_RXL3_P
- net FPGA_0_DP_TXL0_N renamed FPGA_0_TXL0_N
- net FPGA_0_DP_TXL0_P renamed FPGA_0_TXL0_P
- net FPGA_0_DP_TXL1_N renamed FPGA_0_TXL1_N
- net FPGA_0_DP_TXL1_P renamed FPGA_0_TXL1_P
- net FPGA_0_DP_TXL2_N renamed FPGA_0_TXL2_N
- net FPGA_0_DP_TXL2_P renamed FPGA_0_TXL2_P
- net FPGA_0_DP_TXL3_N renamed FPGA_0_TXL3_N
- net FPGA_0_DP_TXL3_P renamed FPGA_0_TXL3_P
- net FPGA_0_GTP_CLK_C_N renamed FPGA_0_GTP_CLK0_C_N
- net FPGA_0_GTP_CLK_C_P renamed FPGA_0_GTP_CLK0_C_P
- net FPGA_0_GTP_CLK_N renamed FPGA_0_GTP_CLK0_N
- net FPGA_0_GTP_CLK_P renamed FPGA_0_GTP_CLK0_P
- net FPGA_0_UER_IO50: no longer names the net of U?.F4 (IO_0_35)
- net FPGA_0_UER_IO51 renamed FPGA_0_PSRAM_CS
- net FPGA_0_UER_IO52 renamed FPGA_0_PSRAM_RESET
- net FPGA_0_UER_IO53 renamed FPGA_0_PSRAM_RWDS
- net FPGA_0_UER_IO54: no longer names the net of U?.B2 (IO_L2N_T0_AD12N_35)
- net FPGA_0_UER_IO55 renamed FPGA_0_PSRAM_D0
- net FPGA_0_UER_IO56 renamed FPGA_0_PSRAM_D1
- net FPGA_0_UER_IO57 renamed FPGA_0_PSRAM_D2
- net FPGA_0_UER_IO58 renamed FPGA_0_PSRAM_D3
- net FPGA_0_UER_IO59 renamed FPGA_0_PSRAM_D4
- net FPGA_0_UER_IO60 renamed FPGA_0_PSRAM_D5
- net FPGA_0_UER_IO61 renamed FPGA_0_PSRAM_D6
- net FPGA_0_UER_IO62 renamed FPGA_0_PSRAM_D7
- net FPGA_0_UER_IO63 renamed FPGA_0_PMOD0_LV_IO0
- net FPGA_0_PMOD0_LV_IO0: now also U?.1 (A1)
- net FPGA_0_UER_IO64 renamed FPGA_0_PMOD0_LV_IO1
- net FPGA_0_PMOD0_LV_IO1: now also U?.3 (A2)
- net FPGA_0_UER_IO65 renamed FPGA_0_PMOD0_LV_IO2
- net FPGA_0_PMOD0_LV_IO2: now also U?.4 (A3)
- net FPGA_0_UER_IO66 renamed FPGA_0_PMOD0_LV_IO3
- net FPGA_0_PMOD0_LV_IO3: now also U?.5 (A4)
- net FPGA_0_UER_IO67 renamed FPGA_0_PMOD0_LV_IO4
- net FPGA_0_PMOD0_LV_IO4: now also U?.6 (A5)
- net FPGA_0_UER_IO68 renamed FPGA_0_PMOD0_LV_IO5
- net FPGA_0_PMOD0_LV_IO5: now also U?.7 (A6)
- net FPGA_0_UER_IO69 renamed FPGA_0_PMOD0_LV_IO6
- net FPGA_0_PMOD0_LV_IO6: now also U?.8 (A7)
- net FPGA_0_UER_IO70 renamed FPGA_0_PMOD0_LV_IO7
- net FPGA_0_PMOD0_LV_IO7: now also U?.9 (A8)
- net FPGA_0_UER_IO71: no longer names the net of U?.H3 (IO_L11P_T1_SRCC_35)
- net FPGA_0_UER_IO72: no longer names the net of U?.G3 (IO_L11N_T1_SRCC_35)
- net FPGA_0_UER_IO73 renamed FPGA_0_PSRAM_CLK_P
- net FPGA_0_UER_IO74 renamed FPGA_0_PSRAM_CLK_N
- net FPGA_0_UER_IO75 renamed FPGA_0_PMOD1_LV_IO0
- net FPGA_0_PMOD1_LV_IO0: now also U?.1 (A1)
- net FPGA_0_UER_IO76 renamed FPGA_0_PMOD1_LV_IO1
- net FPGA_0_PMOD1_LV_IO1: now also U?.3 (A2)
- net FPGA_0_UER_IO77 renamed FPGA_0_PMOD1_LV_IO2
- net FPGA_0_PMOD1_LV_IO2: now also U?.4 (A3)
- net FPGA_0_UER_IO78 renamed FPGA_0_PMOD1_LV_IO3
- net FPGA_0_PMOD1_LV_IO3: now also U?.5 (A4)
- net FPGA_0_UER_IO79 renamed FPGA_0_PMOD1_LV_IO4
- net FPGA_0_PMOD1_LV_IO4: now also U?.6 (A5)
- net FPGA_0_UER_IO80 renamed FPGA_0_PMOD1_LV_IO5
- net FPGA_0_PMOD1_LV_IO5: now also U?.7 (A6)
- net FPGA_0_UER_IO81 renamed FPGA_0_PMOD1_LV_IO6
- net FPGA_0_PMOD1_LV_IO6: now also U?.8 (A7)
- net FPGA_0_UER_IO82 renamed FPGA_0_PMOD1_LV_IO7
- net FPGA_0_PMOD1_LV_IO7: now also U?.9 (A8)
- net FPGA_0_UER_IO83 renamed FPGA_0_PMOD2_LV_IO0
- net FPGA_0_PMOD2_LV_IO0: now also U?.1 (A1)
- net FPGA_0_UER_IO84 renamed FPGA_0_PMOD2_LV_IO1
- net FPGA_0_PMOD2_LV_IO1: now also U?.3 (A2)
- net FPGA_0_UER_IO85 renamed FPGA_0_PMOD2_LV_IO2
- net FPGA_0_PMOD2_LV_IO2: now also U?.4 (A3)
- net FPGA_0_UER_IO86 renamed FPGA_0_PMOD2_LV_IO3
- net FPGA_0_PMOD2_LV_IO3: now also U?.5 (A4)
- net FPGA_0_UER_IO87 renamed FPGA_0_PMOD2_LV_IO4
- net FPGA_0_PMOD2_LV_IO4: now also U?.6 (A5)
- net FPGA_0_UER_IO88 renamed FPGA_0_PMOD2_LV_IO5
- net FPGA_0_PMOD2_LV_IO5: now also U?.7 (A6)
- net FPGA_0_UER_IO89 renamed FPGA_0_PMOD2_LV_IO6
- net FPGA_0_PMOD2_LV_IO6: now also U?.8 (A7)
- net FPGA_0_UER_IO90 renamed FPGA_0_PMOD2_LV_IO7
- net FPGA_0_PMOD2_LV_IO7: now also U?.9 (A8)
- net FPGA_0_UER_IO91 renamed FPGA_0_PMOD3_LV_IO0
- net FPGA_0_PMOD3_LV_IO0: now also U?.1 (A1)
- net FPGA_0_UER_IO92 renamed FPGA_0_PMOD3_LV_IO1
- net FPGA_0_PMOD3_LV_IO1: now also U?.3 (A2)
- net FPGA_0_UER_IO93 renamed FPGA_0_PMOD3_LV_IO2
- net FPGA_0_PMOD3_LV_IO2: now also U?.4 (A3)
- net FPGA_0_UER_IO94 renamed FPGA_0_PMOD3_LV_IO3
- net FPGA_0_PMOD3_LV_IO3: now also U?.5 (A4)
- net FPGA_0_UER_IO95 renamed FPGA_0_PMOD3_LV_IO4
- net FPGA_0_PMOD3_LV_IO4: now also U?.6 (A5)
- net FPGA_0_UER_IO96 renamed FPGA_0_PMOD3_LV_IO5
- net FPGA_0_PMOD3_LV_IO5: now also U?.7 (A6)
- net FPGA_0_UER_IO97 renamed FPGA_0_PMOD3_LV_IO6
- net FPGA_0_PMOD3_LV_IO6: now also U?.8 (A7)
- net FPGA_0_UER_IO98 renamed FPGA_0_PMOD3_LV_IO7
- net FPGA_0_PMOD3_LV_IO7: now also U?.9 (A8)
- net FPGA_0_UER_IO99: no longer names the net of U?.L6 (IO_25_35)
- new net FPGA_0_PMOD0_IO0: U?.20 (B1)
- new net FPGA_0_PMOD0_IO1: U?.18 (B2)
- new net FPGA_0_PMOD0_IO2: U?.17 (B3)
- new net FPGA_0_PMOD0_IO3: U?.16 (B4)
- new net FPGA_0_PMOD0_IO4: U?.15 (B5)
- new net FPGA_0_PMOD0_IO5: U?.14 (B6)
- new net FPGA_0_PMOD0_IO6: U?.13 (B7)
- new net FPGA_0_PMOD0_IO7: U?.12 (B8)
- new net FPGA_0_PMOD1_IO0: U?.20 (B1)
- new net FPGA_0_PMOD1_IO1: U?.18 (B2)
- new net FPGA_0_PMOD1_IO2: U?.17 (B3)
- new net FPGA_0_PMOD1_IO3: U?.16 (B4)
- new net FPGA_0_PMOD1_IO4: U?.15 (B5)
- new net FPGA_0_PMOD1_IO5: U?.14 (B6)
- new net FPGA_0_PMOD1_IO6: U?.13 (B7)
- new net FPGA_0_PMOD1_IO7: U?.12 (B8)
- new net FPGA_0_PMOD2_IO0: U?.20 (B1)
- new net FPGA_0_PMOD2_IO1: U?.18 (B2)
- new net FPGA_0_PMOD2_IO2: U?.17 (B3)
- new net FPGA_0_PMOD2_IO3: U?.16 (B4)
- new net FPGA_0_PMOD2_IO4: U?.15 (B5)
- new net FPGA_0_PMOD2_IO5: U?.14 (B6)
- new net FPGA_0_PMOD2_IO6: U?.13 (B7)
- new net FPGA_0_PMOD2_IO7: U?.12 (B8)
- new net FPGA_0_PMOD3_IO0: U?.20 (B1)
- new net FPGA_0_PMOD3_IO1: U?.18 (B2)
- new net FPGA_0_PMOD3_IO2: U?.17 (B3)
- new net FPGA_0_PMOD3_IO3: U?.16 (B4)
- new net FPGA_0_PMOD3_IO4: U?.15 (B5)
- new net FPGA_0_PMOD3_IO5: U?.14 (B6)
- new net FPGA_0_PMOD3_IO6: U?.13 (B7)
- new net FPGA_0_PMOD3_IO7: U?.12 (B8)
- no-connect marks 4 -> 2
Other:
- note added: "135Mhz Reference CLK"
- note removed: "135Mhz Displayport CLK"

Commit message: Added Footprints
Parts:
- removed SW? (x2): SW_Push, symbol Switch:SW_Push
- removed SW?: SW_DIP_x03, symbol Switch:SW_DIP_x03
- removed U?: DSC1103BI2-135.0000, symbol Oscillator:DSC1103BI2-135.0000
- removed U?: SIT9120AI, symbol Oscillator:SIT9120AI
- removed U?: IS25LP128F, symbol Memory_Flash:IS25LP128F
- added SW? (x2): SW_Push, Button_Switch_SMD:SW_Push_1P1T_NO_CK_KMR2, symbol Switch:SW_Push
- added SW?: SW_DIP_x03, Button_Switch_SMD:SW_DIP_SPSTx03_Slide_9.78x9.8mm_W8.61mm_P2.54mm, symbol Switch:SW_DIP_x03
- added U?: DSC1103BI2-135.0000, Package_DFN_QFN:VDFN-6, symbol Oscillator:DSC1103BI2-135.0000
- added U?: SIT9120AI, Oscillator:Oscillator_SMD_SiTime_SiT9121-6Pin_3.2x2.5mm, symbol Oscillator:SIT9120AI
- added U?: IS25LP128F, Package_SO:SOIC-8_3.9x4.9mm_P1.27mm, symbol Memory_Flash:IS25LP128F
- U?: footprint (none) -> Package_BGA:Xilinx_FGG484
Connections:
- net +3V3: now also U?.1 (EN), U?.3 (WP#(IO2)), U?.6 (VDD), U?.6 (VDD), U?.7 (HOLD#/RESET#), U?.8 (VCC)
- net FPGA_0_CCLK: now also U?.6 (SCK)
- net FPGA_0_DIN: now also U?.2 (SO(I01))
- net FPGA_0_DOUT: now also U?.5 (SI(IO0))
- net FPGA_0_FCS_B: now also U?.1 (CE#)
- net FPGA_0_GTP_CLK0_C_N: now also U?.5 (OUT_N)
- net FPGA_0_GTP_CLK0_C_P: now also U?.4 (OUT_P)
- net FPGA_0_M0: now also SW?.1
- net FPGA_0_M1: now also SW?.2
- net FPGA_0_M2: now also SW?.3
- net FPGA_0_PROGB: now also SW?.1
- net FPGA_0_SYSCLK_N: now also U?.5 (OUT_N)
- net FPGA_0_SYSCLK_P: now also U?.4 (OUT_P)
- net FPGA_0_SYSRST: now also SW?.1
- net GND: now also SW?.2, SW?.2, SW?.4, SW?.5, SW?.6, U?.3 (GND), U?.3 (GND), U?.4 (GND)
- net at R?.2: now also U?.1 (NC/OE/ST)
Other:
- title: (none) -> FPGA 0
Changed lines of the file:
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@@
 (kicad_sch (version 20211123) (generator eeschema)
   (paper "A1")
+  (title_block
+    (title "FPGA 0")
+    (date "2023-03-07")
+    (rev "A")
+    (comment 1 "Designed by DragonEnjoyer :3")
+  )
   (junction (at 246.38 367.03) (diameter 0) (color 0 0 0 0)
   )
@@
     (pin "2")
   )
-  (symbol (lib_id "Switch:SW_Push") (at 745.49 444.5 0) (unit 1)
-    (in_bom yes) (on_board yes) (fields_autoplaced)
-    (property "Reference" "SW?" (id 0) (at 745.49 436.88 0))
-    (property "Value" "SW_Push" (id 1) (at 745.49 439.42 0))
-    (property "Footprint" "" (id 2) (at 745.49 439.42 0)
-      (effects (font (size 1.27 1.27)) hide)
-    )
-    (property "Datasheet" "~" (id 3) (at 745.49 439.42 0)
-      (effects (font (size 1.27 1.27)) hide)
-    )
-    (pin "1")
-    (pin "2")
-  )
   (symbol (lib_id "power:GND") (at 50.8 308.61 0) (unit 1)
     (in_bom yes) (on_board yes) (fields_autoplaced)
@@
     (pin "1")
   )
-  (symbol (lib_id "Oscillator:DSC1103BI2-135.0000") (at 424.18 464.82 0) (unit 1)
-    (in_bom yes) (on_board yes) (fields_autoplaced)
-    (property "Reference" "U?" (id 0) (at 436.245 444.5 0))
-    (property "Value" "DSC1103BI2-135.0000" (id 1) (at 436.245 447.04 0))
-    (property "Footprint" "" (id 2) (at 410.21 452.12 0)
-      (effects (font (size 1.27 1.27)) hide)
-    )
-    (property "Datasheet" "" (id 3) (at 410.21 452.12 0)
-      (effects (font (size 1.27 1.27)) hide)
-    )
-    (pin "1")
-    (pin "2")
-    (pin "3")
-    (pin "4")
-    (pin "5")
-    (pin "6")
-  )
   (symbol (lib_id "power:GND") (at 267.97 53.34 0) (mirror y) (unit 1)
     (in_bom yes) (on_board yes)
@@
     (pin "1")
   )
+  (symbol (lib_id "Switch:SW_Push") (at 745.49 459.74 0) (unit 1)
+    (in_bom yes) (on_board yes) (fields_autoplaced)
+    (property "Reference" "SW?" (id 0) (at 745.49 452.12 0))
+    (property "Value" "SW_Push" (id 1) (at 745.49 454.66 0))
+    (property "Footprint" "Button_Switch_SMD:SW_Push_1P1T_NO_CK_KMR2" (id 2) (at 745.49 454.66 0)
+      (effects (font (size 1.27 1.27)) hide)
+    )
+    (property "Datasheet" "~" (id 3) (at 745.49 454.66 0)
+      (effects (font (size 1.27 1.27)) hide)
+    )
+    (pin "1")
+    (pin "2")
+  )
   (symbol (lib_id "power:GND") (at 580.39 69.85 0) (unit 1)
     (in_bom yes) (on_board yes)
@@
     (pin "2")
   )
+  (symbol (lib_id "Switch:SW_Push") (at 745.49 444.5 0) (unit 1)
+    (in_bom yes) (on_board yes) (fields_autoplaced)
+    (property "Reference" "SW?" (id 0) (at 745.49 436.88 0))
+    (property "Value" "SW_Push" (id 1) (at 745.49 439.42 0))
+    (property "Footprint" "Button_Switch_SMD:SW_Push_1P1T_NO_CK_KMR2" (id 2) (at 745.49 439.42 0)
+      (effects (font (size 1.27 1.27)) hide)
+    )
+    (property "Datasheet" "~" (id 3) (at 745.49 439.42 0)
+      (effects (font (size 1.27 1.27)) hide)
+    )
+    (pin "1")
+    (pin "2")
+  )
   (symbol (lib_id "power:GND") (at 487.68 532.13 0) (unit 1)
     (in_bom yes) (on_board yes)
@@
     (pin "1")
   )
-  (symbol (lib_id "Oscillator:SIT9120AI") (at 195.58 248.92 0) (unit 1)
-    (in_bom yes) (on_board yes) (fields_autoplaced)
-    (property "Reference" "U?" (id 0) (at 208.915 228.6 0))
-    (property "Value" "SIT9120AI" (id 1) (at 208.915 231.14 0))
-    (property "Footprint" "" (id 2) (at 176.53 238.76 0)
-      (effects (font (size 1.27 1.27)) hide)
-    )
-    (property "Datasheet" "" (id 3) (at 176.53 238.76 0)
-      (effects (font (size 1.27 1.27)) hide)
-    )
-    (pin "1")
-    (pin "2")
-    (pin "3")
-    (pin "4")
-    (pin "5")
-    (pin "6")
-  )
   (symbol (lib_id "power:GND") (at 725.17 300.99 0) (mirror y) (unit 1)
     (in_bom yes) (on_board yes)
@@
     (pin "2")
   )
+  (symbol (lib_id "Oscillator:DSC1103BI2-135.0000") (at 424.18 464.82 0) (unit 1)
+    (in_bom yes) (on_board yes) (fields_autoplaced)
+    (property "Reference" "U?" (id 0) (at 436.245 444.5 0))
+    (property "Value" "DSC1103BI2-135.0000" (id 1) (at 436.245 447.04 0))
+    (property "Footprint" "Package_DFN_QFN:VDFN-6" (id 2) (at 410.21 452.12 0)
+      (effects (font (size 1.27 1.27)) hide)
+    )
+    (property "Datasheet" "https://rocelec.widen.net/view/pdf/9j4mxdnz0b/MCHP-S-A0006612827-1.pdf?t.download=true&u=5oefqw" (id 3) (at 410.21 452.12 0)
+      (effects (font (size 1.27 1.27)) hide)
+    )
+    (pin "1")
+    (pin "2")
+    (pin "3")
+    (pin "4")
+    (pin "5")
+    (pin "6")
+  )
   (symbol (lib_id "Device:C_Small") (at 476.25 46.99 0) (mirror y) (unit 1)
     (in_bom yes) (on_board yes) (fields_autoplaced)
@@
     (pin "2")
   )
+  (symbol (lib_id "Oscillator:SIT9120AI") (at 195.58 248.92 0) (unit 1)
+    (in_bom yes) (on_board yes) (fields_autoplaced)
+    (property "Reference" "U?" (id 0) (at 208.915 228.6 0))
+    (property "Value" "SIT9120AI" (id 1) (at 208.915 231.14 0))
+    (property "Footprint" "Oscillator:Oscillator_SMD_SiTime_SiT9121-6Pin_3.2x2.5mm" (id 2) (at 176.53 238.76 0)
+      (effects (font (size 1.27 1.27)) hide)
+    )
+    (property "Datasheet" "https://www.sitime.com/datasheet/SiT9120" (id 3) (at 176.53 238.76 0)
+      (effects (font (size 1.27 1.27)) hide)
+    )
+    (pin "1")
+    (pin "2")
+    (pin "3")
+    (pin "4")
+    (pin "5")
+    (pin "6")
+  )
   (symbol (lib_id "Device:C_Small") (at 742.95 64.77 0) (mirror y) (unit 1)
     (in_bom yes) (on_board yes) (fields_autoplaced)
@@
       (effects (font (size 1.27 1.27)) (justify right))
     )
-    (property "Footprint" "" (id 2) (at 199.39 138.43 0)
+    (property "Footprint" "Package_BGA:Xilinx_FGG484" (id 2) (at 199.39 138.43 0)
       (effects (font (size 1.27 1.27)) hide)
     )
@@
     (pin "2")
   )
-  (symbol (lib_id "Memory_Flash:IS25LP128F") (at 636.27 535.94 0) (unit 1)
-    (in_bom yes) (on_board yes) (fields_autoplaced)
-    (property "Reference" "U?" (id 0) (at 650.24 513.08 0))
-    (property "Value" "IS25LP128F" (id 1) (at 650.24 515.62 0))
-    (property "Footprint" "" (id 2) (at 636.27 535.94 0)
-      (effects (font (size 1.27 1.27)) hide)
-    )
-    (property "Datasheet" "" (id 3) (at 636.27 535.94 0)
-      (effects (font (size 1.27 1.27)) hide)
-    )
-    (pin "1")
-    (pin "2")
-    (pin "3")
-    (pin "4")
-    (pin "5")
-    (pin "6")
-    (pin "7")
-    (pin "8")
-  )
   (symbol (lib_id "power:GND") (at 106.68 377.19 0) (unit 1)
     (in_bom yes) (on_board yes)
@@
     (pin "1")
   )
-  (symbol (lib_id "Switch:SW_DIP_x03") (at 692.15 455.93 0) (unit 1)
-    (in_bom yes) (on_board yes) (fields_autoplaced)
-    (property "Reference" "SW?" (id 0) (at 692.15 443.23 0))
-    (property "Value" "SW_DIP_x03" (id 1) (at 692.15 445.77 0))
-    (property "Footprint" "" (id 2) (at 692.15 455.93 0)
-      (effects (font (size 1.27 1.27)) hide)
-    )
-    (property "Datasheet" "~" (id 3) (at 692.15 455.93 0)
-      (effects (font (size 1.27 1.27)) hide)
-    )
-    (pin "1")
-    (pin "2")
-    (pin "3")
-    (pin "4")
-    (pin "5")
-    (pin "6")
-  )
   (symbol (lib_id "Device:R_US") (at 755.65 398.78 180) (unit 1)
     (in_bom yes) (on_board yes) (fields_autoplaced)
@@
     (pin "1")
   )
+  (symbol (lib_id "Memory_Flash:IS25LP128F") (at 636.27 535.94 0) (unit 1)
+    (in_bom yes) (on_board yes) (fields_autoplaced)
+    (property "Reference" "U?" (id 0) (at 650.24 513.08 0))
+    (property "Value" "IS25LP128F" (id 1) (at 650.24 515.62 0))
+    (property "Footprint" "Package_SO:SOIC-8_3.9x4.9mm_P1.27mm" (id 2) (at 636.27 535.94 0)
+      (effects (font (size 1.27 1.27)) hide)
+    )
+    (property "Datasheet" "https://www.issi.com/WW/pdf/25LP-WP128F.pdf" (id 3) (at 636.27 535.94 0)
+      (effects (font (size 1.27 1.27)) hide)
+    )
+    (property "MFR PN" "IS25LP128F-JBLA3" (id 4) (at 636.27 535.94 0)
+      (effects (font (size 1.27 1.27)) hide)
+    )
+    (pin "1")
+    (pin "2")
+    (pin "3")
+    (pin "4")
+    (pin "5")
+    (pin "6")
+    (pin "7")
+    (pin "8")
+  )
   (symbol (lib_id "power:GND") (at 755.65 243.84 0) (unit 1)
     (in_bom yes) (on_board yes)
@@
     (pin "2")
   )
+  (symbol (lib_id "Switch:SW_DIP_x03") (at 692.15 455.93 0) (unit 1)
+    (in_bom yes) (on_board yes) (fields_autoplaced)
+    (property "Reference" "SW?" (id 0) (at 692.15 443.23 0))
+    (property "Value" "SW_DIP_x03" (id 1) (at 692.15 445.77 0))
+    (property "Footprint" "Button_Switch_SMD:SW_DIP_SPSTx03_Slide_9.78x9.8mm_W8.61mm_P2.54mm" (id 2) (at 692.15 455.93 0)
+      (effects (font (size 1.27 1.27)) hide)
+    )
+    (property "Datasheet" "~" (id 3) (at 692.15 455.93 0)
+      (effects (font (size 1.27 1.27)) hide)
+    )
+    (pin "1")
+    (pin "2")
+    (pin "3")
+    (pin "4")
+    (pin "5")
+    (pin "6")
+  )
   (symbol (lib_id "Device:C_Small") (at 77.47 410.21 0) (unit 1)
     (in_bom yes) (on_board yes) (fields_autoplaced)
@@
       (effects (font (size 1.27 1.27)) hide)
     )
-    (pin "1")
-    (pin "2")
-  )
-  (symbol (lib_id "Switch:SW_Push") (at 745.49 459.74 0) (unit 1)
-    (in_bom yes) (on_board yes) (fields_autoplaced)
-    (property "Reference" "SW?" (id 0) (at 745.49 452.12 0))
-    (property "Value" "SW_Push" (id 1) (at 745.49 454.66 0))
-    (property "Footprint" "" (id 2) (at 745.49 454.66 0)
-      (effects (font (size 1.27 1.27)) hide)
-    )
-    (property "Datasheet" "~" (id 3) (at 745.49 454.66 0)
-      (effects (font (size 1.27 1.27)) hide)
-    )

Commit message: Added component ref des
Parts:
- added C356: 100nF, Capacitor_SMD:C_0402_1005Metric, symbol Device:C_Small
- added U31: TC1047AVNBTR, digikey-footprints:SOT-23-3, symbol dk_Temperature-Sensors-Analog-and-Digital-Output:TC1047AVNBTR
- gave numbers to parts that had none: 140
Connections:
- net +1V8: now also U20.K10 (VCCADC_0)
- net +3V3: now also C356.1, U31.1 (VDD)
- net GND: now also U20.K9 (GNDADC_0), C356.2, U31.3 (GND)
- new net TSNS_FPGA0: U31.2 (VOUT)

Commit message: Fixed all ERC Errors
Warnings can be ignored
Parts:
- added TP15, TP16: TestPoint_Probe, TestPoint:TestPoint_Loop_D2.50mm_Drill1.85mm, symbol Connector:TestPoint_Probe
Connections:
- net FPGA_PROGB is gone; now on net FPGA_0_PROGB: R202.1
- net FPGA_0_VREF_P: now also TP16.1
- net TSNS_FPGA0: now also TP15.1
- net FPGA_0_UER_IO0 renamed FPGA_0_USER_IO0
- net FPGA_0_UER_IO1 renamed FPGA_0_USER_IO1
- net FPGA_0_UER_IO10 renamed FPGA_0_USER_IO10
- net FPGA_0_UER_IO11 renamed FPGA_0_USER_IO11
- net FPGA_0_UER_IO12 renamed FPGA_0_USER_IO12
- net FPGA_0_UER_IO13 renamed FPGA_0_USER_IO13
- net FPGA_0_UER_IO14 renamed FPGA_0_USER_IO14
- net FPGA_0_UER_IO15 renamed FPGA_0_USER_IO15
- net FPGA_0_UER_IO16 renamed FPGA_0_USER_IO16
- net FPGA_0_UER_IO17 renamed FPGA_0_USER_IO17
- net FPGA_0_UER_IO18 renamed FPGA_0_USER_IO18
- net FPGA_0_UER_IO19 renamed FPGA_0_USER_IO19
- net FPGA_0_UER_IO2 renamed FPGA_0_USER_IO2
- net FPGA_0_UER_IO20 renamed FPGA_0_USER_IO20
- net FPGA_0_UER_IO21 renamed FPGA_0_USER_IO21
- net FPGA_0_UER_IO22 renamed FPGA_0_USER_IO22
- net FPGA_0_UER_IO23 renamed FPGA_0_USER_IO23
- net FPGA_0_UER_IO24 renamed FPGA_0_USER_IO24
- net FPGA_0_UER_IO25 renamed FPGA_0_USER_IO25
- net FPGA_0_UER_IO26 renamed FPGA_0_USER_IO26
- net FPGA_0_UER_IO27 renamed FPGA_0_USER_IO27
- net FPGA_0_UER_IO28 renamed FPGA_0_USER_IO28
- net FPGA_0_UER_IO29 renamed FPGA_0_USER_IO29
- net FPGA_0_UER_IO3 renamed FPGA_0_USER_IO3
- net FPGA_0_UER_IO30 renamed FPGA_0_USER_IO30
- net FPGA_0_UER_IO31 renamed FPGA_0_USER_IO31
- net FPGA_0_UER_IO32 renamed FPGA_0_USER_IO32
- net FPGA_0_UER_IO33 renamed FPGA_0_USER_IO33
- net FPGA_0_UER_IO34 renamed FPGA_0_USER_IO34
- net FPGA_0_UER_IO35 renamed FPGA_0_USER_IO35
- net FPGA_0_UER_IO36 renamed FPGA_0_USER_IO36
- net FPGA_0_UER_IO37 renamed FPGA_0_USER_IO37
- net FPGA_0_UER_IO38 renamed FPGA_0_USER_IO38
- net FPGA_0_UER_IO39 renamed FPGA_0_USER_IO39
- net FPGA_0_UER_IO4 renamed FPGA_0_USER_IO4
- net FPGA_0_UER_IO40 renamed FPGA_0_USER_IO40
- net FPGA_0_UER_IO41 renamed FPGA_0_USER_IO41
- net FPGA_0_UER_IO42 renamed FPGA_0_USER_IO42
- net FPGA_0_UER_IO43 renamed FPGA_0_USER_IO43
- net FPGA_0_UER_IO44 renamed FPGA_0_USER_IO44
- net FPGA_0_UER_IO45 renamed FPGA_0_USER_IO45
- net FPGA_0_UER_IO46 renamed FPGA_0_USER_IO46
- net FPGA_0_UER_IO47 renamed FPGA_0_USER_IO47
- net FPGA_0_UER_IO48 renamed FPGA_0_USER_IO48
- net FPGA_0_UER_IO49 renamed FPGA_0_USER_IO49
- net FPGA_0_UER_IO5 renamed FPGA_0_USER_IO5
- net FPGA_0_UER_IO6 renamed FPGA_0_USER_IO6
- net FPGA_0_UER_IO7 renamed FPGA_0_USER_IO7
- net FPGA_0_UER_IO8 renamed FPGA_0_USER_IO8
- net FPGA_0_UER_IO9 renamed FPGA_0_USER_IO9
- no-connect marks 2 -> 8

Commit message: Updated Layout
Connections:
- net FPGA_0_MCU_IO10 is gone; now on net FPGA_0_MCU_IO3: U20.Y21 (IO_L9P_T1_DQS_14)
- net FPGA_0_MCU_IO11 is gone; now on net FPGA_0_MCU_IO4: U20.Y22 (IO_L9N_T1_DQS_D13_14)
- net FPGA_0_MCU_IO12 is gone; now on net FPGA_0_MCU_IO5: U20.AB21 (IO_L10P_T1_D14_14)
- net FPGA_0_MCU_IO13 is gone; now on net FPGA_0_MCU_IO6: U20.AB22 (IO_L10N_T1_D15_14)
- net FPGA_0_MCU_IO14 is gone; now on net FPGA_0_MCU_IO7: U20.U20 (IO_L11P_T1_SRCC_14)
- net FPGA_0_MCU_IO15 is gone; now on net FPGA_0_MCU_IO8: U20.V20 (IO_L11N_T1_SRCC_14)
- net FPGA_0_MCU_IO9 is gone; now on net FPGA_0_MCU_IO2: U20.AA21 (IO_L8N_T1_D12_14)
- net FPGA_0_MCU_IO0: now also U20.W22 (IO_L7N_T1_D10_14); no longer U20.V22 (IO_L3N_T0_DQS_EMCCLK_14)
- net FPGA_0_MCU_IO1: now also U20.AA20 (IO_L8P_T1_D11_14); no longer U20.T21 (IO_L4P_T0_D04_14)
- net FPGA_0_MCU_IO2: no longer U20.U21 (IO_L4N_T0_D05_14)
- net FPGA_0_MCU_IO3: no longer U20.P19 (IO_L5P_T0_D06_14)
- net FPGA_0_MCU_IO4: no longer U20.R19 (IO_L5N_T0_D07_14)
- net FPGA_0_MCU_IO5: no longer U20.T20 (IO_L6N_T0_D08_VREF_14)
- net FPGA_0_MCU_IO6: no longer U20.W21 (IO_L7P_T1_D09_14)
- net FPGA_0_MCU_IO7: no longer U20.W22 (IO_L7N_T1_D10_14)
- net FPGA_0_MCU_IO8: no longer U20.AA20 (IO_L8P_T1_D11_14)
- net FPGA_0_SPI_MCU_CS: no longer names the net of U20.V17 (IO_L16P_T2_CSI_B_14)
- net FPGA_0_SPI_MCU_RX: no longer names the net of U20.W17 (IO_L16N_T2_A15_D31_14)
- net FPGA_0_SPI_MCU_SCLK: no longer names the net of U20.Y19 (IO_L13N_T2_MRCC_14)
- net FPGA_0_SPI_MCU_TX: no longer names the net of U20.AA18 (IO_L17P_T2_A14_D30_14)
- net FPGA_0_SW4: no longer names the net of U20.R14 (IO_L19N_T3_A09_D25_VREF_14)
- net FPGA_0_SW5: no longer names the net of U20.R18 (IO_L20P_T3_A08_D24_14)
- net FPGA_0_SW6: no longer names the net of U20.T18 (IO_L20N_T3_A07_D23_14)
- net FPGA_0_SW7: no longer names the net of U20.N17 (IO_L21P_T3_DQS_14)
- new net SMC_IO0: U20.T21 (IO_L4P_T0_D04_14)
- new net SMC_IO1: U20.U21 (IO_L4N_T0_D05_14)
- no-connect marks 8 -> 21
