File: DSN/FPGA_1.kicad_sch (KiCad schematic)
At the start: 132 parts, among them J5 Conn_Coaxial, Q3 AO3401A, Q4 2N7002K, SW7 SW_DIP_x03, SW8 SW_Push, SW9 SW_Push, U10 XC7A35T_FGG484, U11 SIT9120AI, U12 DSC1103BI2-135.0000, U13 REF3012, U14 IS25LP128F, U30 TC1047AVNBTR

Commit message: Updated Layout
Connections:
- net FPGA_1_MCU_IO10 is gone; now on net FPGA_1_MCU_IO3: U10.Y21 (IO_L9P_T1_DQS_14)
- net FPGA_1_MCU_IO11 is gone; now on net FPGA_1_MCU_IO4: U10.Y22 (IO_L9N_T1_DQS_D13_14)
- net FPGA_1_MCU_IO12 is gone; now on net FPGA_1_MCU_IO5: U10.AB21 (IO_L10P_T1_D14_14)
- net FPGA_1_MCU_IO13 is gone; now on net FPGA_1_MCU_IO6: U10.AB22 (IO_L10N_T1_D15_14)
- net FPGA_1_MCU_IO14 is gone; now on net FPGA_1_MCU_IO7: U10.U20 (IO_L11P_T1_SRCC_14)
- net FPGA_1_MCU_IO15 is gone; now on net FPGA_1_MCU_IO8: U10.V20 (IO_L11N_T1_SRCC_14)
- net FPGA_1_MCU_IO9 is gone; now on net FPGA_1_MCU_IO2: U10.AA21 (IO_L8N_T1_D12_14)
- net FPGA_1_LINK_IO0: now also U10.F21 (IO_25_16); no longer U10.J16 (IO_0_15)
- net FPGA_1_LINK_IO1: now also U10.G22 (IO_L24N_T3_16); no longer U10.H13 (IO_L1P_T0_AD0P_15)
- net FPGA_1_LINK_IO10: now also U10.C22 (IO_L20P_T3_16); no longer U10.H15 (IO_L5N_T0_AD9N_15)
- net FPGA_1_LINK_IO11: now also U10.C20 (IO_L19N_T3_VREF_16); no longer U10.H17 (IO_L6P_T0_15)
- net FPGA_1_LINK_IO12: now also U10.D20 (IO_L19P_T3_16); no longer U10.H18 (IO_L6N_T0_VREF_15)
- net FPGA_1_LINK_IO13: now also U10.F20 (IO_L18N_T2_16); no longer U10.J22 (IO_L7P_T1_AD2P_15)
- net FPGA_1_LINK_IO14: now also U10.F19 (IO_L18P_T2_16); no longer U10.H22 (IO_L7N_T1_AD2N_15)
- net FPGA_1_LINK_IO15: now also U10.A19 (IO_L17N_T2_16); no longer U10.H20 (IO_L8P_T1_AD10P_15)
- net FPGA_1_LINK_IO16: now also U10.A18 (IO_L17P_T2_16); no longer U10.G20 (IO_L8N_T1_AD10N_15)
- net FPGA_1_LINK_IO17: now also U10.A20 (IO_L16N_T2_16); no longer U10.K21 (IO_L9P_T1_DQS_AD3P_15)
- net FPGA_1_LINK_IO18: now also U10.B20 (IO_L16P_T2_16); no longer U10.K22 (IO_L9N_T1_DQS_AD3N_15)
- net FPGA_1_LINK_IO19: now also U10.E18 (IO_L15N_T2_DQS_16); no longer U10.M21 (IO_L10P_T1_AD11P_15)
- net FPGA_1_LINK_IO2: now also U10.G21 (IO_L24P_T3_16); no longer U10.G13 (IO_L1N_T0_AD0N_15)
- net FPGA_1_LINK_IO20: now also U10.F18 (IO_L15P_T2_DQS_16); no longer U10.L21 (IO_L10N_T1_AD11N_15)
- net FPGA_1_LINK_IO21: now also U10.D19 (IO_L14N_T2_SRCC_16); no longer U10.J20 (IO_L11P_T1_SRCC_15)
- net FPGA_1_LINK_IO22: now also U10.E19 (IO_L14P_T2_SRCC_16); no longer U10.J21 (IO_L11N_T1_SRCC_15)
- net FPGA_1_LINK_IO23: now also U10.C19 (IO_L13N_T2_MRCC_16); no longer U10.J19 (IO_L12P_T1_MRCC_15)
- net FPGA_1_LINK_IO24: now also U10.C18 (IO_L13P_T2_MRCC_16); no longer U10.H19 (IO_L12N_T1_MRCC_15)
- net FPGA_1_LINK_IO25: now also U10.C17 (IO_L12N_T1_MRCC_16); no longer U10.K18 (IO_L13P_T2_MRCC_15)
- net FPGA_1_LINK_IO26: now also U10.D17 (IO_L12P_T1_MRCC_16); no longer U10.K19 (IO_L13N_T2_MRCC_15)
- net FPGA_1_LINK_IO27: now also U10.B18 (IO_L11N_T1_SRCC_16); no longer U10.L19 (IO_L14P_T2_SRCC_15)
- net FPGA_1_LINK_IO28: now also U10.B17 (IO_L11P_T1_SRCC_16); no longer U10.L20 (IO_L14N_T2_SRCC_15)
- net FPGA_1_LINK_IO29: now also U10.A14 (IO_L10N_T1_16); no longer U10.N22 (IO_L15P_T2_DQS_15)
- net FPGA_1_LINK_IO3: now also U10.D21 (IO_L23N_T3_16); no longer U10.G15 (IO_L2P_T0_AD8P_15)
- net FPGA_1_LINK_IO30: now also U10.A13 (IO_L10P_T1_16); no longer U10.M22 (IO_L15N_T2_DQS_ADV_B_15)
- net FPGA_1_LINK_IO31: now also U10.A16 (IO_L9N_T1_DQS_16); no longer U10.M18 (IO_L16P_T2_A28_15)
- net FPGA_1_LINK_IO32: now also U10.A15 (IO_L9P_T1_DQS_16); no longer U10.L18 (IO_L16N_T2_A27_15)
- net FPGA_1_LINK_IO33: now also U10.B13 (IO_L8N_T1_16); no longer U10.N18 (IO_L17P_T2_A26_15)
- net FPGA_1_LINK_IO34: now also U10.C13 (IO_L8P_T1_16); no longer U10.N19 (IO_L17N_T2_A25_15)
- net FPGA_1_LINK_IO35: now also U10.B16 (IO_L7N_T1_16); no longer U10.N20 (IO_L18P_T2_A24_15)
- net FPGA_1_LINK_IO36: now also U10.B15 (IO_L7P_T1_16); no longer U10.M20 (IO_L18N_T2_A23_15)
- net FPGA_1_LINK_IO37: now also U10.D15 (IO_L6N_T0_VREF_16); no longer U10.K13 (IO_L19P_T3_A22_15)
- net FPGA_1_LINK_IO38: now also U10.D14 (IO_L6P_T0_16); no longer U10.K14 (IO_L19N_T3_A21_VREF_15)
- net FPGA_1_LINK_IO39: now also U10.D16 (IO_L5N_T0_16); no longer U10.M13 (IO_L20P_T3_A20_15)
- net FPGA_1_LINK_IO4: now also U10.E21 (IO_L23P_T3_16); no longer U10.G16 (IO_L2N_T0_AD8N_15)
- net FPGA_1_LINK_IO40: now also U10.E16 (IO_L5P_T0_16); no longer U10.L13 (IO_L20N_T3_A19_15)
- net FPGA_1_LINK_IO41: now also U10.E14 (IO_L4N_T0_16); no longer U10.K17 (IO_L21P_T3_DQS_15)
- net FPGA_1_LINK_IO42: now also U10.E13 (IO_L4P_T0_16); no longer U10.J17 (IO_L21N_T3_DQS_A18_15)
- net FPGA_1_LINK_IO43: now also U10.C15 (IO_L3N_T0_DQS_16); no longer U10.L14 (IO_L22P_T3_A17_15)
- net FPGA_1_LINK_IO44: now also U10.C14 (IO_L3P_T0_DQS_16); no longer U10.L15 (IO_L22N_T3_A16_15)
- net FPGA_1_LINK_IO45: now also U10.E17 (IO_L2N_T0_16); no longer U10.L16 (IO_L23P_T3_FOE_B_15)
- net FPGA_1_LINK_IO46: now also U10.F16 (IO_L2P_T0_16); no longer U10.K16 (IO_L23N_T3_FWE_B_15)
- net FPGA_1_LINK_IO47: now also U10.F14 (IO_L1N_T0_16); no longer U10.M15 (IO_L24P_T3_RS1_15)
- net FPGA_1_LINK_IO48: now also U10.F13 (IO_L1P_T0_16); no longer U10.M16 (IO_L24N_T3_RS0_15)
- net FPGA_1_LINK_IO49: now also U10.F15 (IO_0_16); no longer U10.M17 (IO_25_15)
- net FPGA_1_LINK_IO5: now also U10.D22 (IO_L22N_T3_16); no longer U10.J14 (IO_L3P_T0_DQS_AD1P_15)
- net FPGA_1_LINK_IO50: now also U10.M17 (IO_25_15); no longer U10.F15 (IO_0_16)
- net FPGA_1_LINK_IO51: now also U10.M16 (IO_L24N_T3_RS0_15); no longer U10.F13 (IO_L1P_T0_16)
- net FPGA_1_LINK_IO52: now also U10.M15 (IO_L24P_T3_RS1_15); no longer U10.F14 (IO_L1N_T0_16)
- net FPGA_1_LINK_IO53: now also U10.K16 (IO_L23N_T3_FWE_B_15); no longer U10.F16 (IO_L2P_T0_16)
- net FPGA_1_LINK_IO54: now also U10.L16 (IO_L23P_T3_FOE_B_15); no longer U10.E17 (IO_L2N_T0_16)
- net FPGA_1_LINK_IO55: now also U10.L15 (IO_L22N_T3_A16_15); no longer U10.C14 (IO_L3P_T0_DQS_16)
- net FPGA_1_LINK_IO56: now also U10.L14 (IO_L22P_T3_A17_15); no longer U10.C15 (IO_L3N_T0_DQS_16)
- net FPGA_1_LINK_IO57: now also U10.J17 (IO_L21N_T3_DQS_A18_15); no longer U10.E13 (IO_L4P_T0_16)
- net FPGA_1_LINK_IO58: now also U10.K17 (IO_L21P_T3_DQS_15); no longer U10.E14 (IO_L4N_T0_16)
- net FPGA_1_LINK_IO59: now also U10.L13 (IO_L20N_T3_A19_15); no longer U10.E16 (IO_L5P_T0_16)
- net FPGA_1_LINK_IO6: now also U10.E22 (IO_L22P_T3_16); no longer U10.H14 (IO_L3N_T0_DQS_AD1N_15)
- net FPGA_1_LINK_IO60: now also U10.M13 (IO_L20P_T3_A20_15); no longer U10.D16 (IO_L5N_T0_16)
- net FPGA_1_LINK_IO61: now also U10.K14 (IO_L19N_T3_A21_VREF_15); no longer U10.D14 (IO_L6P_T0_16)
- net FPGA_1_LINK_IO62: now also U10.K13 (IO_L19P_T3_A22_15); no longer U10.D15 (IO_L6N_T0_VREF_16)
- net FPGA_1_LINK_IO63: now also U10.M20 (IO_L18N_T2_A23_15); no longer U10.B15 (IO_L7P_T1_16)
- net FPGA_1_LINK_IO64: now also U10.N20 (IO_L18P_T2_A24_15); no longer U10.B16 (IO_L7N_T1_16)
- net FPGA_1_LINK_IO65: now also U10.N19 (IO_L17N_T2_A25_15); no longer U10.C13 (IO_L8P_T1_16)
- net FPGA_1_LINK_IO66: now also U10.N18 (IO_L17P_T2_A26_15); no longer U10.B13 (IO_L8N_T1_16)
- net FPGA_1_LINK_IO67: now also U10.L18 (IO_L16N_T2_A27_15); no longer U10.A15 (IO_L9P_T1_DQS_16)
- net FPGA_1_LINK_IO68: now also U10.M18 (IO_L16P_T2_A28_15); no longer U10.A16 (IO_L9N_T1_DQS_16)
- net FPGA_1_LINK_IO69: now also U10.M22 (IO_L15N_T2_DQS_ADV_B_15); no longer U10.A13 (IO_L10P_T1_16)
- net FPGA_1_LINK_IO7: now also U10.A21 (IO_L21N_T3_DQS_16); no longer U10.G17 (IO_L4P_T0_15)
- net FPGA_1_LINK_IO70: now also U10.N22 (IO_L15P_T2_DQS_15); no longer U10.A14 (IO_L10N_T1_16)
- net FPGA_1_LINK_IO71: now also U10.L20 (IO_L14N_T2_SRCC_15); no longer U10.B17 (IO_L11P_T1_SRCC_16)
- net FPGA_1_LINK_IO72: now also U10.L19 (IO_L14P_T2_SRCC_15); no longer U10.B18 (IO_L11N_T1_SRCC_16)
- net FPGA_1_LINK_IO73: now also U10.K19 (IO_L13N_T2_MRCC_15); no longer U10.D17 (IO_L12P_T1_MRCC_16)
- net FPGA_1_LINK_IO74: now also U10.K18 (IO_L13P_T2_MRCC_15); no longer U10.C17 (IO_L12N_T1_MRCC_16)
- net FPGA_1_LINK_IO75: now also U10.H19 (IO_L12N_T1_MRCC_15); no longer U10.C18 (IO_L13P_T2_MRCC_16)
- net FPGA_1_LINK_IO76: now also U10.J19 (IO_L12P_T1_MRCC_15); no longer U10.C19 (IO_L13N_T2_MRCC_16)
- net FPGA_1_LINK_IO77: now also U10.J21 (IO_L11N_T1_SRCC_15); no longer U10.E19 (IO_L14P_T2_SRCC_16)
- net FPGA_1_LINK_IO78: now also U10.J20 (IO_L11P_T1_SRCC_15); no longer U10.D19 (IO_L14N_T2_SRCC_16)
- net FPGA_1_LINK_IO79: now also U10.L21 (IO_L10N_T1_AD11N_15); no longer U10.F18 (IO_L15P_T2_DQS_16)
- net FPGA_1_LINK_IO8: now also U10.B21 (IO_L21P_T3_DQS_16); no longer U10.G18 (IO_L4N_T0_15)
- net FPGA_1_LINK_IO80: now also U10.M21 (IO_L10P_T1_AD11P_15); no longer U10.E18 (IO_L15N_T2_DQS_16)
- net FPGA_1_LINK_IO81: now also U10.K22 (IO_L9N_T1_DQS_AD3N_15); no longer U10.B20 (IO_L16P_T2_16)
- net FPGA_1_LINK_IO82: now also U10.K21 (IO_L9P_T1_DQS_AD3P_15); no longer U10.A20 (IO_L16N_T2_16)
- net FPGA_1_LINK_IO83: now also U10.G20 (IO_L8N_T1_AD10N_15); no longer U10.A18 (IO_L17P_T2_16)
- net FPGA_1_LINK_IO84: now also U10.H20 (IO_L8P_T1_AD10P_15); no longer U10.A19 (IO_L17N_T2_16)
- net FPGA_1_LINK_IO85: now also U10.H22 (IO_L7N_T1_AD2N_15); no longer U10.F19 (IO_L18P_T2_16)
- net FPGA_1_LINK_IO86: now also U10.J22 (IO_L7P_T1_AD2P_15); no longer U10.F20 (IO_L18N_T2_16)
- net FPGA_1_LINK_IO87: now also U10.H18 (IO_L6N_T0_VREF_15); no longer U10.D20 (IO_L19P_T3_16)
- net FPGA_1_LINK_IO88: now also U10.H17 (IO_L6P_T0_15); no longer U10.C20 (IO_L19N_T3_VREF_16)
- net FPGA_1_LINK_IO89: now also U10.H15 (IO_L5N_T0_AD9N_15); no longer U10.C22 (IO_L20P_T3_16)
- net FPGA_1_LINK_IO9: now also U10.B22 (IO_L20N_T3_16); no longer U10.J15 (IO_L5P_T0_AD9P_15)
- net FPGA_1_LINK_IO90: now also U10.J15 (IO_L5P_T0_AD9P_15); no longer U10.B22 (IO_L20N_T3_16)
- net FPGA_1_LINK_IO91: now also U10.G18 (IO_L4N_T0_15); no longer U10.B21 (IO_L21P_T3_DQS_16)
- net FPGA_1_LINK_IO92: now also U10.G17 (IO_L4P_T0_15); no longer U10.A21 (IO_L21N_T3_DQS_16)
- net FPGA_1_LINK_IO93: now also U10.H14 (IO_L3N_T0_DQS_AD1N_15); no longer U10.E22 (IO_L22P_T3_16)
- net FPGA_1_LINK_IO94: now also U10.J14 (IO_L3P_T0_DQS_AD1P_15); no longer U10.D22 (IO_L22N_T3_16)
- net FPGA_1_LINK_IO95: now also U10.G16 (IO_L2N_T0_AD8N_15); no longer U10.E21 (IO_L23P_T3_16)
- net FPGA_1_LINK_IO96: now also U10.G15 (IO_L2P_T0_AD8P_15); no longer U10.D21 (IO_L23N_T3_16)
- net FPGA_1_LINK_IO97: now also U10.G13 (IO_L1N_T0_AD0N_15); no longer U10.G21 (IO_L24P_T3_16)
- net FPGA_1_LINK_IO98: now also U10.H13 (IO_L1P_T0_AD0P_15); no longer U10.G22 (IO_L24N_T3_16)
- net FPGA_1_LINK_IO99: now also U10.J16 (IO_0_15); no longer U10.F21 (IO_25_16)
- net FPGA_1_MCU_IO0: now also U10.W22 (IO_L7N_T1_D10_14); no longer U10.V22 (IO_L3N_T0_DQS_EMCCLK_14)
- net FPGA_1_MCU_IO1: now also U10.AA20 (IO_L8P_T1_D11_14); no longer U10.T21 (IO_L4P_T0_D04_14)
- net FPGA_1_MCU_IO2: no longer U10.U21 (IO_L4N_T0_D05_14)
- net FPGA_1_MCU_IO3: no longer U10.P19 (IO_L5P_T0_D06_14)
- net FPGA_1_MCU_IO4: no longer U10.R19 (IO_L5N_T0_D07_14)
- net FPGA_1_MCU_IO5: no longer U10.T20 (IO_L6N_T0_D08_VREF_14)
- net FPGA_1_MCU_IO6: no longer U10.W21 (IO_L7P_T1_D09_14)
- net FPGA_1_MCU_IO7: no longer U10.W22 (IO_L7N_T1_D10_14)
- net FPGA_1_MCU_IO8: no longer U10.AA20 (IO_L8P_T1_D11_14)
- net FPGA_1_SPI_MCU_CS: no longer names the net of U10.V17 (IO_L16P_T2_CSI_B_14)
- net FPGA_1_SPI_MCU_RX: no longer names the net of U10.W17 (IO_L16N_T2_A15_D31_14)
- net FPGA_1_SPI_MCU_SCLK: no longer names the net of U10.Y19 (IO_L13N_T2_MRCC_14)
- net FPGA_1_SPI_MCU_TX: no longer names the net of U10.AA18 (IO_L17P_T2_A14_D30_14)
- net FPGA_1_SW4: no longer names the net of U10.R14 (IO_L19N_T3_A09_D25_VREF_14)
- net FPGA_1_SW5: no longer names the net of U10.R18 (IO_L20P_T3_A08_D24_14)
- net FPGA_1_SW6: no longer names the net of U10.T18 (IO_L20N_T3_A07_D23_14)
- net FPGA_1_SW7: no longer names the net of U10.N17 (IO_L21P_T3_DQS_14)
- new net SMC_IO2: U10.T21 (IO_L4P_T0_D04_14)
- new net SMC_IO3: U10.U21 (IO_L4N_T0_D05_14)
- no-connect marks 17 -> 30
