File: DSN/RP2040_MCU.kicad_sch (KiCad schematic)
At the start: 41 parts

Commit message: Updated Layout
Parts:
- removed D?: BZV55B5V6, Diode_SMD:D_MiniMELF, symbol Diode:BZV55B5V6
- removed TP? (x3): TestPoint_Probe, TestPoint:TestPoint_Loop_D2.50mm_Drill1.85mm, symbol Connector:TestPoint_Probe
- removed Y?: Crystal_GND23, Crystal:Crystal_SMD_3225-4Pin_3.2x2.5mm, symbol Device:Crystal_GND23
- added D8: 5.6V Zener, Diode_SMD:D_SOD-123, symbol Device:D_Zener
- added TP19, TP20, TP4: TestPoint_Probe, TestPoint:TestPoint_Loop_D1.80mm_Drill1.0mm_Beaded, symbol Connector:TestPoint_Probe
- added Y2: Crystal_GND24, Crystal:Crystal_SMD_3225-4Pin_3.2x2.5mm, symbol Device:Crystal_GND24
- gave numbers to parts that had none: 36
Connections:
- net +3V3_RPi22_AUX is gone; now on net +3V3_RPi2_AUX: R11.2
- net +3V3_RPi2_AUX: now also TP19.1
- net +5V: now also D8.1 (K)
- net GND: now also Y2.2, Y2.4
- net RPi2_1V1: now also TP4.1
- net VBUS_AUX_RPi2: now also TP20.1
- net XI_RPi2: now also Y2.1
- net XO_RPi2: now also Y2.3
- net at Q2.4 (G), R20.1: now also D8.2 (A)
- net FPGA_0_GPIO1: now reaches U32.11 (GPIO8)
- net FPGA_0_GPIO2: now reaches U32.12 (GPIO9)
- net FPGA_0_GPIO3: now reaches U32.13 (GPIO10)
- net FPGA_0_GPIO4: now reaches U32.14 (GPIO11)
- net FPGA_0_GPIO5: now reaches U32.15 (GPIO12)
- net FPGA_0_GPIO6: now reaches U32.16 (GPIO13)
- net FPGA_0_GPIO7: now reaches U32.17 (GPIO14)
- net FPGA_0_GPIO8: now reaches U32.18 (GPIO15)
- net FPGA_1_GPIO0: now reaches U32.27 (GPIO16)
- net FPGA_1_GPIO1: now reaches U32.28 (GPIO17)
- net FPGA_1_GPIO2: now reaches U32.29 (GPIO18)
- net FPGA_1_GPIO3: now reaches U32.30 (GPIO19)
- net FPGA_1_GPIO4: now reaches U32.31 (GPIO20)
- net FPGA_1_GPIO5: now reaches U32.32 (GPIO21)
- net FPGA_1_GPIO6: now reaches U32.34 (GPIO22)
- net FPGA_1_GPIO7: now reaches U32.35 (GPIO23)
- net FPGA_1_GPIO8: now reaches U32.36 (GPIO24)
- net FPGA_0_GPIO0: now reaches U32.9 (GPIO7)
- no-connect marks 5 -> 15
Other:
- note added: "MCU"
- note added: "MCU Power"
- note removed: "SMC"
- note removed: "SMC Power"
