File: DSN/ArtixDuo.kicad_sch (KiCad schematic)
At the start: 0 parts

Commit message: Updated Layout
Other:
- note removed: "MMXRT1062 Teensy 4.1"

Commit message: Layout Update
Other:
- note added: "100-Bit Interface Bus Multi_purpose"
- note added: "50X GPIO"
- note added: "512Mb PSRAM"
- note added: "9X GPIO"
- note added: "Octal SPI Interface 400MB/s"
- note removed: "16X GPIO"
- note removed: "48X GPIO"
- note removed: "512Mb DDR3"
- note removed: "64_Bit Interface Bus Multi_purpose, SPI, I2C. Parallel, SERDES, GTX Gb/s"
- note removed: "DDR3 Memory Interface"
- note removed: "SPI1 40Mb/s"
- note removed: "SPI2 40Mb/s"
Changed lines of the file:
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@@
     (stroke (width 0.5) (type solid) (color 0 0 0 0))
-  )
-  (polyline (pts (xy 278.765 217.17) (xy 278.765 183.515))
-    (stroke (width 0.5) (type solid) (color 255 54 39 1))
   )
   (polyline (pts (xy 273.05 217.17) (xy 273.05 177.165))
@@
     (stroke (width 0) (type default) (color 0 0 0 0))
   )
-  (polyline (pts (xy 256.54 182.88) (xy 218.44 182.88))
-    (stroke (width 0.5) (type solid) (color 255 54 39 1))
-  )
   (polyline (pts (xy 219.71 252.73) (xy 219.71 217.17))
     (stroke (width 0) (type default) (color 0 0 0 0))
@@
     (stroke (width 0.5) (type solid) (color 0 0 0 0))
   )
-  (polyline (pts (xy 278.765 183.515) (xy 304.8 183.515))
-    (stroke (width 0.5) (type solid) (color 255 54 39 1))
-  )
   (polyline (pts (xy 304.8 187.96) (xy 341.63 187.96))
     (stroke (width 0) (type default) (color 0 0 0 0))
@@
     (stroke (width 1) (type solid) (color 255 54 52 1))
   )
-  (polyline (pts (xy 256.54 217.17) (xy 256.54 182.88))
-    (stroke (width 0.5) (type solid) (color 255 54 39 1))
-  )
   (polyline (pts (xy 199.39 132.08) (xy 199.39 152.4))
     (stroke (width 0.5) (type solid) (color 255 48 222 1))
@@
     (effects (font (size 1.27 1.27)) (justify left bottom))
   )
-  (text "64_Bit Interface Bus\nMulti_purpose,\nSPI, I2C. Parallel, \nSERDES, GTX Gb/s "
-    (at 253.365 167.64 0)
+  (text "100-Bit Interface Bus\nMulti_purpose\n" (at 253.365 167.64 0)
     (effects (font (size 1.27 1.27)) (justify left bottom))
   )
-  (text "SPI2\n40Mb/s" (at 287.02 187.96 0)
+  (text "512Mb PSRAM\n" (at 372.745 170.18 0)
     (effects (font (size 1.27 1.27)) (justify left bottom))
   )
-  (text "512Mb DDR3" (at 372.745 170.18 0)
+  (text "Octal SPI Interface \n400MB/s" (at 345.44 165.735 0)
     (effects (font (size 1.27 1.27)) (justify left bottom))
   )
-  (text "DDR3 Memory Interface" (at 345.44 165.735 0)
-    (effects (font (size 1.27 1.27)) (justify left bottom))
-  )
-  (text "48X GPIO" (at 342.265 137.795 0)
+  (text "50X GPIO" (at 342.265 137.795 0)
     (effects (font (size 1.27 1.27)) (justify left bottom))
   )
@@
     (effects (font (size 1.27 1.27)) (justify left bottom))
   )
-  (text "SPI1\n40Mb/s" (at 233.045 187.325 0)
-    (effects (font (size 1.27 1.27)) (justify left bottom))
-  )
-  (text "16X GPIO" (at 233.68 174.625 0)
+  (text "9X GPIO" (at 233.68 174.625 0)
     (effects (font (size 1.27 1.27)) (justify left bottom))
   )
@@
     (effects (font (size 1.27 1.27)) (justify left bottom))
   )
-  (text "48X GPIO" (at 218.44 138.43 0)
+  (text "50X GPIO" (at 218.44 138.43 0)
     (effects (font (size 1.27 1.27)) (justify left bottom))
   )
-  (text "16X GPIO" (at 286.385 175.26 0)
+  (text "9X GPIO" (at 286.385 175.26 0)
     (effects (font (size 1.27 1.27)) (justify left bottom))
   )
@@
       (reference "#PWR0591") (unit 1) (value "GND") (footprint "")
     )
+    (path "/f0a2a446-6282-4abd-9508-b4877da61a24/f98464e5-a153-4f40-ae54-207e51516a2b/a42956c4-cbfd-424b-90c1-d40a89ebf59a"
+      (reference "#PWR?") (unit 1) (value "GND") (footprint "")
+    )
     (path "/f0a2a446-6282-4abd-9508-b4877da61a24/24a28848-987b-4c21-a6fa-86d9002a4152"
