File: DSN/IO.kicad_sch (KiCad schematic)
At the start: 49 parts

Commit message: Updates
Changed FPGA user io from 100 to 50 per chip, added 4 pmod per FPGA, added 8x buttons + led's, added SMA connectors for FPGA0 GTP.
Parts:
- removed C? (x4): 10uF, Capacitor_SMD:C_0805_2012Metric, symbol Device:C_Small
- removed J? (x2): Conn_02x40_Odd_Even, symbol Connector_Generic:Conn_02x40_Odd_Even
- added C? (x8): 100nF, Capacitor_SMD:C_0402_1005Metric, symbol Device:C
- added C? (x18): DNF, Capacitor_SMD:C_0402_1005Metric, symbol Device:C_Small
- added D? (x8): LED GREEN, LED_SMD:LED_0603_1608Metric, symbol Device:LED
- added J? (x8): Conn_02x06_Odd_Even, symbol Connector_Generic:Conn_02x06_Odd_Even
- added J? (x9): 5-1814832-1, digikey-footprints:RF_SMA_Vertical_5-1814832-1, symbol dk_Coaxial-Connectors-RF:5-1814832-1
- added Q? (x8): 2N7002, digikey-footprints:SOT-23-3, symbol dk_Transistors-FETs-MOSFETs-Single:2N7002
- added R? (x24): 3K3, Resistor_SMD:R_0402_1005Metric, symbol Device:R_US
- added R? (x9): 0R, Resistor_SMD:R_0402_1005Metric, symbol Device:R_US
- added R? (x8): 100K, Resistor_SMD:R_0402_1005Metric, symbol Device:R_US
- added SW? (x8): SW_Push, symbol Switch:SW_Push
Connections:
- net FPGA_1_USER_IO50 is gone; now on net FPGA_1_USER_IO42: J?.21 (Pin_21)
- net FPGA_1_USER_IO51 is gone; now on net FPGA_1_USER_IO43: J?.23 (Pin_23)
- net FPGA_1_USER_IO52 is gone; now on net FPGA_1_USER_IO44: J?.25 (Pin_25)
- net FPGA_1_USER_IO53 is gone; now on net FPGA_1_USER_IO45: J?.27 (Pin_27)
- net FPGA_1_USER_IO54 is gone; now on net FPGA_1_USER_IO46: J?.29 (Pin_29)
- net FPGA_1_USER_IO55 is gone; now on net FPGA_1_USER_IO47: J?.31 (Pin_31)
- net FPGA_1_USER_IO56 is gone; now on net FPGA_1_USER_IO48: J?.33 (Pin_33)
- net FPGA_1_USER_IO57 is gone; now on net FPGA_1_USER_IO49: J?.35 (Pin_35)
- net FPGA_1_USER_IO58 is gone; now on net FPGA_0_USER_IO0: J?.37 (Pin_37)
- net FPGA_1_USER_IO59 is gone; now on net FPGA_0_USER_IO1: J?.39 (Pin_39)
- net FPGA_1_USER_IO60 is gone; now on net FPGA_0_USER_IO2: J?.41 (Pin_41)
- net FPGA_1_USER_IO61 is gone; now on net FPGA_0_USER_IO3: J?.43 (Pin_43)
- net FPGA_1_USER_IO62 is gone; now on net FPGA_0_USER_IO4: J?.45 (Pin_45)
- net FPGA_1_USER_IO63 is gone; now on net FPGA_0_USER_IO5: J?.47 (Pin_47)
- net FPGA_1_USER_IO64 is gone; now on net FPGA_0_USER_IO6: J?.49 (Pin_49)
- net FPGA_1_USER_IO65 is gone; now on net FPGA_0_USER_IO7: J?.51 (Pin_51)
- net FPGA_1_USER_IO66 is gone; now on net FPGA_0_USER_IO8: J?.53 (Pin_53)
- net FPGA_1_USER_IO67 is gone; now on net FPGA_0_USER_IO9: J?.55 (Pin_55)
- net FPGA_1_USER_IO68 is gone; now on net FPGA_0_USER_IO10: J?.57 (Pin_57)
- net FPGA_1_USER_IO69 is gone; now on net FPGA_0_USER_IO11: J?.59 (Pin_59)
- net FPGA_1_USER_IO70 is gone; now on net FPGA_0_USER_IO12: J?.61 (Pin_61)
- net FPGA_1_USER_IO71 is gone; now on net FPGA_0_USER_IO13: J?.63 (Pin_63)
- net FPGA_1_USER_IO72 is gone; now on net FPGA_0_USER_IO14: J?.65 (Pin_65)
- net FPGA_1_USER_IO73 is gone; now on net FPGA_0_USER_IO15: J?.67 (Pin_67)
- net FPGA_1_USER_IO74 is gone; now on net FPGA_0_USER_IO16: J?.69 (Pin_69)
- net FPGA_1_USER_IO75 is gone; now on net FPGA_0_USER_IO17: J?.71 (Pin_71)
- net FPGA_1_USER_IO76 is gone; now on net FPGA_0_USER_IO18: J?.73 (Pin_73)
- net FPGA_1_USER_IO77 is gone; now on net FPGA_0_USER_IO19: J?.75 (Pin_75)
- net FPGA_1_USER_IO78 is gone; now on net FPGA_0_USER_IO20: J?.77 (Pin_77)
- net FPGA_1_USER_IO79 is gone; now on net FPGA_0_USER_IO21: J?.79 (Pin_79)
- net FPGA_1_USER_IO80 is gone; now on net +3V3: J?.1 (Pin_1)
- net FPGA_1_USER_IO81 is gone; now on net +3V3: J?.3 (Pin_3)
- net FPGA_1_USER_IO82 is gone; now on net +5V: J?.5 (Pin_5)
- net FPGA_1_USER_IO83 is gone; now on net +5V: J?.7 (Pin_7)
- net FPGA_1_USER_IO84 is gone; now on net FPGA_0_USER_IO22: J?.9 (Pin_9)
- net FPGA_1_USER_IO85 is gone; now on net FPGA_0_USER_IO23: J?.11 (Pin_11)
- net FPGA_1_USER_IO86 is gone; now on net FPGA_0_USER_IO24: J?.13 (Pin_13)
- net FPGA_1_USER_IO87 is gone; now on net FPGA_0_USER_IO25: J?.15 (Pin_15)
- net FPGA_1_USER_IO88 is gone; now on net FPGA_0_USER_IO26: J?.17 (Pin_17)
- net FPGA_1_USER_IO89 is gone; now on net FPGA_0_USER_IO27: J?.19 (Pin_19)
- net FPGA_1_USER_IO90 is gone; now on net FPGA_0_USER_IO28: J?.21 (Pin_21)
- net FPGA_1_USER_IO91 is gone; now on net FPGA_0_USER_IO29: J?.23 (Pin_23)
- net FPGA_1_USER_IO92 is gone; now on net FPGA_0_USER_IO30: J?.25 (Pin_25)
- net FPGA_1_USER_IO93 is gone; now on net FPGA_0_USER_IO31: J?.27 (Pin_27)
- net FPGA_1_USER_IO94 is gone; now on net FPGA_0_USER_IO32: J?.29 (Pin_29)
- net FPGA_1_USER_IO95 is gone; now on net FPGA_0_USER_IO33: J?.31 (Pin_31)
- net FPGA_1_USER_IO96 is gone; now on net FPGA_0_USER_IO34: J?.33 (Pin_33)
- net FPGA_1_USER_IO97 is gone; now on net FPGA_0_USER_IO35: J?.35 (Pin_35)
- net FPGA_1_USER_IO98 is gone; now on net FPGA_0_USER_IO36: J?.37 (Pin_37)
- net FPGA_1_USER_IO99 is gone; now on net FPGA_0_USER_IO37: J?.39 (Pin_39)
- net +3V3: now also J?.1 (Pin_1), J?.1 (Pin_1), J?.3 (Pin_3), J?.3 (Pin_3), J?.1 (Pin_1), J?.1 (Pin_1), J?.1 (Pin_1), J?.1 (Pin_1), J?.1 (Pin_1), J?.1 (Pin_1), J?.1 (Pin_1), J?.1 (Pin_1), J?.2 (Pin_2), J?.2 (Pin_2), J?.2 (Pin_2), J?.2 (Pin_2), J?.2 (Pin_2), J?.2 (Pin_2), J?.2 (Pin_2), J?.2 (Pin_2), R?.1, R?.1, R?.1, R?.1, R?.1, R?.1, R?.1, R?.1, R?.1, R?.1, R?.1, R?.1, R?.1, R?.1, R?.1, R?.1
- net +5V: now also J?.5 (Pin_5), J?.5 (Pin_5), J?.7 (Pin_7), J?.7 (Pin_7)
- net FPGA_0_USER_IO0: no longer J?.41 (Pin_41)
- net FPGA_0_USER_IO1: no longer J?.43 (Pin_43)
- net FPGA_0_USER_IO10: no longer J?.61 (Pin_61)
- net FPGA_0_USER_IO11: no longer J?.63 (Pin_63)
- net FPGA_0_USER_IO12: no longer J?.65 (Pin_65)
- net FPGA_0_USER_IO13: no longer J?.67 (Pin_67)
- net FPGA_0_USER_IO14: no longer J?.69 (Pin_69)
- net FPGA_0_USER_IO15: no longer J?.71 (Pin_71)
- net FPGA_0_USER_IO16: no longer J?.73 (Pin_73)
- net FPGA_0_USER_IO17: no longer J?.75 (Pin_75)
- net FPGA_0_USER_IO18: no longer J?.77 (Pin_77)
- net FPGA_0_USER_IO19: no longer J?.79 (Pin_79)
- net FPGA_0_USER_IO2: no longer J?.45 (Pin_45)
- net FPGA_0_USER_IO3: no longer J?.47 (Pin_47)
- net FPGA_0_USER_IO38: now also J?.41 (Pin_41)
- net FPGA_0_USER_IO39: now also J?.43 (Pin_43)
- net FPGA_0_USER_IO4: no longer J?.49 (Pin_49)
- net FPGA_0_USER_IO40: now also J?.45 (Pin_45)
- net FPGA_0_USER_IO41: now also J?.47 (Pin_47)
- net FPGA_0_USER_IO42: now also J?.49 (Pin_49)
- net FPGA_0_USER_IO43: now also J?.51 (Pin_51)
- net FPGA_0_USER_IO44: now also J?.53 (Pin_53)
- net FPGA_0_USER_IO45: now also J?.55 (Pin_55)
- net FPGA_0_USER_IO46: now also J?.57 (Pin_57)
- net FPGA_0_USER_IO47: now also J?.59 (Pin_59)
- net FPGA_0_USER_IO48: now also J?.61 (Pin_61)
- net FPGA_0_USER_IO49: now also J?.63 (Pin_63)
- net FPGA_0_USER_IO5: no longer J?.51 (Pin_51)
- net FPGA_0_USER_IO6: no longer J?.53 (Pin_53)
- net FPGA_0_USER_IO7: no longer J?.55 (Pin_55)
- net FPGA_0_USER_IO8: no longer J?.57 (Pin_57)
- net FPGA_0_USER_IO9: no longer J?.59 (Pin_59)
- net FPGA_1_USER_IO0: now also J?.9 (Pin_9); no longer J?.1 (Pin_1)
- net FPGA_1_USER_IO1: now also J?.11 (Pin_11); no longer J?.3 (Pin_3)
- net FPGA_1_USER_IO10: now also J?.29 (Pin_29); no longer J?.21 (Pin_21)
- net FPGA_1_USER_IO11: now also J?.31 (Pin_31); no longer J?.23 (Pin_23)
- net FPGA_1_USER_IO12: now also J?.33 (Pin_33); no longer J?.25 (Pin_25)
- net FPGA_1_USER_IO13: now also J?.35 (Pin_35); no longer J?.27 (Pin_27)
- net FPGA_1_USER_IO14: now also J?.37 (Pin_37); no longer J?.29 (Pin_29)
- net FPGA_1_USER_IO15: now also J?.39 (Pin_39); no longer J?.31 (Pin_31)
- net FPGA_1_USER_IO16: now also J?.41 (Pin_41); no longer J?.33 (Pin_33)
- net FPGA_1_USER_IO17: now also J?.43 (Pin_43); no longer J?.35 (Pin_35)
- net FPGA_1_USER_IO18: now also J?.45 (Pin_45); no longer J?.37 (Pin_37)
- net FPGA_1_USER_IO19: now also J?.47 (Pin_47); no longer J?.39 (Pin_39)
- net FPGA_1_USER_IO2: now also J?.13 (Pin_13); no longer J?.5 (Pin_5)
- net FPGA_1_USER_IO20: now also J?.49 (Pin_49); no longer J?.41 (Pin_41)
- net FPGA_1_USER_IO21: now also J?.51 (Pin_51); no longer J?.43 (Pin_43)
- net FPGA_1_USER_IO22: now also J?.53 (Pin_53); no longer J?.45 (Pin_45)
- net FPGA_1_USER_IO23: now also J?.55 (Pin_55); no longer J?.47 (Pin_47)
- net FPGA_1_USER_IO24: now also J?.57 (Pin_57); no longer J?.49 (Pin_49)
- net FPGA_1_USER_IO25: now also J?.59 (Pin_59); no longer J?.51 (Pin_51)
- net FPGA_1_USER_IO26: now also J?.61 (Pin_61); no longer J?.53 (Pin_53)
- net FPGA_1_USER_IO27: now also J?.63 (Pin_63); no longer J?.55 (Pin_55)
- net FPGA_1_USER_IO28: now also J?.65 (Pin_65); no longer J?.57 (Pin_57)
- net FPGA_1_USER_IO29: now also J?.67 (Pin_67); no longer J?.59 (Pin_59)
- net FPGA_1_USER_IO3: now also J?.15 (Pin_15); no longer J?.7 (Pin_7)
- net FPGA_1_USER_IO30: now also J?.69 (Pin_69); no longer J?.61 (Pin_61)
- net FPGA_1_USER_IO31: now also J?.71 (Pin_71); no longer J?.63 (Pin_63)
- net FPGA_1_USER_IO32: now also J?.73 (Pin_73); no longer J?.65 (Pin_65)
- net FPGA_1_USER_IO33: now also J?.75 (Pin_75); no longer J?.67 (Pin_67)
- net FPGA_1_USER_IO34: now also J?.77 (Pin_77); no longer J?.69 (Pin_69)
- net FPGA_1_USER_IO35: now also J?.79 (Pin_79); no longer J?.71 (Pin_71)
- net FPGA_1_USER_IO36: now also J?.9 (Pin_9); no longer J?.73 (Pin_73)
- net FPGA_1_USER_IO37: now also J?.11 (Pin_11); no longer J?.75 (Pin_75)
- net FPGA_1_USER_IO38: now also J?.13 (Pin_13); no longer J?.77 (Pin_77)
- net FPGA_1_USER_IO39: now also J?.15 (Pin_15); no longer J?.79 (Pin_79)
- net FPGA_1_USER_IO4: now also J?.17 (Pin_17); no longer J?.9 (Pin_9)
- net FPGA_1_USER_IO40: now also J?.17 (Pin_17); no longer J?.1 (Pin_1)
- net FPGA_1_USER_IO41: now also J?.19 (Pin_19); no longer J?.3 (Pin_3)
- net FPGA_1_USER_IO42: no longer J?.5 (Pin_5)
- net FPGA_1_USER_IO43: no longer J?.7 (Pin_7)
- net FPGA_1_USER_IO44: no longer J?.9 (Pin_9)
- net FPGA_1_USER_IO45: no longer J?.11 (Pin_11)
- net FPGA_1_USER_IO46: no longer J?.13 (Pin_13)
- net FPGA_1_USER_IO47: no longer J?.15 (Pin_15)
- net FPGA_1_USER_IO48: no longer J?.17 (Pin_17)
- net FPGA_1_USER_IO49: no longer J?.19 (Pin_19)
- net FPGA_1_USER_IO5: now also J?.19 (Pin_19); no longer J?.11 (Pin_11)
- net FPGA_1_USER_IO6: now also J?.21 (Pin_21); no longer J?.13 (Pin_13)
- net FPGA_1_USER_IO7: now also J?.23 (Pin_23); no longer J?.15 (Pin_15)
- net FPGA_1_USER_IO8: now also J?.25 (Pin_25); no longer J?.17 (Pin_17)
- net FPGA_1_USER_IO9: now also J?.27 (Pin_27); no longer J?.19 (Pin_19)
- net GND: now also J?.65 (Pin_65), J?.67 (Pin_67), J?.69 (Pin_69), J?.71 (Pin_71), J?.73 (Pin_73), J?.75 (Pin_75), J?.77 (Pin_77), J?.79 (Pin_79), C?.2, C?.2, C?.2, C?.2, C?.2, C?.2, C?.2, C?.2, J?.3 (Pin_3), J?.3 (Pin_3), J?.3 (Pin_3), J?.3 (Pin_3), J?.3 (Pin_3), J?.3 (Pin_3), J?.3 (Pin_3), J?.4 (Pin_4), J?.4 (Pin_4), J?.4 (Pin_4), J?.4 (Pin_4), J?.4 (Pin_4), J?.4 (Pin_4), J?.4 (Pin_4), Q?.2 (S), Q?.2 (S), Q?.2 (S), Q?.2 (S), Q?.2 (S), Q?.2 (S), Q?.2 (S), Q?.2 (S), R?.2, R?.2, R?.2, R?.2, R?.2, R?.2, R?.2, R?.2, SW?.1, SW?.1, SW?.1, SW?.1, SW?.1, SW?.1, SW?.1, SW?.1
- new net: D?.1 (K), Q?.3 (D) (x8)
- new net: D?.2 (A), R?.2 (x8)
- new net FPGA_0_CLK1_N: C?.2, C?.2, J?.1
- new net FPGA_0_CLK1_P: C?.1, R?.2
- new net FPGA_0_PMOD_1_IO0: J?.12 (Pin_12)
- new net FPGA_0_PMOD_1_IO1: J?.10 (Pin_10)
- new net FPGA_0_PMOD_1_IO2: J?.8 (Pin_8)
- new net FPGA_0_PMOD_1_IO3: J?.6 (Pin_6)
- new net FPGA_0_PMOD_1_IO4: J?.11 (Pin_11)
- new net FPGA_0_PMOD_1_IO5: J?.9 (Pin_9)
- new net FPGA_0_PMOD_1_IO6: J?.7 (Pin_7)
- new net FPGA_0_PMOD_1_IO7: J?.5 (Pin_5)
- new net FPGA_0_PMOD_2_IO0: J?.12 (Pin_12)
- new net FPGA_0_PMOD_2_IO1: J?.10 (Pin_10)
- new net FPGA_0_PMOD_2_IO2: J?.8 (Pin_8)
- new net FPGA_0_PMOD_2_IO3: J?.6 (Pin_6)
- new net FPGA_0_PMOD_2_IO4: J?.11 (Pin_11)
- new net FPGA_0_PMOD_2_IO5: J?.9 (Pin_9)
- new net FPGA_0_PMOD_2_IO6: J?.7 (Pin_7)
- new net FPGA_0_PMOD_2_IO7: J?.5 (Pin_5)
- new net FPGA_0_PMOD_3_IO0: J?.12 (Pin_12)
- new net FPGA_0_PMOD_3_IO1: J?.10 (Pin_10)
- new net FPGA_0_PMOD_3_IO2: J?.8 (Pin_8)
- new net FPGA_0_PMOD_3_IO3: J?.6 (Pin_6)
- new net FPGA_0_PMOD_3_IO4: J?.11 (Pin_11)
- new net FPGA_0_PMOD_3_IO5: J?.9 (Pin_9)
- new net FPGA_0_PMOD_3_IO6: J?.7 (Pin_7)
- new net FPGA_0_PMOD_3_IO7: J?.5 (Pin_5)
- new net FPGA_0_PMOD_4_IO0: J?.12 (Pin_12)
- new net FPGA_0_PMOD_4_IO1: J?.10 (Pin_10)
- new net FPGA_0_PMOD_4_IO2: J?.8 (Pin_8)
- new net FPGA_0_PMOD_4_IO3: J?.6 (Pin_6)
- new net FPGA_0_PMOD_4_IO4: J?.11 (Pin_11)
- new net FPGA_0_PMOD_4_IO5: J?.9 (Pin_9)
- new net FPGA_0_PMOD_4_IO6: J?.7 (Pin_7)
- new net FPGA_0_PMOD_4_IO7: J?.5 (Pin_5)
- new net FPGA_0_RC_CLK1_P: C?.1, J?.2, R?.1
- new net FPGA_0_RC_RX0_P: C?.1, J?.2, R?.1
- new net FPGA_0_RC_RX1_P: C?.1, J?.2, R?.1
- new net FPGA_0_RC_RX2_P: C?.1, J?.2, R?.1
- new net FPGA_0_RC_RX3_P: C?.1, J?.2, R?.1
- new net FPGA_0_RC_TX0_P: C?.1, J?.2, R?.1
- new net FPGA_0_RC_TX1_P: C?.1, J?.2, R?.1
- new net FPGA_0_RC_TX2_P: C?.1, J?.2, R?.1
- new net FPGA_0_RC_TX3_P: C?.1, J?.2, R?.1
- new net FPGA_0_RX0_N: C?.2, C?.2, J?.1
- new net FPGA_0_RX0_P: C?.1, R?.2
- new net FPGA_0_RX1_N: C?.2, C?.2, J?.1
- new net FPGA_0_RX1_P: C?.1, R?.2
- new net FPGA_0_RX2_N: C?.2, C?.2, J?.1
- new net FPGA_0_RX2_P: C?.1, R?.2
- new net FPGA_0_RX3_N: C?.2, C?.2, J?.1
- new net FPGA_0_RX3_P: C?.1, R?.2
- new net FPGA_0_TX0_N: C?.2, C?.2, J?.1
- new net FPGA_0_TX0_P: C?.1, R?.2
- new net FPGA_0_TX1_N: C?.2, C?.2, J?.1
- new net FPGA_0_TX1_P: C?.1, R?.2
- new net FPGA_0_TX2_N: C?.2, C?.2, J?.1
- new net FPGA_0_TX2_P: C?.1, R?.2
- new net FPGA_0_TX3_N: C?.2, C?.2, J?.1
- new net FPGA_0_TX3_P: C?.1, R?.2
- new net FPGA_1_PMOD_1_IO0: J?.12 (Pin_12)
- new net FPGA_1_PMOD_1_IO1: J?.10 (Pin_10)
- new net FPGA_1_PMOD_1_IO2: J?.8 (Pin_8)
- new net FPGA_1_PMOD_1_IO3: J?.6 (Pin_6)
- new net FPGA_1_PMOD_1_IO4: J?.11 (Pin_11)
- new net FPGA_1_PMOD_1_IO5: J?.9 (Pin_9)
- new net FPGA_1_PMOD_1_IO6: J?.7 (Pin_7)
- new net FPGA_1_PMOD_1_IO7: J?.5 (Pin_5)
- new net FPGA_1_PMOD_2_IO0: J?.12 (Pin_12)
- new net FPGA_1_PMOD_2_IO1: J?.10 (Pin_10)
- new net FPGA_1_PMOD_2_IO2: J?.8 (Pin_8)
- new net FPGA_1_PMOD_2_IO3: J?.6 (Pin_6)
- new net FPGA_1_PMOD_2_IO4: J?.11 (Pin_11)
- new net FPGA_1_PMOD_2_IO5: J?.9 (Pin_9)
- new net FPGA_1_PMOD_2_IO6: J?.7 (Pin_7)
- new net FPGA_1_PMOD_2_IO7: J?.5 (Pin_5)
- new net FPGA_1_PMOD_3_IO0: J?.12 (Pin_12)
- new net FPGA_1_PMOD_3_IO1: J?.10 (Pin_10)
- new net FPGA_1_PMOD_3_IO2: J?.8 (Pin_8)
- new net FPGA_1_PMOD_3_IO3: J?.6 (Pin_6)
- new net FPGA_1_PMOD_3_IO4: J?.11 (Pin_11)
- new net FPGA_1_PMOD_3_IO5: J?.9 (Pin_9)
- new net FPGA_1_PMOD_3_IO6: J?.7 (Pin_7)
- new net FPGA_1_PMOD_3_IO7: J?.5 (Pin_5)
- new net FPGA_1_PMOD_4_IO0: J?.12 (Pin_12)
- new net FPGA_1_PMOD_4_IO1: J?.10 (Pin_10)
- new net FPGA_1_PMOD_4_IO2: J?.8 (Pin_8)
- new net FPGA_1_PMOD_4_IO3: J?.6 (Pin_6)
- new net FPGA_1_PMOD_4_IO4: J?.11 (Pin_11)
- new net FPGA_1_PMOD_4_IO5: J?.9 (Pin_9)
- new net FPGA_1_PMOD_4_IO6: J?.7 (Pin_7)
- new net FPGA_1_PMOD_4_IO7: J?.5 (Pin_5)
- new net FPGA_SW0: R?.2
- new net FPGA_SW0_R: C?.1, R?.1, R?.2, SW?.2
- new net FPGA_SW1: R?.2
- new net FPGA_SW1_R: C?.1, R?.1, R?.2, SW?.2
- new net FPGA_SW2: R?.2
- new net FPGA_SW2_R: C?.1, R?.1, R?.2, SW?.2
- new net FPGA_SW3: R?.2
- new net FPGA_SW3_R: C?.1, R?.1, R?.2, SW?.2
- new net FPGA_SW4: R?.2
- new net FPGA_SW4_R: C?.1, R?.1, R?.2, SW?.2
- new net FPGA_SW5: R?.2
- new net FPGA_SW5_R: C?.1, R?.1, R?.2, SW?.2
- new net FPGA_SW6: R?.2
- new net FPGA_SW6_R: C?.1, R?.1, R?.2, SW?.2
- new net FPGA_SW7: R?.2
- new net FPGA_SW7_R: C?.1, R?.1, R?.2, SW?.2
- new net LED0: Q?.1 (G), R?.1
- new net LED1: Q?.1 (G), R?.1
- new net LED2: Q?.1 (G), R?.1
- new net LED3: Q?.1 (G), R?.1
- new net LED4: Q?.1 (G), R?.1
- new net LED5: Q?.1 (G), R?.1
- new net LED6: Q?.1 (G), R?.1
- new net LED7: Q?.1 (G), R?.1
Other:
- moved on the sheet: C?, F?, J?, R?

Commit message: Added PSRAM, Finished Schematic
Footprint assignment required, some minor changes to be made to schematic. Sheet naming and commenting to be done.
Parts:
- removed J? (x4): Conn_02x06_Odd_Even, symbol Connector_Generic:Conn_02x06_Odd_Even
- added C? (x8): 100nF, Capacitor_SMD:C_0402_1005Metric, symbol Device:C
- added D? (x8): LED GREEN, LED_SMD:LED_0603_1608Metric, symbol Device:LED
- added J? (x4): Conn_02x06_Odd_Even, symbol Connector_Generic:Conn_02x06_Odd_Even
- added Q? (x8): 2N7002, digikey-footprints:SOT-23-3, symbol dk_Transistors-FETs-MOSFETs-Single:2N7002
- added R? (x24): 3K3, Resistor_SMD:R_0402_1005Metric, symbol Device:R_US
- added R? (x8): 100K, Resistor_SMD:R_0402_1005Metric, symbol Device:R_US
- added SW? (x8): SW_Push, symbol Switch:SW_Push
Connections:
- net +3V3: now also J?.1 (Pin_1), J?.1 (Pin_1), J?.1 (Pin_1), J?.1 (Pin_1), J?.2 (Pin_2), J?.2 (Pin_2), J?.2 (Pin_2), J?.2 (Pin_2), R?.1, R?.1, R?.1, R?.1, R?.1, R?.1, R?.1, R?.1, R?.1, R?.1, R?.1, R?.1, R?.1, R?.1, R?.1, R?.1
- net GND: now also C?.2, C?.2, C?.2, C?.2, C?.2, C?.2, C?.2, C?.2, J?.3 (Pin_3), J?.3 (Pin_3), J?.3 (Pin_3), J?.3 (Pin_3), J?.4 (Pin_4), J?.4 (Pin_4), J?.4 (Pin_4), J?.4 (Pin_4), Q?.2 (S), Q?.2 (S), Q?.2 (S), Q?.2 (S), Q?.2 (S), Q?.2 (S), Q?.2 (S), Q?.2 (S), R?.2, R?.2, R?.2, R?.2, R?.2, R?.2, R?.2, R?.2, SW?.1, SW?.1, SW?.1, SW?.1, SW?.1, SW?.1, SW?.1, SW?.1
- net FPGA_0_PMOD_1_IO0 renamed FPGA_0_PMOD0_IO0
- net FPGA_0_PMOD_1_IO1 renamed FPGA_0_PMOD0_IO1
- net FPGA_0_PMOD_1_IO2 renamed FPGA_0_PMOD0_IO2
- net FPGA_0_PMOD_1_IO3 renamed FPGA_0_PMOD0_IO3
- net FPGA_0_PMOD_1_IO4 renamed FPGA_0_PMOD0_IO4
- net FPGA_0_PMOD_1_IO5 renamed FPGA_0_PMOD0_IO5
- net FPGA_0_PMOD_1_IO6 renamed FPGA_0_PMOD0_IO6
- net FPGA_0_PMOD_1_IO7 renamed FPGA_0_PMOD0_IO7
- net FPGA_0_PMOD_2_IO0 renamed FPGA_0_PMOD1_IO0
- net FPGA_0_PMOD_2_IO1 renamed FPGA_0_PMOD1_IO1
- net FPGA_0_PMOD_2_IO2 renamed FPGA_0_PMOD1_IO2
- net FPGA_0_PMOD_2_IO3 renamed FPGA_0_PMOD1_IO3
- net FPGA_0_PMOD_2_IO4 renamed FPGA_0_PMOD1_IO4
- net FPGA_0_PMOD_2_IO5 renamed FPGA_0_PMOD1_IO5
- net FPGA_0_PMOD_2_IO6 renamed FPGA_0_PMOD1_IO6
- net FPGA_0_PMOD_2_IO7 renamed FPGA_0_PMOD1_IO7
- net FPGA_0_PMOD_3_IO0 renamed FPGA_0_PMOD2_IO0
- net FPGA_0_PMOD_3_IO1 renamed FPGA_0_PMOD2_IO1
- net FPGA_0_PMOD_3_IO2 renamed FPGA_0_PMOD2_IO2
- net FPGA_0_PMOD_3_IO3 renamed FPGA_0_PMOD2_IO3
- net FPGA_0_PMOD_3_IO4 renamed FPGA_0_PMOD2_IO4
- net FPGA_0_PMOD_3_IO5 renamed FPGA_0_PMOD2_IO5
- net FPGA_0_PMOD_3_IO6 renamed FPGA_0_PMOD2_IO6
- net FPGA_0_PMOD_3_IO7 renamed FPGA_0_PMOD2_IO7
- net FPGA_0_PMOD_4_IO0 renamed FPGA_0_PMOD3_IO0
- net FPGA_0_PMOD_4_IO1 renamed FPGA_0_PMOD3_IO1
- net FPGA_0_PMOD_4_IO2 renamed FPGA_0_PMOD3_IO2
- net FPGA_0_PMOD_4_IO3 renamed FPGA_0_PMOD3_IO3
- net FPGA_0_PMOD_4_IO4 renamed FPGA_0_PMOD3_IO4
- net FPGA_0_PMOD_4_IO5 renamed FPGA_0_PMOD3_IO5
- net FPGA_0_PMOD_4_IO6 renamed FPGA_0_PMOD3_IO6
- net FPGA_0_PMOD_4_IO7 renamed FPGA_0_PMOD3_IO7
- net FPGA_SW0 renamed FPGA_1_SW0
- net FPGA_SW0_R renamed FPGA_1_SW0_R
- net FPGA_SW1 renamed FPGA_1_SW1
- net FPGA_SW1_R renamed FPGA_1_SW1_R
- net FPGA_SW2 renamed FPGA_1_SW2
- net FPGA_SW2_R renamed FPGA_1_SW2_R
- net FPGA_SW3 renamed FPGA_1_SW3
- net FPGA_SW3_R renamed FPGA_1_SW3_R
- net FPGA_SW4 renamed FPGA_1_SW4
- net FPGA_SW4_R renamed FPGA_1_SW4_R
- net FPGA_SW5 renamed FPGA_1_SW5
- net FPGA_SW5_R renamed FPGA_1_SW5_R
- net FPGA_SW6 renamed FPGA_1_SW6
- net FPGA_SW6_R renamed FPGA_1_SW6_R
- net FPGA_SW7 renamed FPGA_1_SW7
- net FPGA_SW7_R renamed FPGA_1_SW7_R
- net LED0 renamed FPGA_1_LED0
- net LED1 renamed FPGA_1_LED1
- net LED2 renamed FPGA_1_LED2
- net LED3 renamed FPGA_1_LED3
- net LED4 renamed FPGA_1_LED4
- net LED5 renamed FPGA_1_LED5
- net LED6 renamed FPGA_1_LED6
- net LED7 renamed FPGA_1_LED7
- new net: D?.1 (K), Q?.3 (D) (x8)
- new net: D?.2 (A), R?.2 (x8)
- new net FPGA_0_LED0: Q?.1 (G), R?.1
- new net FPGA_0_LED1: Q?.1 (G), R?.1
- new net FPGA_0_LED2: Q?.1 (G), R?.1
- new net FPGA_0_LED3: Q?.1 (G), R?.1
- new net FPGA_0_LED4: Q?.1 (G), R?.1
- new net FPGA_0_LED5: Q?.1 (G), R?.1
- new net FPGA_0_LED6: Q?.1 (G), R?.1
- new net FPGA_0_LED7: Q?.1 (G), R?.1
- new net FPGA_0_SW0: R?.2
- new net FPGA_0_SW0_R: C?.1, R?.1, R?.2, SW?.2
- new net FPGA_0_SW1: R?.2
- new net FPGA_0_SW1_R: C?.1, R?.1, R?.2, SW?.2
- new net FPGA_0_SW2: R?.2
- new net FPGA_0_SW2_R: C?.1, R?.1, R?.2, SW?.2
- new net FPGA_0_SW3: R?.2
- new net FPGA_0_SW3_R: C?.1, R?.1, R?.2, SW?.2
- new net FPGA_0_SW4: R?.2
- new net FPGA_0_SW4_R: C?.1, R?.1, R?.2, SW?.2
- new net FPGA_0_SW5: R?.2
- new net FPGA_0_SW5_R: C?.1, R?.1, R?.2, SW?.2
- new net FPGA_0_SW6: R?.2
- new net FPGA_0_SW6_R: C?.1, R?.1, R?.2, SW?.2
- new net FPGA_0_SW7: R?.2
- new net FPGA_0_SW7_R: C?.1, R?.1, R?.2, SW?.2
- new net FPGA_1_PMOD0_IO0: J?.12 (Pin_12)
- new net FPGA_1_PMOD0_IO1: J?.10 (Pin_10)
- new net FPGA_1_PMOD0_IO2: J?.8 (Pin_8)
- new net FPGA_1_PMOD0_IO3: J?.6 (Pin_6)
- new net FPGA_1_PMOD0_IO4: J?.11 (Pin_11)
- new net FPGA_1_PMOD0_IO5: J?.9 (Pin_9)
- new net FPGA_1_PMOD0_IO6: J?.7 (Pin_7)
- new net FPGA_1_PMOD0_IO7: J?.5 (Pin_5)
- new net FPGA_1_PMOD1_IO0: J?.12 (Pin_12)
- new net FPGA_1_PMOD1_IO1: J?.10 (Pin_10)
- new net FPGA_1_PMOD1_IO2: J?.8 (Pin_8)
- new net FPGA_1_PMOD1_IO3: J?.6 (Pin_6)
- new net FPGA_1_PMOD1_IO4: J?.11 (Pin_11)
- new net FPGA_1_PMOD1_IO5: J?.9 (Pin_9)
- new net FPGA_1_PMOD1_IO6: J?.7 (Pin_7)
- new net FPGA_1_PMOD1_IO7: J?.5 (Pin_5)
- new net FPGA_1_PMOD2_IO0: J?.12 (Pin_12)
- new net FPGA_1_PMOD2_IO1: J?.10 (Pin_10)
- new net FPGA_1_PMOD2_IO2: J?.8 (Pin_8)
- new net FPGA_1_PMOD2_IO3: J?.6 (Pin_6)
- new net FPGA_1_PMOD2_IO4: J?.11 (Pin_11)
- new net FPGA_1_PMOD2_IO5: J?.9 (Pin_9)
- new net FPGA_1_PMOD2_IO6: J?.7 (Pin_7)
- new net FPGA_1_PMOD2_IO7: J?.5 (Pin_5)
- new net FPGA_1_PMOD3_IO0: J?.12 (Pin_12)
- new net FPGA_1_PMOD3_IO1: J?.10 (Pin_10)
- new net FPGA_1_PMOD3_IO2: J?.8 (Pin_8)
- new net FPGA_1_PMOD3_IO3: J?.6 (Pin_6)
- new net FPGA_1_PMOD3_IO4: J?.11 (Pin_11)
- new net FPGA_1_PMOD3_IO5: J?.9 (Pin_9)
- new net FPGA_1_PMOD3_IO6: J?.7 (Pin_7)
- new net FPGA_1_PMOD3_IO7: J?.5 (Pin_5)
Other:
- moved on the sheet: C?, D?, Q?, R?, SW?

Commit message: Added Footprints
Parts:
- removed J? (x7): Conn_02x06_Odd_Even, symbol Connector_Generic:Conn_02x06_Odd_Even
- removed J? (x2): Conn_02x40_Odd_Even, symbol Connector_Generic:Conn_02x40_Odd_Even
- removed SW? (x15): SW_Push, symbol Switch:SW_Push
- added J? (x6): Conn_02x06_Odd_Even, Connector_PinHeader_2.54mm:PinHeader_2x06_P2.54mm_Horizontal, symbol Connector_Generic:Conn_02x06_Odd_Even
- added J? (x2): Conn_02x40_Odd_Even, Connector_PinHeader_2.54mm:PinHeader_2x40_P2.54mm_Vertical_SMD, symbol Connector_Generic:Conn_02x40_Odd_Even
- added SW? (x15): SW_Push, Button_Switch_SMD:SW_SPST_EVQQ2, symbol Switch:SW_Push
- F? (x2): footprint (none) -> Fuse:Fuse_0603_1608Metric
- J?: footprint (none) -> Connector_PinHeader_2.54mm:PinHeader_2x40_P2.54mm_Vertical_SMD
- J?: footprint (none) -> Connector_PinHeader_2.54mm:PinHeader_2x06_P2.54mm_Horizontal
- SW?: footprint (none) -> Button_Switch_SMD:SW_SPST_EVQQ2
Connections:
- net +3V3: now also J?.1 (Pin_1), J?.1 (Pin_1), J?.1 (Pin_1), J?.1 (Pin_1), J?.1 (Pin_1), J?.1 (Pin_1), J?.1 (Pin_1), J?.1 (Pin_1), J?.2 (Pin_2), J?.2 (Pin_2), J?.2 (Pin_2), J?.2 (Pin_2), J?.2 (Pin_2), J?.2 (Pin_2), J?.2 (Pin_2), J?.2 (Pin_2), J?.3 (Pin_3), J?.3 (Pin_3), J?.4 (Pin_4), J?.4 (Pin_4)
- net +5V: now also J?.5 (Pin_5), J?.5 (Pin_5), J?.6 (Pin_6), J?.6 (Pin_6), J?.7 (Pin_7), J?.7 (Pin_7), J?.8 (Pin_8), J?.8 (Pin_8)
- net FPGA_0_PMOD0_IO0: now also J?.12 (Pin_12)
- net FPGA_0_PMOD0_IO1: now also J?.10 (Pin_10)
- net FPGA_0_PMOD0_IO2: now also J?.8 (Pin_8)
- net FPGA_0_PMOD0_IO3: now also J?.6 (Pin_6)
- net FPGA_0_PMOD0_IO4: now also J?.11 (Pin_11)
- net FPGA_0_PMOD0_IO5: now also J?.9 (Pin_9)
- net FPGA_0_PMOD0_IO6: now also J?.7 (Pin_7)
- net FPGA_0_PMOD0_IO7: now also J?.5 (Pin_5)
- net FPGA_0_PMOD1_IO0: now also J?.12 (Pin_12)
- net FPGA_0_PMOD1_IO1: now also J?.10 (Pin_10)
- net FPGA_0_PMOD1_IO2: now also J?.8 (Pin_8)
- net FPGA_0_PMOD1_IO3: now also J?.6 (Pin_6)
- net FPGA_0_PMOD1_IO4: now also J?.11 (Pin_11)
- net FPGA_0_PMOD1_IO5: now also J?.9 (Pin_9)
- net FPGA_0_PMOD1_IO6: now also J?.7 (Pin_7)
- net FPGA_0_PMOD1_IO7: now also J?.5 (Pin_5)
- net FPGA_0_PMOD3_IO0: now also J?.12 (Pin_12)
- net FPGA_0_PMOD3_IO1: now also J?.10 (Pin_10)
- net FPGA_0_PMOD3_IO2: now also J?.8 (Pin_8)
- net FPGA_0_PMOD3_IO3: now also J?.6 (Pin_6)
- net FPGA_0_PMOD3_IO4: now also J?.11 (Pin_11)
- net FPGA_0_PMOD3_IO5: now also J?.9 (Pin_9)
- net FPGA_0_PMOD3_IO6: now also J?.7 (Pin_7)
- net FPGA_0_PMOD3_IO7: now also J?.5 (Pin_5)
- net FPGA_0_SW0_R: now also SW?.2
- net FPGA_0_SW1_R: now also SW?.2
- net FPGA_0_SW2_R: now also SW?.2
- net FPGA_0_SW3_R: now also SW?.2
- net FPGA_0_SW4_R: now also SW?.2
- net FPGA_0_SW5_R: now also SW?.2
- net FPGA_0_SW6_R: now also SW?.2
- net FPGA_0_SW7_R: now also SW?.2
- net FPGA_0_USER_IO0: now also J?.37 (Pin_37)
- net FPGA_0_USER_IO1: now also J?.39 (Pin_39)
- net FPGA_0_USER_IO10: now also J?.57 (Pin_57)
- net FPGA_0_USER_IO11: now also J?.59 (Pin_59)
- net FPGA_0_USER_IO12: now also J?.61 (Pin_61)
- net FPGA_0_USER_IO13: now also J?.63 (Pin_63)
- net FPGA_0_USER_IO14: now also J?.65 (Pin_65)
- net FPGA_0_USER_IO15: now also J?.67 (Pin_67)
- net FPGA_0_USER_IO16: now also J?.69 (Pin_69)
- net FPGA_0_USER_IO17: now also J?.71 (Pin_71)
- net FPGA_0_USER_IO18: now also J?.73 (Pin_73)
- net FPGA_0_USER_IO19: now also J?.75 (Pin_75)
- net FPGA_0_USER_IO2: now also J?.41 (Pin_41)
- net FPGA_0_USER_IO20: now also J?.77 (Pin_77)
- net FPGA_0_USER_IO21: now also J?.79 (Pin_79)
- net FPGA_0_USER_IO22: now also J?.9 (Pin_9)
- net FPGA_0_USER_IO23: now also J?.11 (Pin_11)
- net FPGA_0_USER_IO24: now also J?.13 (Pin_13)
- net FPGA_0_USER_IO25: now also J?.15 (Pin_15)
- net FPGA_0_USER_IO26: now also J?.17 (Pin_17)
- net FPGA_0_USER_IO27: now also J?.19 (Pin_19)
- net FPGA_0_USER_IO28: now also J?.21 (Pin_21)
- net FPGA_0_USER_IO29: now also J?.23 (Pin_23)
- net FPGA_0_USER_IO3: now also J?.43 (Pin_43)
- net FPGA_0_USER_IO30: now also J?.25 (Pin_25)
- net FPGA_0_USER_IO31: now also J?.27 (Pin_27)
- net FPGA_0_USER_IO32: now also J?.29 (Pin_29)
- net FPGA_0_USER_IO33: now also J?.31 (Pin_31)
- net FPGA_0_USER_IO34: now also J?.33 (Pin_33)
- net FPGA_0_USER_IO35: now also J?.35 (Pin_35)
- net FPGA_0_USER_IO36: now also J?.37 (Pin_37)
- net FPGA_0_USER_IO37: now also J?.39 (Pin_39)
- net FPGA_0_USER_IO38: now also J?.41 (Pin_41)
- net FPGA_0_USER_IO39: now also J?.43 (Pin_43)
- net FPGA_0_USER_IO4: now also J?.45 (Pin_45)
- net FPGA_0_USER_IO40: now also J?.45 (Pin_45)
- net FPGA_0_USER_IO41: now also J?.47 (Pin_47)
- net FPGA_0_USER_IO42: now also J?.49 (Pin_49)
- net FPGA_0_USER_IO43: now also J?.51 (Pin_51)
- net FPGA_0_USER_IO44: now also J?.53 (Pin_53)
- net FPGA_0_USER_IO45: now also J?.55 (Pin_55)
- net FPGA_0_USER_IO46: now also J?.57 (Pin_57)
- net FPGA_0_USER_IO47: now also J?.59 (Pin_59)
- net FPGA_0_USER_IO48: now also J?.61 (Pin_61)
- net FPGA_0_USER_IO49: now also J?.63 (Pin_63)
- net FPGA_0_USER_IO5: now also J?.47 (Pin_47)
- net FPGA_0_USER_IO6: now also J?.49 (Pin_49)
- net FPGA_0_USER_IO7: now also J?.51 (Pin_51)
- net FPGA_0_USER_IO8: now also J?.53 (Pin_53)
- net FPGA_0_USER_IO9: now also J?.55 (Pin_55)
- net FPGA_1_PMOD1_IO0: now also J?.12 (Pin_12)
- net FPGA_1_PMOD1_IO1: now also J?.10 (Pin_10)
- net FPGA_1_PMOD1_IO2: now also J?.8 (Pin_8)
- net FPGA_1_PMOD1_IO3: now also J?.6 (Pin_6)
- net FPGA_1_PMOD1_IO4: now also J?.11 (Pin_11)
- net FPGA_1_PMOD1_IO5: now also J?.9 (Pin_9)
- net FPGA_1_PMOD1_IO6: now also J?.7 (Pin_7)
- net FPGA_1_PMOD1_IO7: now also J?.5 (Pin_5)
- net FPGA_1_PMOD2_IO0: now also J?.12 (Pin_12)
- net FPGA_1_PMOD2_IO1: now also J?.10 (Pin_10)
- net FPGA_1_PMOD2_IO2: now also J?.8 (Pin_8)
- net FPGA_1_PMOD2_IO3: now also J?.6 (Pin_6)
- net FPGA_1_PMOD2_IO4: now also J?.11 (Pin_11)
- net FPGA_1_PMOD2_IO5: now also J?.9 (Pin_9)
- net FPGA_1_PMOD2_IO6: now also J?.7 (Pin_7)
- net FPGA_1_PMOD2_IO7: now also J?.5 (Pin_5)
- net FPGA_1_PMOD3_IO0: now also J?.12 (Pin_12)
- net FPGA_1_PMOD3_IO1: now also J?.10 (Pin_10)
- net FPGA_1_PMOD3_IO2: now also J?.8 (Pin_8)
- net FPGA_1_PMOD3_IO3: now also J?.6 (Pin_6)
- net FPGA_1_PMOD3_IO4: now also J?.11 (Pin_11)
- net FPGA_1_PMOD3_IO5: now also J?.9 (Pin_9)
- net FPGA_1_PMOD3_IO6: now also J?.7 (Pin_7)
- net FPGA_1_PMOD3_IO7: now also J?.5 (Pin_5)
- net FPGA_1_SW1_R: now also SW?.2
- net FPGA_1_SW2_R: now also SW?.2
- net FPGA_1_SW3_R: now also SW?.2
- net FPGA_1_SW4_R: now also SW?.2
- net FPGA_1_SW5_R: now also SW?.2
- net FPGA_1_SW6_R: now also SW?.2
- net FPGA_1_SW7_R: now also SW?.2
- net FPGA_1_USER_IO36: now also J?.9 (Pin_9)
- net FPGA_1_USER_IO37: now also J?.11 (Pin_11)
- net FPGA_1_USER_IO38: now also J?.13 (Pin_13)
- net FPGA_1_USER_IO39: now also J?.15 (Pin_15)
- net FPGA_1_USER_IO40: now also J?.17 (Pin_17)
- net FPGA_1_USER_IO41: now also J?.19 (Pin_19)
- net FPGA_1_USER_IO42: now also J?.21 (Pin_21)
- net FPGA_1_USER_IO43: now also J?.23 (Pin_23)
- net FPGA_1_USER_IO44: now also J?.25 (Pin_25)
- net FPGA_1_USER_IO45: now also J?.27 (Pin_27)
- net FPGA_1_USER_IO46: now also J?.29 (Pin_29)
- net FPGA_1_USER_IO47: now also J?.31 (Pin_31)
- net FPGA_1_USER_IO48: now also J?.33 (Pin_33)
- net FPGA_1_USER_IO49: now also J?.35 (Pin_35)
- net GND: now also J?.10 (Pin_10), J?.10 (Pin_10), J?.12 (Pin_12), J?.12 (Pin_12), J?.14 (Pin_14), J?.14 (Pin_14), J?.16 (Pin_16), J?.16 (Pin_16), J?.18 (Pin_18), J?.18 (Pin_18), J?.20 (Pin_20), J?.20 (Pin_20), J?.22 (Pin_22), J?.22 (Pin_22), J?.24 (Pin_24), J?.24 (Pin_24), J?.26 (Pin_26), J?.26 (Pin_26), J?.28 (Pin_28), J?.28 (Pin_28), J?.3 (Pin_3), J?.3 (Pin_3), J?.3 (Pin_3), J?.3 (Pin_3), J?.3 (Pin_3), J?.3 (Pin_3), J?.30 (Pin_30), J?.30 (Pin_30), J?.32 (Pin_32), J?.32 (Pin_32), J?.34 (Pin_34), J?.34 (Pin_34), J?.36 (Pin_36), J?.36 (Pin_36), J?.38 (Pin_38), J?.38 (Pin_38), J?.4 (Pin_4), J?.4 (Pin_4), J?.4 (Pin_4), J?.4 (Pin_4), J?.4 (Pin_4), J?.4 (Pin_4), J?.40 (Pin_40), J?.40 (Pin_40), J?.42 (Pin_42), J?.42 (Pin_42), J?.44 (Pin_44), J?.44 (Pin_44), J?.46 (Pin_46), J?.46 (Pin_46), J?.48 (Pin_48), J?.48 (Pin_48), J?.50 (Pin_50), J?.50 (Pin_50), J?.52 (Pin_52), J?.52 (Pin_52), J?.54 (Pin_54), J?.54 (Pin_54), J?.56 (Pin_56), J?.56 (Pin_56), J?.58 (Pin_58), J?.58 (Pin_58), J?.60 (Pin_60), J?.60 (Pin_60), J?.62 (Pin_62), J?.62 (Pin_62), J?.64 (Pin_64), J?.64 (Pin_64), J?.65 (Pin_65), J?.66 (Pin_66), J?.66 (Pin_66), J?.67 (Pin_67), J?.68 (Pin_68), J?.68 (Pin_68), J?.69 (Pin_69), J?.70 (Pin_70), J?.70 (Pin_70), J?.71 (Pin_71), J?.72 (Pin_72), J?.72 (Pin_72), J?.73 (Pin_73), J?.74 (Pin_74), J?.74 (Pin_74), J?.75 (Pin_75), J?.76 (Pin_76), J?.76 (Pin_76), J?.77 (Pin_77), J?.78 (Pin_78), J?.78 (Pin_78), J?.79 (Pin_79), J?.80 (Pin_80), J?.80 (Pin_80), SW?.1, SW?.1, SW?.1, SW?.1, SW?.1, SW?.1, SW?.1, SW?.1, SW?.1, SW?.1, SW?.1, SW?.1, SW?.1, SW?.1, SW?.1
Other:
- note added: "High Density 3V3 User IO"
- note added: "USER BUTTONS"
- note added: "USER DISPLAYPORT (ONLY ON FPGA_1)"
- note added: "USER GTP (ONLY ON FPGA_0)"
- note added: "USER LED's"
- note added: "USER PMOD"
- title: (none) -> User IO
- moved on the sheet: C?, D?, Q?, R?, SW?

Commit message: Added component ref des
Parts:
- gave numbers to parts that had none: 214

Commit message: Fixed all ERC Errors
Warnings can be ignored
Parts:
- removed C201, C202, C203, C204, C205, C206, C207, C208, C209, C210, C211, C212, C213, C214, C215, C216, C217, C218: DNF, Capacitor_SMD:C_0402_1005Metric, symbol Device:C_Small
- added J33: Conn_02x06_Odd_Even, Connector_PinHeader_2.54mm:PinHeader_2x06_P2.54mm_Horizontal, symbol Connector_Generic:Conn_02x06_Odd_Even
- added R207, R208, R209, R210, R211, R217, R218, R219, R220, R221, R222, R223, R224, R225, R230, R231, R232, R233: DNF, Resistor_SMD:R_0402_1005Metric, symbol Device:R_US
- added R212, R213, R214, R215, R216, R226, R227, R228, R229: 0R, Resistor_SMD:R_0402_1005Metric, symbol Device:R_US
Connections:
- net +3V3: now also J33.1 (Pin_1), J33.2 (Pin_2)
- net FPGA_0_CLK1_N: now also R216.2, R221.1; no longer J15.1
- net FPGA_0_CLK1_P: now also R221.2
- net FPGA_0_PMOD2_IO0: now also J33.12 (Pin_12)
- net FPGA_0_PMOD2_IO1: now also J33.10 (Pin_10)
- net FPGA_0_PMOD2_IO2: now also J33.8 (Pin_8)
- net FPGA_0_PMOD2_IO3: now also J33.6 (Pin_6)
- net FPGA_0_PMOD2_IO4: now also J33.11 (Pin_11)
- net FPGA_0_PMOD2_IO5: now also J33.9 (Pin_9)
- net FPGA_0_PMOD2_IO6: now also J33.7 (Pin_7)
- net FPGA_0_PMOD2_IO7: now also J33.5 (Pin_5)
- net FPGA_0_RC_CLK1_P: now also R211.2
- net FPGA_0_RC_RX0_P: now also R222.2
- net FPGA_0_RC_RX1_P: now also R223.2
- net FPGA_0_RC_RX2_P: now also R224.2
- net FPGA_0_RC_RX3_P: now also R225.2
- net FPGA_0_RC_TX0_P: now also R207.2
- net FPGA_0_RC_TX1_P: now also R208.2
- net FPGA_0_RC_TX2_P: now also R209.2
- net FPGA_0_RC_TX3_P: now also R210.2
- net FPGA_0_RX0_N: now also R226.2, R230.1; no longer J16.1
- net FPGA_0_RX0_P: now also R230.2
- net FPGA_0_RX1_N: now also R227.2, R231.1; no longer J17.1
- net FPGA_0_RX1_P: now also R231.2
- net FPGA_0_RX2_N: now also R228.2, R232.1; no longer J18.1
- net FPGA_0_RX2_P: now also R232.2
- net FPGA_0_RX3_N: now also R229.2, R233.1; no longer J19.1
- net FPGA_0_RX3_P: now also R233.2
- net FPGA_0_TX0_N: now also R212.2, R217.1; no longer J11.1
- net FPGA_0_TX0_P: now also R217.2
- net FPGA_0_TX1_N: now also R213.2, R218.1; no longer J12.1
- net FPGA_0_TX1_P: now also R218.2
- net FPGA_0_TX2_N: now also R214.2, R219.1; no longer J13.1
- net FPGA_0_TX2_P: now also R219.2
- net FPGA_0_TX3_N: now also R215.2, R220.1; no longer J14.1
- net FPGA_0_TX3_P: now also R220.2
- net GND: now also J33.3 (Pin_3), J33.4 (Pin_4)
- new net FPGA_0_RC_CLK1_N: J15.1, R211.1, R216.1
- new net FPGA_0_RC_RX0_N: J16.1, R222.1, R226.1
- new net FPGA_0_RC_RX1_N: J17.1, R223.1, R227.1
- new net FPGA_0_RC_RX2_N: J18.1, R224.1, R228.1
- new net FPGA_0_RC_RX3_N: J19.1, R225.1, R229.1
- new net FPGA_0_RC_TX0_N: J11.1, R207.1, R212.1
- new net FPGA_0_RC_TX1_N: J12.1, R208.1, R213.1
- new net FPGA_0_RC_TX2_N: J13.1, R209.1, R214.1
- new net FPGA_0_RC_TX3_N: J14.1, R210.1, R215.1
