File: DSN/IO.kicad_sch (KiCad schematic)
At the start: 224 parts, among them J10 2040210-1_NonStock, J11 5-1814832-1, J12 5-1814832-1, J13 5-1814832-1, J14 5-1814832-1, J15 5-1814832-1, J16 5-1814832-1, J17 5-1814832-1, J18 5-1814832-1, J19 5-1814832-1, J20 Conn_02x06_Odd_Even, J21 Conn_02x06_Odd_Even, J22 Conn_02x06_Odd_Even, J23 Conn_02x06_Odd_Even, J24 Conn_02x06_Odd_Even, J25 Conn_02x06_Odd_Even, J26 Conn_02x06_Odd_Even, J33 Conn_02x06_Odd_Even, J6 Conn_02x40_Odd_Even, J7 2040210-1_NonStock, J8 Conn_02x40_Odd_Even, J9 Conn_02x40_Odd_Even, Q10 2N7002, Q11 2N7002, Q12 2N7002, Q13 2N7002, Q14 2N7002, Q15 2N7002, Q16 2N7002, Q17 2N7002, Q18 2N7002, Q19 2N7002, Q20 2N7002, Q5 2N7002, Q6 2N7002, Q7 2N7002, Q8 2N7002, Q9 2N7002, SW10 SW_Push, SW11 SW_Push, SW12 SW_Push, SW13 SW_Push, SW14 SW_Push, SW15 SW_Push, SW16 SW_Push, SW17 SW_Push, SW18 SW_Push, SW19 SW_Push, SW20 SW_Push, SW21 SW_Push, SW22 SW_Push, SW23 SW_Push, SW24 SW_Push, SW25 SW_Push

Commit message: Initial PCB Layout
Initial layout and part placement
Parts:
- removed J6, J8, J9: Conn_02x40_Odd_Even, Connector_PinHeader_2.54mm:PinHeader_2x40_P2.54mm_Vertical_SMD, symbol Connector_Generic:Conn_02x40_Odd_Even
- added J6, J8, J9: Conn_02x40_Top_Bottom, Connector_PinSocket_2.54mm:PinSocket_2x40_P2.54mm_Vertical, symbol Connector_Generic:Conn_02x40_Top_Bottom
- J10, J7: value 2040210-1_NonStock -> 47272-0001; footprint digikey-footprints:DisplayPort_2040210-1 -> Lib:MOLEX_47272-0001; DK_Datasheet_Link https://www.te.com/commerce/DocumentDelivery/DDEController?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 -> (none); DK_Detail_Page /product-detail/en/te-connectivity-amp-connectors/2040210-1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 -> (none); Digi-Key_PN A99344-ND -> (none); MFR PN (none) -> 47272-0001; MPN 2040210-1 -> (none); Manufacturer TE Connectivity AMP Connectors -> (none); Status Active NonStock -> (none)
Connections:
- net +3V3: now also J6.1 (Pin_1), J6.2 (Pin_2), J6.41 (Pin_41), J6.42 (Pin_42), J8.1 (Pin_1), J8.2 (Pin_2), J8.41 (Pin_41), J8.42 (Pin_42), J9.1 (Pin_1), J9.2 (Pin_2), J9.41 (Pin_41), J9.42 (Pin_42)
- net +5V: now also J6.3 (Pin_3), J6.4 (Pin_4), J6.43 (Pin_43), J6.44 (Pin_44), J8.3 (Pin_3), J8.4 (Pin_4), J8.43 (Pin_43), J8.44 (Pin_44), J9.3 (Pin_3), J9.4 (Pin_4), J9.43 (Pin_43), J9.44 (Pin_44)
- net FPGA_0_USER_IO0: now also J8.33 (Pin_33)
- net FPGA_0_USER_IO1: now also J8.46 (Pin_46)
- net FPGA_0_USER_IO10: now also J9.7 (Pin_7)
- net FPGA_0_USER_IO11: now also J8.56 (Pin_56)
- net FPGA_0_USER_IO12: now also J9.9 (Pin_9)
- net FPGA_0_USER_IO13: now also J8.58 (Pin_58)
- net FPGA_0_USER_IO14: now also J9.11 (Pin_11)
- net FPGA_0_USER_IO15: now also J8.60 (Pin_60)
- net FPGA_0_USER_IO16: now also J9.13 (Pin_13)
- net FPGA_0_USER_IO17: now also J8.62 (Pin_62)
- net FPGA_0_USER_IO18: now also J9.15 (Pin_15)
- net FPGA_0_USER_IO19: now also J8.64 (Pin_64)
- net FPGA_0_USER_IO2: now also J8.35 (Pin_35)
- net FPGA_0_USER_IO20: now also J9.17 (Pin_17)
- net FPGA_0_USER_IO21: now also J8.66 (Pin_66)
- net FPGA_0_USER_IO22: now also J9.19 (Pin_19)
- net FPGA_0_USER_IO23: now also J8.68 (Pin_68)
- net FPGA_0_USER_IO24: now also J9.21 (Pin_21)
- net FPGA_0_USER_IO25: now also J8.70 (Pin_70)
- net FPGA_0_USER_IO26: now also J9.23 (Pin_23)
- net FPGA_0_USER_IO27: now also J8.72 (Pin_72)
- net FPGA_0_USER_IO28: now also J9.25 (Pin_25)
- net FPGA_0_USER_IO29: now also J8.74 (Pin_74)
- net FPGA_0_USER_IO3: now also J8.48 (Pin_48)
- net FPGA_0_USER_IO30: now also J9.27 (Pin_27)
- net FPGA_0_USER_IO31: now also J8.76 (Pin_76)
- net FPGA_0_USER_IO32: now also J9.29 (Pin_29)
- net FPGA_0_USER_IO33: now also J8.78 (Pin_78)
- net FPGA_0_USER_IO34: now also J9.31 (Pin_31)
- net FPGA_0_USER_IO35: now also J8.80 (Pin_80)
- net FPGA_0_USER_IO36: now also J9.33 (Pin_33)
- net FPGA_0_USER_IO37: now also J9.46 (Pin_46)
- net FPGA_0_USER_IO38: now also J9.35 (Pin_35)
- net FPGA_0_USER_IO39: now also J9.48 (Pin_48)
- net FPGA_0_USER_IO4: now also J8.37 (Pin_37)
- net FPGA_0_USER_IO40: now also J9.37 (Pin_37)
- net FPGA_0_USER_IO41: now also J9.50 (Pin_50)
- net FPGA_0_USER_IO42: now also J9.39 (Pin_39)
- net FPGA_0_USER_IO43: now also J9.52 (Pin_52)
- net FPGA_0_USER_IO44: now also J9.60 (Pin_60)
- net FPGA_0_USER_IO45: now also J9.54 (Pin_54)
- net FPGA_0_USER_IO46: now also J9.62 (Pin_62)
- net FPGA_0_USER_IO47: now also J9.56 (Pin_56)
- net FPGA_0_USER_IO48: now also J9.64 (Pin_64)
- net FPGA_0_USER_IO49: now also J9.58 (Pin_58)
- net FPGA_0_USER_IO5: now also J8.50 (Pin_50)
- net FPGA_0_USER_IO6: now also J8.39 (Pin_39)
- net FPGA_0_USER_IO7: now also J8.52 (Pin_52)
- net FPGA_0_USER_IO8: now also J9.5 (Pin_5)
- net FPGA_0_USER_IO9: now also J8.54 (Pin_54)
- net FPGA_1_USER_IO0: now also J6.5 (Pin_5)
- net FPGA_1_USER_IO1: now also J6.46 (Pin_46)
- net FPGA_1_USER_IO10: now also J6.15 (Pin_15)
- net FPGA_1_USER_IO11: now also J6.56 (Pin_56)
- net FPGA_1_USER_IO12: now also J6.17 (Pin_17)
- net FPGA_1_USER_IO13: now also J6.58 (Pin_58)
- net FPGA_1_USER_IO14: now also J6.19 (Pin_19)
- net FPGA_1_USER_IO15: now also J6.60 (Pin_60)
- net FPGA_1_USER_IO16: now also J6.21 (Pin_21)
- net FPGA_1_USER_IO17: now also J6.62 (Pin_62)
- net FPGA_1_USER_IO18: now also J6.23 (Pin_23)
- net FPGA_1_USER_IO19: now also J6.64 (Pin_64)
- net FPGA_1_USER_IO2: now also J6.7 (Pin_7)
- net FPGA_1_USER_IO20: now also J6.25 (Pin_25)
- net FPGA_1_USER_IO21: now also J6.66 (Pin_66)
- net FPGA_1_USER_IO22: now also J6.27 (Pin_27)
- net FPGA_1_USER_IO23: now also J6.68 (Pin_68)
- net FPGA_1_USER_IO24: now also J6.29 (Pin_29)
- net FPGA_1_USER_IO25: now also J6.70 (Pin_70)
- net FPGA_1_USER_IO26: now also J6.31 (Pin_31)
- net FPGA_1_USER_IO27: now also J6.72 (Pin_72)
- net FPGA_1_USER_IO28: now also J6.33 (Pin_33)
- net FPGA_1_USER_IO29: now also J6.74 (Pin_74)
- net FPGA_1_USER_IO3: now also J6.48 (Pin_48)
- net FPGA_1_USER_IO30: now also J6.35 (Pin_35)
- net FPGA_1_USER_IO31: now also J6.76 (Pin_76)
- net FPGA_1_USER_IO32: now also J6.37 (Pin_37)
- net FPGA_1_USER_IO33: now also J6.78 (Pin_78)
- net FPGA_1_USER_IO34: now also J6.39 (Pin_39)
- net FPGA_1_USER_IO35: now also J6.80 (Pin_80)
- net FPGA_1_USER_IO36: now also J8.19 (Pin_19)
- net FPGA_1_USER_IO37: now also J8.5 (Pin_5)
- net FPGA_1_USER_IO38: now also J8.21 (Pin_21)
- net FPGA_1_USER_IO39: now also J8.7 (Pin_7)
- net FPGA_1_USER_IO4: now also J6.9 (Pin_9)
- net FPGA_1_USER_IO40: now also J8.23 (Pin_23)
- net FPGA_1_USER_IO41: now also J8.9 (Pin_9)
- net FPGA_1_USER_IO42: now also J8.25 (Pin_25)
- net FPGA_1_USER_IO43: now also J8.11 (Pin_11)
- net FPGA_1_USER_IO44: now also J8.27 (Pin_27)
- net FPGA_1_USER_IO45: now also J8.13 (Pin_13)
- net FPGA_1_USER_IO46: now also J8.29 (Pin_29)
- net FPGA_1_USER_IO47: now also J8.15 (Pin_15)
- net FPGA_1_USER_IO48: now also J8.31 (Pin_31)
- net FPGA_1_USER_IO49: now also J8.17 (Pin_17)
- net FPGA_1_USER_IO5: now also J6.50 (Pin_50)
- net FPGA_1_USER_IO6: now also J6.11 (Pin_11)
- net FPGA_1_USER_IO7: now also J6.52 (Pin_52)
- net FPGA_1_USER_IO8: now also J6.13 (Pin_13)
- net FPGA_1_USER_IO9: now also J6.54 (Pin_54)
- net GND: now also J6.10 (Pin_10), J6.12 (Pin_12), J6.14 (Pin_14), J6.16 (Pin_16), J6.18 (Pin_18), J6.20 (Pin_20), J6.22 (Pin_22), J6.24 (Pin_24), J6.26 (Pin_26), J6.28 (Pin_28), J6.30 (Pin_30), J6.32 (Pin_32), J6.34 (Pin_34), J6.36 (Pin_36), J6.38 (Pin_38), J6.40 (Pin_40), J6.45 (Pin_45), J6.47 (Pin_47), J6.49 (Pin_49), J6.51 (Pin_51), J6.53 (Pin_53), J6.55 (Pin_55), J6.57 (Pin_57), J6.59 (Pin_59), J6.6 (Pin_6), J6.61 (Pin_61), J6.63 (Pin_63), J6.65 (Pin_65), J6.67 (Pin_67), J6.69 (Pin_69), J6.71 (Pin_71), J6.73 (Pin_73), J6.75 (Pin_75), J6.77 (Pin_77), J6.79 (Pin_79), J6.8 (Pin_8), J8.10 (Pin_10), J8.12 (Pin_12), J8.14 (Pin_14), J8.16 (Pin_16), J8.18 (Pin_18), J8.20 (Pin_20), J8.22 (Pin_22), J8.24 (Pin_24), J8.26 (Pin_26), J8.28 (Pin_28), J8.30 (Pin_30), J8.32 (Pin_32), J8.34 (Pin_34), J8.36 (Pin_36), J8.38 (Pin_38), J8.40 (Pin_40), J8.45 (Pin_45), J8.47 (Pin_47), J8.49 (Pin_49), J8.51 (Pin_51), J8.53 (Pin_53), J8.55 (Pin_55), J8.57 (Pin_57), J8.59 (Pin_59), J8.6 (Pin_6), J8.61 (Pin_61), J8.63 (Pin_63), J8.65 (Pin_65), J8.67 (Pin_67), J8.69 (Pin_69), J8.71 (Pin_71), J8.73 (Pin_73), J8.75 (Pin_75), J8.77 (Pin_77), J8.79 (Pin_79), J8.8 (Pin_8), J9.10 (Pin_10), J9.12 (Pin_12), J9.14 (Pin_14), J9.16 (Pin_16), J9.18 (Pin_18), J9.20 (Pin_20), J9.22 (Pin_22), J9.24 (Pin_24), J9.26 (Pin_26), J9.28 (Pin_28), J9.30 (Pin_30), J9.32 (Pin_32), J9.34 (Pin_34), J9.36 (Pin_36), J9.38 (Pin_38), J9.40 (Pin_40), J9.45 (Pin_45), J9.47 (Pin_47), J9.49 (Pin_49), J9.51 (Pin_51), J9.53 (Pin_53), J9.55 (Pin_55), J9.57 (Pin_57), J9.59 (Pin_59), J9.6 (Pin_6), J9.61 (Pin_61), J9.63 (Pin_63), J9.65 (Pin_65), J9.66 (Pin_66), J9.67 (Pin_67), J9.68 (Pin_68), J9.69 (Pin_69), J9.70 (Pin_70), J9.71 (Pin_71), J9.72 (Pin_72), J9.73 (Pin_73), J9.74 (Pin_74), J9.75 (Pin_75), J9.76 (Pin_76), J9.77 (Pin_77), J9.78 (Pin_78), J9.79 (Pin_79), J9.8 (Pin_8), J9.80 (Pin_80)
Other:
- moved on the sheet: C178, C179, C185, C186, C194, C196

Commit message: Updated Layout
Parts:
- removed C173, C174, C175, C176, C191, C192, C193, C195: 100nF, Capacitor_SMD:C_0402_1005Metric, symbol Device:C
- removed R100, R101, R102, R103, R78, R79, R80, R81: 100K, Resistor_SMD:R_0402_1005Metric, symbol Device:R_US
- removed R69, R70, R71, R73, R92, R93, R94, R95: 3K3, Resistor_SMD:R_0402_1005Metric, symbol Device:R_US
- removed SW14, SW15, SW16, SW17, SW22, SW23, SW24, SW25: SW_Push, Button_Switch_SMD:SW_SPST_EVQQ2, symbol Switch:SW_Push
Connections:
- net GND: no longer SW18.1, SW19.1, SW20.1, SW21.1
- new net: SW18.1, SW19.1, SW20.1, SW21.1
Other:
- moved on the sheet: C163, C164, C165, C172, C187, C188, C189, C190, R129, R65, R66, R67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

Commit message: Layout Update
Connections:
- net GND: now also SW18.1, SW19.1, SW20.1, SW21.1
Changed lines of the file:
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@@
   (junction (at 567.69 516.89) (diameter 0) (color 0 0 0 0)
   )
+  (junction (at 262.89 322.58) (diameter 0) (color 0 0 0 0)
+  )
   (junction (at 214.63 96.52) (diameter 0) (color 0 0 0 0)
   )
@@
     (stroke (width 0) (type default) (color 0 0 0 0))
   )
+  (wire (pts (xy 262.89 322.58) (xy 262.89 336.55))
+    (stroke (width 0) (type default) (color 0 0 0 0))
+  )
   (wire (pts (xy 143.51 262.89) (xy 161.29 262.89))
     (stroke (width 0) (type default) (color 0 0 0 0))
@@
     (pin "2")
   )
+  (symbol (lib_id "power:GND") (at 262.89 336.55 0) (unit 1)
+    (in_bom yes) (on_board yes)
+    (property "Reference" "#PWR?" (id 0) (at 262.89 342.9 0)
+      (effects (font (size 1.27 1.27)) hide)
+    )
+    (property "Value" "GND" (id 1) (at 262.89 340.36 0))
+    (property "Footprint" "" (id 2) (at 262.89 336.55 0)
+      (effects (font (size 1.27 1.27)) hide)
+    )
+    (property "Datasheet" "" (id 3) (at 262.89 336.55 0)
+      (effects (font (size 1.27 1.27)) hide)
+    )
+    (pin "1")
+  )
   (symbol (lib_id "Device:R_US") (at 557.53 497.84 90) (unit 1)
