File: DSN/IO.kicad_sch (KiCad schematic)
At the start: 192 parts, among them J10 47272-0001, J11 5-1814832-1, J12 5-1814832-1, J13 5-1814832-1, J14 5-1814832-1, J15 5-1814832-1, J16 5-1814832-1, J17 5-1814832-1, J18 5-1814832-1, J19 5-1814832-1, J20 Conn_02x06_Odd_Even, J21 Conn_02x06_Odd_Even, J22 Conn_02x06_Odd_Even, J23 Conn_02x06_Odd_Even, J24 Conn_02x06_Odd_Even, J25 Conn_02x06_Odd_Even, J26 Conn_02x06_Odd_Even, J33 Conn_02x06_Odd_Even, J6 Conn_02x40_Top_Bottom, J7 47272-0001, J8 Conn_02x40_Top_Bottom, J9 Conn_02x40_Top_Bottom, Q10 2N7002, Q11 2N7002, Q12 2N7002, Q13 2N7002, Q14 2N7002, Q15 2N7002, Q16 2N7002, Q17 2N7002, Q18 2N7002, Q19 2N7002, Q20 2N7002, Q5 2N7002, Q6 2N7002, Q7 2N7002, Q8 2N7002, Q9 2N7002, SW10 SW_Push, SW11 SW_Push, SW12 SW_Push, SW13 SW_Push, SW18 SW_Push, SW19 SW_Push, SW20 SW_Push, SW21 SW_Push

Commit message: Layout Update
Parts:
- removed C180, C181, C182, C183, C184, C198, C199, C200: 100nF, Capacitor_SMD:C_0402_1005Metric, symbol Device:C_Small
- removed R105, R106, R109, R110, R83: 1Meg, Resistor_SMD:R_0402_1005Metric, symbol Device:R_US
- removed R107, R84, R86, R87: 100K, Resistor_SMD:R_0402_1005Metric, symbol Device:R_US
- removed R108: 0R, Resistor_SMD:R_0402_1005Metric, symbol Device:R_US
- removed R85: 1K, Resistor_SMD:R_0402_1005Metric, symbol Device:R_US
- added C38, C39, C40, C41, C51, C52, C53, C54: 100nF, Capacitor_SMD:C_0402_1005Metric, symbol Device:C_Small
- added R26, R27, R73, R78, R79, R80: 1Meg, Resistor_SMD:R_0402_1005Metric, symbol Device:R_US
- added R28, R69, R71, R81: 100K, Resistor_SMD:R_0402_1005Metric, symbol Device:R_US
- added R70: 1K, Resistor_SMD:R_0402_1005Metric, symbol Device:R_US
- C171: MFR PN GRM155R71E104KE14J -> GRM155R71H104ME14J
- R82: value 1Meg -> 0R
Connections:
- net DP_RX_C_HPD is gone; now on net GND: J10.2
- net DP_TX_C_HPD is gone; now on net GND: J7.2
- net +3V3: now also R28.1, R79.2
- net DP_RX_AUX_N: now also C169.2
- net DP_RX_AUX_P: now also C170.1
- net DP_RX_CFG1: now also J10.13, R73.2; no longer J10.4
- net DP_RX_CFG2: now also J10.14, R78.2; no longer J10.6
- net DP_RX_C_AUX_N: now also C169.1, J10.17, R79.1; no longer J10.18
- net DP_RX_C_AUX_P: now also C170.2, J10.15, R80.1; no longer J10.16
- net DP_RX_HPD: now also R82.2
- net DP_RX_LANE1_N: now also J10.7; no longer J10.15
- net DP_RX_LANE1_P: now also J10.9; no longer J10.17
- net DP_RX_LANE2_N: now also J10.4; no longer J10.9
- net DP_RX_LANE2_P: now also J10.6; no longer J10.11
- net DP_RX_LANE3_N: now also J10.1; no longer J10.3
- net DP_RX_LANE3_P: now also J10.3; no longer J10.5
- net DP_RX_PWR: now also C171.1
- net DP_TX_AUX_N: now also C38.2
- net DP_TX_AUX_P: now also C41.1
- net DP_TX_CFG1: now also J7.13, R26.2; no longer J7.4, R82.2
- net DP_TX_CFG2: now also J7.14, R27.2; no longer J7.6
- net DP_TX_C_AUX_N: now also J7.17, C38.1, R28.2; no longer J7.18
- net DP_TX_C_AUX_P: now also J7.15, C41.2, R69.2; no longer J7.16
- net DP_TX_C_LANE0_N: now also J7.3, C39.1; no longer C166.1, J7.5
- net DP_TX_C_LANE0_P: now also J7.1, C51.2; no longer C169.2, J7.3
- net DP_TX_C_LANE1_N: now also J7.6; no longer J7.11
- net DP_TX_C_LANE1_P: now also J7.4, C54.2; no longer C170.2, J7.9
- net DP_TX_C_LANE2_N: now also J7.9, C40.1; no longer C168.1, J7.17
- net DP_TX_C_LANE2_P: now also J7.7, C52.2; no longer C171.2, J7.15
- net DP_TX_C_LANE3_N: now also C168.1
- net DP_TX_C_LANE3_P: now also C166.2
- net DP_TX_HPD: now also R70.2
- net DP_TX_LANE0_N: now also C39.2; no longer C166.2
- net DP_TX_LANE0_P: now also C51.1; no longer C169.1
- net DP_TX_LANE1_P: now also C54.1; no longer C170.1
- net DP_TX_LANE2_N: now also C40.2; no longer C168.2
- net DP_TX_LANE2_P: now also C52.1; no longer C171.1
- net DP_TX_LANE3_N: now also C168.2
- net DP_TX_LANE3_P: now also C166.1
- net DP_TX_PWR: now also C53.1
- net GND: now also C171.2, J10.11, J10.16, J10.18, J10.5, J7.11, J7.16, J7.18, J7.5, C53.2, R26.1, R27.1, R69.1, R70.1, R71.1, R71.2, R73.1, R78.1, R80.2, R81.1, R81.2; no longer J10.1, J10.13, J10.14, J10.7, J7.1, J7.13, J7.14, J7.7

Commit message: Layout Update
Parts:
- J6, J8, J9: symbol Connector_Generic:Conn_02x40_Top_Bottom -> Connector_Generic:Conn_02x40_Odd_Even
Connections:
- net +3V3: now also J6.3 (Pin_3), J6.4 (Pin_4), J8.3 (Pin_3), J8.4 (Pin_4), J9.3 (Pin_3), J9.4 (Pin_4); no longer J6.41 (Pin_41), J6.42 (Pin_42), J8.41 (Pin_41), J8.42 (Pin_42), J9.41 (Pin_41), J9.42 (Pin_42)
- net +5V: now also J6.5 (Pin_5), J6.6 (Pin_6), J6.7 (Pin_7), J6.8 (Pin_8), J8.5 (Pin_5), J8.6 (Pin_6), J8.7 (Pin_7), J8.8 (Pin_8), J9.5 (Pin_5), J9.6 (Pin_6), J9.7 (Pin_7), J9.8 (Pin_8); no longer J6.3 (Pin_3), J6.4 (Pin_4), J6.43 (Pin_43), J6.44 (Pin_44), J8.3 (Pin_3), J8.4 (Pin_4), J8.43 (Pin_43), J8.44 (Pin_44), J9.3 (Pin_3), J9.4 (Pin_4), J9.43 (Pin_43), J9.44 (Pin_44)
- net FPGA_0_USER_IO0: now also J8.65 (Pin_65); no longer J8.33 (Pin_33)
- net FPGA_0_USER_IO1: now also J8.12 (Pin_12); no longer J8.46 (Pin_46)
- net FPGA_0_USER_IO10: now also J9.13 (Pin_13); no longer J9.7 (Pin_7)
- net FPGA_0_USER_IO11: now also J8.32 (Pin_32); no longer J8.56 (Pin_56)
- net FPGA_0_USER_IO12: now also J9.17 (Pin_17); no longer J9.9 (Pin_9)
- net FPGA_0_USER_IO13: now also J8.36 (Pin_36); no longer J8.58 (Pin_58)
- net FPGA_0_USER_IO14: now also J9.21 (Pin_21); no longer J9.11 (Pin_11)
- net FPGA_0_USER_IO15: now also J8.40 (Pin_40); no longer J8.60 (Pin_60)
- net FPGA_0_USER_IO16: now also J9.25 (Pin_25); no longer J9.13 (Pin_13)
- net FPGA_0_USER_IO17: now also J8.44 (Pin_44); no longer J8.62 (Pin_62)
- net FPGA_0_USER_IO18: now also J9.29 (Pin_29); no longer J9.15 (Pin_15)
- net FPGA_0_USER_IO19: now also J8.48 (Pin_48); no longer J8.64 (Pin_64)
- net FPGA_0_USER_IO2: now also J8.69 (Pin_69); no longer J8.35 (Pin_35)
- net FPGA_0_USER_IO20: now also J9.33 (Pin_33); no longer J9.17 (Pin_17)
- net FPGA_0_USER_IO21: now also J8.52 (Pin_52); no longer J8.66 (Pin_66)
- net FPGA_0_USER_IO22: now also J9.37 (Pin_37); no longer J9.19 (Pin_19)
- net FPGA_0_USER_IO23: now also J8.56 (Pin_56); no longer J8.68 (Pin_68)
- net FPGA_0_USER_IO24: now also J9.41 (Pin_41); no longer J9.21 (Pin_21)
- net FPGA_0_USER_IO25: now also J8.60 (Pin_60); no longer J8.70 (Pin_70)
- net FPGA_0_USER_IO26: now also J9.45 (Pin_45); no longer J9.23 (Pin_23)
- net FPGA_0_USER_IO27: now also J8.64 (Pin_64); no longer J8.72 (Pin_72)
- net FPGA_0_USER_IO28: now also J9.49 (Pin_49); no longer J9.25 (Pin_25)
- net FPGA_0_USER_IO29: now also J8.68 (Pin_68); no longer J8.74 (Pin_74)
- net FPGA_0_USER_IO3: now also J8.16 (Pin_16); no longer J8.48 (Pin_48)
- net FPGA_0_USER_IO30: now also J9.53 (Pin_53); no longer J9.27 (Pin_27)
- net FPGA_0_USER_IO31: now also J8.72 (Pin_72); no longer J8.76 (Pin_76)
- net FPGA_0_USER_IO32: now also J9.57 (Pin_57); no longer J9.29 (Pin_29)
- net FPGA_0_USER_IO33: now also J8.76 (Pin_76); no longer J8.78 (Pin_78)
- net FPGA_0_USER_IO34: now also J9.61 (Pin_61); no longer J9.31 (Pin_31)
- net FPGA_0_USER_IO36: now also J9.65 (Pin_65); no longer J9.33 (Pin_33)
- net FPGA_0_USER_IO37: now also J9.12 (Pin_12); no longer J9.46 (Pin_46)
- net FPGA_0_USER_IO38: now also J9.69 (Pin_69); no longer J9.35 (Pin_35)
- net FPGA_0_USER_IO39: now also J9.16 (Pin_16); no longer J9.48 (Pin_48)
- net FPGA_0_USER_IO4: now also J8.73 (Pin_73); no longer J8.37 (Pin_37)
- net FPGA_0_USER_IO40: now also J9.73 (Pin_73); no longer J9.37 (Pin_37)
- net FPGA_0_USER_IO41: now also J9.20 (Pin_20); no longer J9.50 (Pin_50)
- net FPGA_0_USER_IO42: now also J9.77 (Pin_77); no longer J9.39 (Pin_39)
- net FPGA_0_USER_IO43: now also J9.24 (Pin_24); no longer J9.52 (Pin_52)
- net FPGA_0_USER_IO44: now also J9.40 (Pin_40); no longer J9.60 (Pin_60)
- net FPGA_0_USER_IO45: now also J9.28 (Pin_28); no longer J9.54 (Pin_54)
- net FPGA_0_USER_IO46: now also J9.44 (Pin_44); no longer J9.62 (Pin_62)
- net FPGA_0_USER_IO47: now also J9.32 (Pin_32); no longer J9.56 (Pin_56)
- net FPGA_0_USER_IO48: now also J9.48 (Pin_48); no longer J9.64 (Pin_64)
- net FPGA_0_USER_IO49: now also J9.36 (Pin_36); no longer J9.58 (Pin_58)
- net FPGA_0_USER_IO5: now also J8.20 (Pin_20); no longer J8.50 (Pin_50)
- net FPGA_0_USER_IO6: now also J8.77 (Pin_77); no longer J8.39 (Pin_39)
- net FPGA_0_USER_IO7: now also J8.24 (Pin_24); no longer J8.52 (Pin_52)
- net FPGA_0_USER_IO8: now also J9.9 (Pin_9); no longer J9.5 (Pin_5)
- net FPGA_0_USER_IO9: now also J8.28 (Pin_28); no longer J8.54 (Pin_54)
- net FPGA_1_USER_IO0: now also J6.9 (Pin_9); no longer J6.5 (Pin_5)
- net FPGA_1_USER_IO1: now also J6.12 (Pin_12); no longer J6.46 (Pin_46)
- net FPGA_1_USER_IO10: now also J6.29 (Pin_29); no longer J6.15 (Pin_15)
- net FPGA_1_USER_IO11: now also J6.32 (Pin_32); no longer J6.56 (Pin_56)
- net FPGA_1_USER_IO12: now also J6.33 (Pin_33); no longer J6.17 (Pin_17)
- net FPGA_1_USER_IO13: now also J6.36 (Pin_36); no longer J6.58 (Pin_58)
- net FPGA_1_USER_IO14: now also J6.37 (Pin_37); no longer J6.19 (Pin_19)
- net FPGA_1_USER_IO15: now also J6.40 (Pin_40); no longer J6.60 (Pin_60)
- net FPGA_1_USER_IO16: now also J6.41 (Pin_41); no longer J6.21 (Pin_21)
- net FPGA_1_USER_IO17: now also J6.44 (Pin_44); no longer J6.62 (Pin_62)
- net FPGA_1_USER_IO18: now also J6.45 (Pin_45); no longer J6.23 (Pin_23)
- net FPGA_1_USER_IO19: now also J6.48 (Pin_48); no longer J6.64 (Pin_64)
- net FPGA_1_USER_IO2: now also J6.13 (Pin_13); no longer J6.7 (Pin_7)
- net FPGA_1_USER_IO20: now also J6.49 (Pin_49); no longer J6.25 (Pin_25)
- net FPGA_1_USER_IO21: now also J6.52 (Pin_52); no longer J6.66 (Pin_66)
- net FPGA_1_USER_IO22: now also J6.53 (Pin_53); no longer J6.27 (Pin_27)
- net FPGA_1_USER_IO23: now also J6.56 (Pin_56); no longer J6.68 (Pin_68)
- net FPGA_1_USER_IO24: now also J6.57 (Pin_57); no longer J6.29 (Pin_29)
- net FPGA_1_USER_IO25: now also J6.60 (Pin_60); no longer J6.70 (Pin_70)
- net FPGA_1_USER_IO26: now also J6.61 (Pin_61); no longer J6.31 (Pin_31)
- net FPGA_1_USER_IO27: now also J6.64 (Pin_64); no longer J6.72 (Pin_72)
- net FPGA_1_USER_IO28: now also J6.65 (Pin_65); no longer J6.33 (Pin_33)
- net FPGA_1_USER_IO29: now also J6.68 (Pin_68); no longer J6.74 (Pin_74)
- net FPGA_1_USER_IO3: now also J6.16 (Pin_16); no longer J6.48 (Pin_48)
- net FPGA_1_USER_IO30: now also J6.69 (Pin_69); no longer J6.35 (Pin_35)
- net FPGA_1_USER_IO31: now also J6.72 (Pin_72); no longer J6.76 (Pin_76)
- net FPGA_1_USER_IO32: now also J6.73 (Pin_73); no longer J6.37 (Pin_37)
- net FPGA_1_USER_IO33: now also J6.76 (Pin_76); no longer J6.78 (Pin_78)
- net FPGA_1_USER_IO34: now also J6.77 (Pin_77); no longer J6.39 (Pin_39)
- net FPGA_1_USER_IO36: now also J8.37 (Pin_37); no longer J8.19 (Pin_19)
- net FPGA_1_USER_IO37: now also J8.9 (Pin_9); no longer J8.5 (Pin_5)
- net FPGA_1_USER_IO38: now also J8.41 (Pin_41); no longer J8.21 (Pin_21)
- net FPGA_1_USER_IO39: now also J8.13 (Pin_13); no longer J8.7 (Pin_7)
- net FPGA_1_USER_IO4: now also J6.17 (Pin_17); no longer J6.9 (Pin_9)
- net FPGA_1_USER_IO40: now also J8.45 (Pin_45); no longer J8.23 (Pin_23)
- net FPGA_1_USER_IO41: now also J8.17 (Pin_17); no longer J8.9 (Pin_9)
- net FPGA_1_USER_IO42: now also J8.49 (Pin_49); no longer J8.25 (Pin_25)
- net FPGA_1_USER_IO43: now also J8.21 (Pin_21); no longer J8.11 (Pin_11)
- net FPGA_1_USER_IO44: now also J8.53 (Pin_53); no longer J8.27 (Pin_27)
- net FPGA_1_USER_IO45: now also J8.25 (Pin_25); no longer J8.13 (Pin_13)
- net FPGA_1_USER_IO46: now also J8.57 (Pin_57); no longer J8.29 (Pin_29)
- net FPGA_1_USER_IO47: now also J8.29 (Pin_29); no longer J8.15 (Pin_15)
- net FPGA_1_USER_IO48: now also J8.61 (Pin_61); no longer J8.31 (Pin_31)
- net FPGA_1_USER_IO49: now also J8.33 (Pin_33); no longer J8.17 (Pin_17)
- net FPGA_1_USER_IO5: now also J6.20 (Pin_20); no longer J6.50 (Pin_50)
- net FPGA_1_USER_IO6: now also J6.21 (Pin_21); no longer J6.11 (Pin_11)
- net FPGA_1_USER_IO7: now also J6.24 (Pin_24); no longer J6.52 (Pin_52)
- net FPGA_1_USER_IO8: now also J6.25 (Pin_25); no longer J6.13 (Pin_13)
- net FPGA_1_USER_IO9: now also J6.28 (Pin_28); no longer J6.54 (Pin_54)
- net GND: now also J6.11 (Pin_11), J6.15 (Pin_15), J6.19 (Pin_19), J6.23 (Pin_23), J6.27 (Pin_27), J6.31 (Pin_31), J6.35 (Pin_35), J6.39 (Pin_39), J6.42 (Pin_42), J6.43 (Pin_43), J6.46 (Pin_46), J6.50 (Pin_50), J6.54 (Pin_54), J6.58 (Pin_58), J6.62 (Pin_62), J6.66 (Pin_66), J6.70 (Pin_70), J6.74 (Pin_74), J6.78 (Pin_78), J8.11 (Pin_11), J8.15 (Pin_15), J8.19 (Pin_19), J8.23 (Pin_23), J8.27 (Pin_27), J8.31 (Pin_31), J8.35 (Pin_35), J8.39 (Pin_39), J8.42 (Pin_42), J8.43 (Pin_43), J8.46 (Pin_46), J8.50 (Pin_50), J8.54 (Pin_54), J8.58 (Pin_58), J8.62 (Pin_62), J8.66 (Pin_66), J8.70 (Pin_70), J8.74 (Pin_74), J8.78 (Pin_78), J9.11 (Pin_11), J9.15 (Pin_15), J9.19 (Pin_19), J9.23 (Pin_23), J9.27 (Pin_27), J9.31 (Pin_31), J9.35 (Pin_35), J9.39 (Pin_39), J9.42 (Pin_42), J9.43 (Pin_43), J9.46 (Pin_46), J9.50 (Pin_50), J9.52 (Pin_52), J9.54 (Pin_54), J9.56 (Pin_56), J9.58 (Pin_58), J9.60 (Pin_60), J9.62 (Pin_62), J9.64 (Pin_64); no longer J6.12 (Pin_12), J6.16 (Pin_16), J6.20 (Pin_20), J6.24 (Pin_24), J6.28 (Pin_28), J6.32 (Pin_32), J6.36 (Pin_36), J6.40 (Pin_40), J6.45 (Pin_45), J6.49 (Pin_49), J6.53 (Pin_53), J6.57 (Pin_57), J6.6 (Pin_6), J6.61 (Pin_61), J6.65 (Pin_65), J6.69 (Pin_69), J6.73 (Pin_73), J6.77 (Pin_77), J6.8 (Pin_8), J8.12 (Pin_12), J8.16 (Pin_16), J8.20 (Pin_20), J8.24 (Pin_24), J8.28 (Pin_28), J8.32 (Pin_32), J8.36 (Pin_36), J8.40 (Pin_40), J8.45 (Pin_45), J8.49 (Pin_49), J8.53 (Pin_53), J8.57 (Pin_57), J8.6 (Pin_6), J8.61 (Pin_61), J8.65 (Pin_65), J8.69 (Pin_69), J8.73 (Pin_73), J8.77 (Pin_77), J8.8 (Pin_8), J9.12 (Pin_12), J9.16 (Pin_16), J9.20 (Pin_20), J9.24 (Pin_24), J9.28 (Pin_28), J9.32 (Pin_32), J9.36 (Pin_36), J9.40 (Pin_40), J9.45 (Pin_45), J9.49 (Pin_49), J9.53 (Pin_53), J9.57 (Pin_57), J9.6 (Pin_6), J9.61 (Pin_61), J9.65 (Pin_65), J9.69 (Pin_69), J9.73 (Pin_73), J9.77 (Pin_77), J9.8 (Pin_8)
Changed lines of the file:
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@@
     (pin "2")
   )
-  (symbol (lib_id "Connector_Generic:Conn_02x40_Top_Bottom") (at 220.98 91.44 0) (unit 1)
+  (symbol (lib_id "Connector_Generic:Conn_02x40_Odd_Even") (at 220.98 91.44 0) (unit 1)
     (in_bom yes) (on_board yes) (fields_autoplaced)
     (property "Reference" "J8" (id 0) (at 222.25 36.83 0))
@@
     (pin "2")
   )
-  (symbol (lib_id "Connector_Generic:Conn_02x40_Top_Bottom") (at 316.23 91.44 0) (unit 1)
+  (symbol (lib_id "Connector_Generic:Conn_02x40_Odd_Even") (at 316.23 91.44 0) (unit 1)
     (in_bom yes) (on_board yes) (fields_autoplaced)
     (property "Reference" "J9" (id 0) (at 317.5 36.83 0))
@@
     (pin "1")
   )
-  (symbol (lib_id "Connector_Generic:Conn_02x40_Top_Bottom") (at 124.46 91.44 0) (unit 1)
+  (symbol (lib_id "Connector_Generic:Conn_02x40_Odd_Even") (at 124.46 91.44 0) (unit 1)
     (in_bom yes) (on_board yes) (fields_autoplaced)
     (property "Reference" "J6" (id 0) (at 125.73 36.83 0))
