File: DSN/ArtixDuo.kicad_pcb (KiCad board)
At the start: 8 copper layers, 203.2 x 127 mm, 771 parts, among them J1 Conn_01x03_Male, J10 47272-0001, J11 5-1814832-1, J12 5-1814832-1, J13 5-1814832-1, J14 5-1814832-1, J15 5-1814832-1, J16 5-1814832-1, J17 5-1814832-1, J18 5-1814832-1, J19 5-1814832-1, J2 USB_C_Receptacle_USB2.0, J20 Conn_02x06_Odd_Even, J21 Conn_02x06_Odd_Even, J22 Conn_02x06_Odd_Even, J23 Conn_02x06_Odd_Even, J24 Conn_02x06_Odd_Even, J25 Conn_02x06_Odd_Even, J26 Conn_02x06_Odd_Even, J27 USB_C_Receptacle_USB2.0, J28 Conn_02x07_Odd_Even, J29 Conn_01x03_Male, J3 Conn_01x08, J30 Conn_01x03_Male, J31 Conn_02x07_Odd_Even, J32 Conn_Coaxial, J33 Conn_02x06_Odd_Even, J4 USB_C_Receptacle_USB2.0, J5 Conn_Coaxial, J6 Conn_02x40_Top_Bottom, J7 47272-0001, J8 Conn_02x40_Top_Bottom, J9 Conn_02x40_Top_Bottom, Q1 AON6411, Q10 2N7002, Q11 2N7002, Q12 2N7002, Q13 2N7002, Q14 2N7002, Q15 2N7002, Q16 2N7002, Q17 2N7002, Q18 2N7002, Q19 2N7002, Q2 AON6411, Q20 2N7002, Q21 AON6411, Q22 AO3401A, Q23 2N7002K, Q3 AO3401A, Q4 2N7002K, Q5 2N7002, Q6 2N7002, Q7 2N7002, Q8 2N7002, Q9 2N7002, SW1 SW_SPST, SW10 SW_Push, SW11 SW_Push, SW12 SW_Push, SW13 SW_Push, SW14 SW_Push, SW15 SW_Push, SW16 SW_Push, SW17 SW_Push, SW18 SW_Push, SW19 SW_Push, SW2 SW_Push, SW20 SW_Push, SW21 SW_Push, SW22 SW_Push, SW23 SW_Push, SW24 SW_Push, SW25 SW_Push, SW26 SW_DIP_x03, SW27 SW_Push, SW28 SW_Push, SW3 SW_Push, SW4 SW_Push, SW5 SW_Push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

Commit message: Updated Layout
Parts:
- removed C38, C39, C40, C41, C51, C52, C53, C54: 22uF, Capacitor_SMD:C_1206_3216Metric
- removed H11, H12, H6, H7, H8: MountingHole, MountingHole:MountingHole_3.5mm
- removed R26: 5.1K, Resistor_SMD:R_0402_1005Metric
- removed R27, R28: 27R, Resistor_SMD:R_0402_1005Metric
- removed SW3, SW4, SW6: SW_Push, Button_Switch_SMD:SW_SPST_B3SL-1022P
- added D42: TPD1E05U06QDPYRQ1, Diode_SMD:D_0402_1005Metric, F.Cu at (202.0, 90.0)
- added J34: USB_C_Receptacle_USB2.0, Connector_USB:USB_C_Receptacle_GCT_USB4085, F.Cu at (206.6, 87.5)
- added TP19: TestPoint_Probe, TestPoint:TestPoint_Loop_D1.80mm_Drill1.0mm_Beaded, F.Cu at (215.2, 106.0)
- added TP20: TestPoint_Probe, TestPoint:TestPoint_Loop_D1.80mm_Drill1.0mm_Beaded, F.Cu at (215.4, 82.7)
- added TP21: TestPoint_Probe, TestPoint:TestPoint_Loop_D1.80mm_Drill1.0mm_Beaded, F.Cu at (107.7, 37.1)
- added U32: RP2040, Package_DFN_QFN:QFN-56-1EP_7x7mm_P0.4mm_EP3.2x3.2mm, F.Cu at (203.6, 103.1)
- added Y3: Crystal_GND24, Crystal:Crystal_SMD_3225-4Pin_3.2x2.5mm, F.Cu at (156.8, 95.3)
- C174, C176: value 100nF -> 20pF
- C191, C193: value 100nF -> 2.2uF
- C229, C231, C232, C233, C240, C26, C63, L6, L7, R162, R163, R172: moved to B.Cu
- C28: value 10uF -> 2.2uF; footprint Capacitor_SMD:C_0805_2012Metric -> Capacitor_SMD:C_0402_1005Metric
- C30: value 2.2uF -> 100nF
- C31: value 10uF -> 100nF; footprint Capacitor_SMD:C_0805_2012Metric -> Capacitor_SMD:C_0402_1005Metric; moved to B.Cu
- D3, D37: value BZV55B5V6 -> 5.6V Zener; footprint Diode_SMD:D_MiniMELF -> Diode_SMD:D_SOD-123
- D6: value TPD1E10B06DPYR -> LED; footprint Diode_SMD:D_0402_1005Metric -> LED_SMD:LED_0603_1608Metric
- D7: value BZV55B5V6 -> TPD1E10B06DPYR; footprint Diode_SMD:D_MiniMELF -> Diode_SMD:D_0402_1005Metric
- D8: value TPD1E05U06QDPYRQ1 -> 5.6V Zener; footprint Diode_SMD:D_0402_1005Metric -> Diode_SMD:D_SOD-123
- J4: value USB_C_Receptacle_USB2.0 -> Conn_01x03_Male; footprint Connector_USB:USB_C_Receptacle_GCT_USB4085 -> Connector_PinHeader_2.54mm:PinHeader_1x03_P2.54mm_Vertical
- R11: value 3K3 -> 0R
- R13: value 3K3 -> 1K
- R15: value 3K3 -> 470R
- R16: value 3K3 -> 200R
- R18: value 100K -> 1R
- R19: value 100K -> 1Meg
- R20: value 100K -> 10K
- R21: value 100K -> 5.1K; moved to B.Cu
- R23: value 1Meg -> 5.1K; moved to B.Cu
- R24: value 10K -> 27R
- R25: value 5.1K -> 27R
- SW2: value SW_Push -> SW_SPST; footprint Button_Switch_SMD:SW_SPST_B3SL-1022P -> Button_Switch_SMD:SW_SPST_B3U-1000P
- TP1, TP10, TP13, TP14, TP17, TP18, TP2, TP3, TP4, TP5, TP6, TP7, TP8, TP9: footprint TestPoint:TestPoint_Loop_D2.50mm_Drill1.85mm -> TestPoint:TestPoint_Loop_D1.80mm_Drill1.0mm_Beaded
- U3: value Teensy4.1 -> W25Q16JVUXIQ; footprint teensy:Teensy41 -> Package_SON:WSON-8-1EP_4x4mm_P0.8mm_EP2.2x3mm_ThermalVias
- Y1: value Crystal_GND23 -> Crystal_GND24
- Y2: value 12Mhz -> Crystal_GND24; footprint Crystal:Crystal_SMD_ECS_CSM3X-2Pin_7.6x4.1mm -> Crystal:Crystal_SMD_3225-4Pin_3.2x2.5mm
- moved H3 618.2 mm to (119.4, 200.7)
- moved C6 522.2 mm to (217.7, 163.6), turned to 90 degrees
- moved C4 520.8 mm to (213.9, 120.7), turned to -90 degrees
- moved C2 518.0 mm to (221.8, 107.0)
- moved H4 517.4 mm to (218.6, 63.8)
- moved C5 517.1 mm to (213.7, 163.6), turned to 90 degrees
- moved C3 516.9 mm to (217.9, 120.7), turned to -90 degrees
- moved C1 514.4 mm to (216.7, 100.9), turned to -90 degrees
- moved H1 444.4 mm to (312.4, 200.7)
- moved C173 417.4 mm to (204.4, 96.9), turned to 90 degrees
- moved U3 414.4 mm to (198.7, 93.2), turned to 90 degrees
- moved R49 404.1 mm to (169.1, 118.5), turned to -45 degrees
- moved C62 402.5 mm to (169.8, 126.3), turned to 135 degrees
- moved R40 399.3 mm to (210.0, 142.5)
- moved R33 397.4 mm to (211.0, 132.5), turned to 180 degrees
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Connections:
- C173 pad 1: /TopSheet/UserIO/FPGA_1_SW4_R -> /TopSheet/RP2040 MCU/+3V3_RPi2_AUX
- C174 pad 1: /TopSheet/UserIO/FPGA_1_SW5_R -> /TopSheet/RP2040 MCU/XI_RPi2
- C175 pad 1: /TopSheet/UserIO/FPGA_1_SW6_R -> /TopSheet/RP2040 MCU/+3V3_RPi2_AUX
- C176 pad 1: /TopSheet/UserIO/FPGA_1_SW7_R -> /TopSheet/RP2040 MCU/XO_RPi2
- C191 pad 1: /TopSheet/UserIO/FPGA_0_SW4_R -> Net-(C191-Pad1)
- C192 pad 1: /TopSheet/UserIO/FPGA_0_SW5_R -> +5V
- C193 pad 1: /TopSheet/UserIO/FPGA_0_SW6_R -> +5V
- C21 pad 1: /TopSheet/SMC/RPi_SW2_R -> /TopSheet/RP2040 MCU/RPi2_1V1
- C22 pad 1: /TopSheet/SMC/RPi_SW3_R -> /TopSheet/RP2040 MCU/+3V3_RPi2_AUX
- C24 pad 1: /TopSheet/SMC/RPi_SW4_R -> /TopSheet/RP2040 MCU/RPi2_1V1
- C26 pad 1: /TopSheet/SMC/RPi_SW5_R -> /TopSheet/RP2040 MCU/RPi2_1V1
- C28 pad 1: +3V3 -> /TopSheet/RP2040 MCU/RPi2_1V1
- C29 pad 1: +5V -> /TopSheet/RP2040 MCU/+3V3_RPi2_AUX
- C30 pad 1: +5V -> /TopSheet/RP2040 MCU/+3V3_RPi2_AUX
- C31 pad 1: +3V3 -> /TopSheet/RP2040 MCU/+3V3_RPi2_AUX
- C56 pad 1: Net-(C52-Pad1) -> Net-(C56-Pad1)
- C58 pad 1: Net-(C52-Pad1) -> Net-(C56-Pad1)
- D6 pad 2: /TopSheet/Teensy41 MCU/VBUS_AUX_MCU -> Net-(D6-Pad2)
- D7 pad 1: +5V -> GND
- D7 pad 2: Net-(D7-Pad2) -> /TopSheet/RP2040 MCU/VBUS_AUX_RPi2
- D8 pad 1: GND -> +5V
- D8 pad 2: /TopSheet/Teensy41 MCU/USB_D_MCU_P -> Net-(Q2-Pad4)
- D9 pad 2: /TopSheet/Teensy41 MCU/USB_D_MCU_N -> /TopSheet/RP2040 MCU/USB_D_RPi2_P
- L4 pad 2: Net-(C52-Pad1) -> Net-(C56-Pad1)
- Q2 pad 4: Net-(D7-Pad2) -> Net-(Q2-Pad4)
- Q2 pad 5: /TopSheet/Teensy41 MCU/VBUS_AUX_MCU -> /TopSheet/RP2040 MCU/VBUS_AUX_RPi2
- R11 pad 1: /TopSheet/SMC/+3V3_RPi_AUX -> +3.3VA
- R11 pad 2: /TopSheet/SMC/RPi_SW2_R -> /TopSheet/RP2040 MCU/+3V3_RPi2_AUX
- R13 pad 1: /TopSheet/SMC/+3V3_RPi_AUX -> /TopSheet/RP2040 MCU/QSPI2_CS
- R13 pad 2: /TopSheet/SMC/RPi_SW3_R -> Net-(R13-Pad2)
- R15 pad 1: /TopSheet/SMC/+3V3_RPi_AUX -> Net-(R15-Pad1)
- R15 pad 2: /TopSheet/SMC/RPi_SW4_R -> Net-(D6-Pad2)
- R16 pad 1: /TopSheet/SMC/+3V3_RPi_AUX -> /TopSheet/RP2040 MCU/+3V3_RPi2_AUX
- R16 pad 2: /TopSheet/SMC/RPi_SW5_R -> /TopSheet/RP2040 MCU/RPi2_ADC_REF
- R18 pad 1: /TopSheet/SMC/RPi_SW2_R -> /TopSheet/RP2040 MCU/RPi2_ADC_REF
- R18 pad 2: /TopSheet/SMC/RPi_SW2 -> Net-(C191-Pad1)
- R19 pad 1: /TopSheet/SMC/RPi_SW3_R -> GND
- R19 pad 2: /TopSheet/SMC/RPi_SW3 -> Net-(J34-PadS1)
- R20 pad 1: /TopSheet/SMC/RPi_SW4_R -> Net-(Q2-Pad4)
- R20 pad 2: /TopSheet/SMC/RPi_SW4 -> GND
- R21 pad 1: /TopSheet/SMC/RPi_SW5_R -> Net-(J34-PadA5)
- R21 pad 2: /TopSheet/SMC/RPi_SW5 -> GND
- R23 pad 1: GND -> Net-(J34-PadB5)
- R23 pad 2: Net-(J4-PadS1) -> GND
- R24 pad 1: Net-(D7-Pad2) -> /TopSheet/RP2040 MCU/USB_D_RPi2_R_P
- R24 pad 2: GND -> /TopSheet/RP2040 MCU/USB_D_RPi2_P
- R25 pad 1: Net-(J4-PadA5) -> /TopSheet/RP2040 MCU/USB_D_RPi2_R_N
- R25 pad 2: GND -> /TopSheet/RP2040 MCU/USB_D_RPi2_N
- R47 pad 1: Net-(C52-Pad1) -> Net-(C56-Pad1)
- SW18 pad 1: GND -> Net-(SW18-Pad1)
- SW19 pad 1: GND -> Net-(SW18-Pad1)
- SW2 pad 1: GND -> Net-(R13-Pad2)
- SW2 pad 2: /TopSheet/SMC/RPi_SW3_R -> GND
- SW20 pad 1: GND -> Net-(SW18-Pad1)
- SW21 pad 1: GND -> Net-(SW18-Pad1)
- TP10 pad 1: Net-(C52-Pad1) -> Net-(C56-Pad1)
- TP13 pad 1: /TopSheet/USB_UART_JTAG/+3V3_VCCIO -> /TopSheet/USB_UART_JTAG/VBUS_AUX_PROG
- TP14 pad 1: /TopSheet/USB_UART_JTAG/FT_VCORE -> /TopSheet/USB_UART_JTAG/+3V3_VCCIO
- TP17 pad 1: +5V -> /TopSheet/USB_UART_JTAG/FT_VCORE
- TP18 pad 1: +3.3VA -> +5V
- TP4 pad 1: /TopSheet/Teensy41 MCU/VBUS_AUX_MCU -> /TopSheet/RP2040 MCU/RPi2_1V1
- U10 pad A13: /TopSheet/FPGA_0/FPGA_0_LINK_IO69 -> /TopSheet/FPGA_0/FPGA_0_LINK_IO30
- U10 pad A14: /TopSheet/FPGA_0/FPGA_0_LINK_IO70 -> /TopSheet/FPGA_0/FPGA_0_LINK_IO29
- U10 pad A15: /TopSheet/FPGA_0/FPGA_0_LINK_IO67 -> /TopSheet/FPGA_0/FPGA_0_LINK_IO32
- U10 pad A16: /TopSheet/FPGA_0/FPGA_0_LINK_IO68 -> /TopSheet/FPGA_0/FPGA_0_LINK_IO31
- U10 pad A18: /TopSheet/FPGA_0/FPGA_0_LINK_IO83 -> /TopSheet/FPGA_0/FPGA_0_LINK_IO16
- U10 pad A19: /TopSheet/FPGA_0/FPGA_0_LINK_IO84 -> /TopSheet/FPGA_0/FPGA_0_LINK_IO15
- U10 pad A20: /TopSheet/FPGA_0/FPGA_0_LINK_IO82 -> /TopSheet/FPGA_0/FPGA_0_LINK_IO17
- U10 pad A21: /TopSheet/FPGA_0/FPGA_0_LINK_IO92 -> /TopSheet/FPGA_0/FPGA_0_LINK_IO7
- U10 pad AA18: /TopSheet/FPGA_1/FPGA_1_SPI_MCU_TX -> unconnected-(U10-PadAA18)
- U10 pad AA20: /TopSheet/FPGA_1/FPGA_1_MCU_IO8 -> /TopSheet/FPGA_1/FPGA_1_MCU_IO1
- U10 pad AA21: /TopSheet/FPGA_1/FPGA_1_MCU_IO9 -> /TopSheet/FPGA_1/FPGA_1_MCU_IO2
- U10 pad AB21: /TopSheet/FPGA_1/FPGA_1_MCU_IO12 -> /TopSheet/FPGA_1/FPGA_1_MCU_IO5
- U10 pad AB22: /TopSheet/FPGA_1/FPGA_1_MCU_IO13 -> /TopSheet/FPGA_1/FPGA_1_MCU_IO6
- U10 pad B13: /TopSheet/FPGA_0/FPGA_0_LINK_IO66 -> /TopSheet/FPGA_0/FPGA_0_LINK_IO33
- U10 pad B15: /TopSheet/FPGA_0/FPGA_0_LINK_IO63 -> /TopSheet/FPGA_0/FPGA_0_LINK_IO36
- U10 pad B16: /TopSheet/FPGA_0/FPGA_0_LINK_IO64 -> /TopSheet/FPGA_0/FPGA_0_LINK_IO35
- U10 pad B17: /TopSheet/FPGA_0/FPGA_0_LINK_IO71 -> /TopSheet/FPGA_0/FPGA_0_LINK_IO28
- U10 pad B18: /TopSheet/FPGA_0/FPGA_0_LINK_IO72 -> /TopSheet/FPGA_0/FPGA_0_LINK_IO27
- U10 pad B20: /TopSheet/FPGA_0/FPGA_0_LINK_IO81 -> /TopSheet/FPGA_0/FPGA_0_LINK_IO18
- U10 pad B21: /TopSheet/FPGA_0/FPGA_0_LINK_IO91 -> /TopSheet/FPGA_0/FPGA_0_LINK_IO8
- U10 pad B22: /TopSheet/FPGA_0/FPGA_0_LINK_IO90 -> /TopSheet/FPGA_0/FPGA_0_LINK_IO9
- U10 pad C13: /TopSheet/FPGA_0/FPGA_0_LINK_IO65 -> /TopSheet/FPGA_0/FPGA_0_LINK_IO34
- U10 pad C14: /TopSheet/FPGA_0/FPGA_0_LINK_IO55 -> /TopSheet/FPGA_0/FPGA_0_LINK_IO44
- U10 pad C15: /TopSheet/FPGA_0/FPGA_0_LINK_IO56 -> /TopSheet/FPGA_0/FPGA_0_LINK_IO43
- U10 pad C17: /TopSheet/FPGA_0/FPGA_0_LINK_IO74 -> /TopSheet/FPGA_0/FPGA_0_LINK_IO25
- U10 pad C18: /TopSheet/FPGA_0/FPGA_0_LINK_IO75 -> /TopSheet/FPGA_0/FPGA_0_LINK_IO24
- U10 pad C19: /TopSheet/FPGA_0/FPGA_0_LINK_IO76 -> /TopSheet/FPGA_0/FPGA_0_LINK_IO23
- U10 pad C20: /TopSheet/FPGA_0/FPGA_0_LINK_IO88 -> /TopSheet/FPGA_0/FPGA_0_LINK_IO11
- U10 pad C22: /TopSheet/FPGA_0/FPGA_0_LINK_IO89 -> /TopSheet/FPGA_0/FPGA_0_LINK_IO10
- U10 pad D14: /TopSheet/FPGA_0/FPGA_0_LINK_IO61 -> /TopSheet/FPGA_0/FPGA_0_LINK_IO38
- U10 pad D15: /TopSheet/FPGA_0/FPGA_0_LINK_IO62 -> /TopSheet/FPGA_0/FPGA_0_LINK_IO37
- U10 pad D16: /TopSheet/FPGA_0/FPGA_0_LINK_IO60 -> /TopSheet/FPGA_0/FPGA_0_LINK_IO39
- U10 pad D17: /TopSheet/FPGA_0/FPGA_0_LINK_IO73 -> /TopSheet/FPGA_0/FPGA_0_LINK_IO26
- U10 pad D19: /TopSheet/FPGA_0/FPGA_0_LINK_IO78 -> /TopSheet/FPGA_0/FPGA_0_LINK_IO21
- U10 pad D20: /TopSheet/FPGA_0/FPGA_0_LINK_IO87 -> /TopSheet/FPGA_0/FPGA_0_LINK_IO12
- U10 pad D21: /TopSheet/FPGA_0/FPGA_0_LINK_IO96 -> /TopSheet/FPGA_0/FPGA_0_LINK_IO3
- U10 pad D22: /TopSheet/FPGA_0/FPGA_0_LINK_IO94 -> /TopSheet/FPGA_0/FPGA_0_LINK_IO5
- U10 pad E13: /TopSheet/FPGA_0/FPGA_0_LINK_IO57 -> /TopSheet/FPGA_0/FPGA_0_LINK_IO42
- U10 pad E14: /TopSheet/FPGA_0/FPGA_0_LINK_IO58 -> /TopSheet/FPGA_0/FPGA_0_LINK_IO41
- U10 pad E16: /TopSheet/FPGA_0/FPGA_0_LINK_IO59 -> /TopSheet/FPGA_0/FPGA_0_LINK_IO40
- U10 pad E17: /TopSheet/FPGA_0/FPGA_0_LINK_IO54 -> /TopSheet/FPGA_0/FPGA_0_LINK_IO45
- U10 pad E18: /TopSheet/FPGA_0/FPGA_0_LINK_IO80 -> /TopSheet/FPGA_0/FPGA_0_LINK_IO19
- U10 pad E19: /TopSheet/FPGA_0/FPGA_0_LINK_IO77 -> /TopSheet/FPGA_0/FPGA_0_LINK_IO22
- U10 pad E21: /TopSheet/FPGA_0/FPGA_0_LINK_IO95 -> /TopSheet/FPGA_0/FPGA_0_LINK_IO4
- U10 pad E22: /TopSheet/FPGA_0/FPGA_0_LINK_IO93 -> /TopSheet/FPGA_0/FPGA_0_LINK_IO6
- U10 pad F13: /TopSheet/FPGA_0/FPGA_0_LINK_IO51 -> /TopSheet/FPGA_0/FPGA_0_LINK_IO48
- U10 pad F14: /TopSheet/FPGA_0/FPGA_0_LINK_IO52 -> /TopSheet/FPGA_0/FPGA_0_LINK_IO47
- U10 pad F15: /TopSheet/FPGA_0/FPGA_0_LINK_IO50 -> /TopSheet/FPGA_0/FPGA_0_LINK_IO49
- U10 pad F16: /TopSheet/FPGA_0/FPGA_0_LINK_IO53 -> /TopSheet/FPGA_0/FPGA_0_LINK_IO46
- U10 pad F18: /TopSheet/FPGA_0/FPGA_0_LINK_IO79 -> /TopSheet/FPGA_0/FPGA_0_LINK_IO20
- U10 pad F19: /TopSheet/FPGA_0/FPGA_0_LINK_IO85 -> /TopSheet/FPGA_0/FPGA_0_LINK_IO14
- U10 pad F20: /TopSheet/FPGA_0/FPGA_0_LINK_IO86 -> /TopSheet/FPGA_0/FPGA_0_LINK_IO13
- U10 pad F21: /TopSheet/FPGA_0/FPGA_0_LINK_IO99 -> /TopSheet/FPGA_0/FPGA_0_LINK_IO0
- U10 pad G13: /TopSheet/FPGA_0/FPGA_0_LINK_IO2 -> /TopSheet/FPGA_0/FPGA_0_LINK_IO97
- U10 pad G15: /TopSheet/FPGA_0/FPGA_0_LINK_IO3 -> /TopSheet/FPGA_0/FPGA_0_LINK_IO96
- U10 pad G16: /TopSheet/FPGA_0/FPGA_0_LINK_IO4 -> /TopSheet/FPGA_0/FPGA_0_LINK_IO95
- U10 pad G17: /TopSheet/FPGA_0/FPGA_0_LINK_IO7 -> /TopSheet/FPGA_0/FPGA_0_LINK_IO92
- U10 pad G18: /TopSheet/FPGA_0/FPGA_0_LINK_IO8 -> /TopSheet/FPGA_0/FPGA_0_LINK_IO91
- U10 pad G20: /TopSheet/FPGA_0/FPGA_0_LINK_IO16 -> /TopSheet/FPGA_0/FPGA_0_LINK_IO83
- U10 pad G21: /TopSheet/FPGA_0/FPGA_0_LINK_IO97 -> /TopSheet/FPGA_0/FPGA_0_LINK_IO2
- U10 pad G22: /TopSheet/FPGA_0/FPGA_0_LINK_IO98 -> /TopSheet/FPGA_0/FPGA_0_LINK_IO1
- U10 pad H13: /TopSheet/FPGA_0/FPGA_0_LINK_IO1 -> /TopSheet/FPGA_0/FPGA_0_LINK_IO98
- U10 pad H14: /TopSheet/FPGA_0/FPGA_0_LINK_IO6 -> /TopSheet/FPGA_0/FPGA_0_LINK_IO93
- U10 pad H15: /TopSheet/FPGA_0/FPGA_0_LINK_IO10 -> /TopSheet/FPGA_0/FPGA_0_LINK_IO89
- U10 pad H17: /TopSheet/FPGA_0/FPGA_0_LINK_IO11 -> /TopSheet/FPGA_0/FPGA_0_LINK_IO88
- U10 pad H18: /TopSheet/FPGA_0/FPGA_0_LINK_IO12 -> /TopSheet/FPGA_0/FPGA_0_LINK_IO87
- U10 pad H19: /TopSheet/FPGA_0/FPGA_0_LINK_IO24 -> /TopSheet/FPGA_0/FPGA_0_LINK_IO75
- U10 pad H20: /TopSheet/FPGA_0/FPGA_0_LINK_IO15 -> /TopSheet/FPGA_0/FPGA_0_LINK_IO84
- U10 pad H22: /TopSheet/FPGA_0/FPGA_0_LINK_IO14 -> /TopSheet/FPGA_0/FPGA_0_LINK_IO85
- U10 pad J14: /TopSheet/FPGA_0/FPGA_0_LINK_IO5 -> /TopSheet/FPGA_0/FPGA_0_LINK_IO94
- U10 pad J15: /TopSheet/FPGA_0/FPGA_0_LINK_IO9 -> /TopSheet/FPGA_0/FPGA_0_LINK_IO90
- U10 pad J16: /TopSheet/FPGA_0/FPGA_0_LINK_IO0 -> /TopSheet/FPGA_0/FPGA_0_LINK_IO99
- U10 pad J17: /TopSheet/FPGA_0/FPGA_0_LINK_IO42 -> /TopSheet/FPGA_0/FPGA_0_LINK_IO57
- U10 pad J19: /TopSheet/FPGA_0/FPGA_0_LINK_IO23 -> /TopSheet/FPGA_0/FPGA_0_LINK_IO76
- U10 pad J20: /TopSheet/FPGA_0/FPGA_0_LINK_IO21 -> /TopSheet/FPGA_0/FPGA_0_LINK_IO78
- U10 pad J21: /TopSheet/FPGA_0/FPGA_0_LINK_IO22 -> /TopSheet/FPGA_0/FPGA_0_LINK_IO77
- U10 pad J22: /TopSheet/FPGA_0/FPGA_0_LINK_IO13 -> /TopSheet/FPGA_0/FPGA_0_LINK_IO86
- U10 pad K13: /TopSheet/FPGA_0/FPGA_0_LINK_IO37 -> /TopSheet/FPGA_0/FPGA_0_LINK_IO62
- U10 pad K14: /TopSheet/FPGA_0/FPGA_0_LINK_IO38 -> /TopSheet/FPGA_0/FPGA_0_LINK_IO61
- U10 pad K16: /TopSheet/FPGA_0/FPGA_0_LINK_IO46 -> /TopSheet/FPGA_0/FPGA_0_LINK_IO53
- U10 pad K17: /TopSheet/FPGA_0/FPGA_0_LINK_IO41 -> /TopSheet/FPGA_0/FPGA_0_LINK_IO58
- U10 pad K18: /TopSheet/FPGA_0/FPGA_0_LINK_IO25 -> /TopSheet/FPGA_0/FPGA_0_LINK_IO74
- U10 pad K19: /TopSheet/FPGA_0/FPGA_0_LINK_IO26 -> /TopSheet/FPGA_0/FPGA_0_LINK_IO73
- U10 pad K21: /TopSheet/FPGA_0/FPGA_0_LINK_IO17 -> /TopSheet/FPGA_0/FPGA_0_LINK_IO82
- U10 pad K22: /TopSheet/FPGA_0/FPGA_0_LINK_IO18 -> /TopSheet/FPGA_0/FPGA_0_LINK_IO81
- U10 pad L13: /TopSheet/FPGA_0/FPGA_0_LINK_IO40 -> /TopSheet/FPGA_0/FPGA_0_LINK_IO59
- U10 pad L14: /TopSheet/FPGA_0/FPGA_0_LINK_IO43 -> /TopSheet/FPGA_0/FPGA_0_LINK_IO56
- U10 pad L15: /TopSheet/FPGA_0/FPGA_0_LINK_IO44 -> /TopSheet/FPGA_0/FPGA_0_LINK_IO55
- U10 pad L16: /TopSheet/FPGA_0/FPGA_0_LINK_IO45 -> /TopSheet/FPGA_0/FPGA_0_LINK_IO54
- U10 pad L18: /TopSheet/FPGA_0/FPGA_0_LINK_IO32 -> /TopSheet/FPGA_0/FPGA_0_LINK_IO67
- U10 pad L19: /TopSheet/FPGA_0/FPGA_0_LINK_IO27 -> /TopSheet/FPGA_0/FPGA_0_LINK_IO72
- U10 pad L20: /TopSheet/FPGA_0/FPGA_0_LINK_IO28 -> /TopSheet/FPGA_0/FPGA_0_LINK_IO71
- U10 pad L21: /TopSheet/FPGA_0/FPGA_0_LINK_IO20 -> /TopSheet/FPGA_0/FPGA_0_LINK_IO79
- U10 pad M13: /TopSheet/FPGA_0/FPGA_0_LINK_IO39 -> /TopSheet/FPGA_0/FPGA_0_LINK_IO60
- U10 pad M15: /TopSheet/FPGA_0/FPGA_0_LINK_IO47 -> /TopSheet/FPGA_0/FPGA_0_LINK_IO52
- U10 pad M16: /TopSheet/FPGA_0/FPGA_0_LINK_IO48 -> unconnected-(U10-PadM16)
- U10 pad M17: /TopSheet/FPGA_0/FPGA_0_LINK_IO49 -> /TopSheet/FPGA_0/FPGA_0_LINK_IO50
- U10 pad M18: /TopSheet/FPGA_0/FPGA_0_LINK_IO31 -> /TopSheet/FPGA_0/FPGA_0_LINK_IO68
- U10 pad M20: /TopSheet/FPGA_0/FPGA_0_LINK_IO36 -> /TopSheet/FPGA_0/FPGA_0_LINK_IO63
- U10 pad M21: /TopSheet/FPGA_0/FPGA_0_LINK_IO19 -> /TopSheet/FPGA_0/FPGA_0_LINK_IO80
- U10 pad M22: /TopSheet/FPGA_0/FPGA_0_LINK_IO30 -> /TopSheet/FPGA_0/FPGA_0_LINK_IO69
- U10 pad N17: /TopSheet/FPGA_1/FPGA_1_SW7 -> unconnected-(U10-PadN17)
- U10 pad N18: /TopSheet/FPGA_0/FPGA_0_LINK_IO33 -> /TopSheet/FPGA_0/FPGA_0_LINK_IO66
- U10 pad N19: /TopSheet/FPGA_0/FPGA_0_LINK_IO34 -> /TopSheet/FPGA_0/FPGA_0_LINK_IO65
- U10 pad N20: /TopSheet/FPGA_0/FPGA_0_LINK_IO35 -> /TopSheet/FPGA_0/FPGA_0_LINK_IO64
- U10 pad N22: /TopSheet/FPGA_0/FPGA_0_LINK_IO29 -> /TopSheet/FPGA_0/FPGA_0_LINK_IO70
- U10 pad P19: /TopSheet/FPGA_1/FPGA_1_MCU_IO3 -> unconnected-(U10-PadP19)
- U10 pad R14: /TopSheet/FPGA_1/FPGA_1_SW4 -> unconnected-(U10-PadR14)
- U10 pad R18: /TopSheet/FPGA_1/FPGA_1_SW5 -> unconnected-(U10-PadR18)
- U10 pad R19: /TopSheet/FPGA_1/FPGA_1_MCU_IO4 -> unconnected-(U10-PadR19)
- U10 pad T18: /TopSheet/FPGA_1/FPGA_1_SW6 -> unconnected-(U10-PadT18)
- U10 pad T20: /TopSheet/FPGA_1/FPGA_1_MCU_IO5 -> unconnected-(U10-PadT20)
- U10 pad T21: /TopSheet/FPGA_1/FPGA_1_MCU_IO1 -> /TopSheet/FPGA_1/SMC_IO2
- U10 pad U20: /TopSheet/FPGA_1/FPGA_1_MCU_IO14 -> /TopSheet/FPGA_1/FPGA_1_MCU_IO7
- U10 pad U21: /TopSheet/FPGA_1/FPGA_1_MCU_IO2 -> /TopSheet/FPGA_1/SMC_IO3
- U10 pad V17: /TopSheet/FPGA_1/FPGA_1_SPI_MCU_CS -> unconnected-(U10-PadV17)
- U10 pad V20: /TopSheet/FPGA_1/FPGA_1_MCU_IO15 -> /TopSheet/FPGA_1/FPGA_1_MCU_IO8
- U10 pad V22: /TopSheet/FPGA_1/FPGA_1_MCU_IO0 -> unconnected-(U10-PadV22)
- U10 pad W17: /TopSheet/FPGA_1/FPGA_1_SPI_MCU_RX -> unconnected-(U10-PadW17)
- U10 pad W21: /TopSheet/FPGA_1/FPGA_1_MCU_IO6 -> unconnected-(U10-PadW21)
- U10 pad W22: /TopSheet/FPGA_1/FPGA_1_MCU_IO7 -> /TopSheet/FPGA_1/FPGA_1_MCU_IO0
- U10 pad Y19: /TopSheet/FPGA_1/FPGA_1_SPI_MCU_SCLK -> unconnected-(U10-PadY19)
- U10 pad Y21: /TopSheet/FPGA_1/FPGA_1_MCU_IO10 -> /TopSheet/FPGA_1/FPGA_1_MCU_IO3
- U10 pad Y22: /TopSheet/FPGA_1/FPGA_1_MCU_IO11 -> /TopSheet/FPGA_1/FPGA_1_MCU_IO4
- U2 pad 32: /TopSheet/SMC/RPi_SW2 -> /TopSheet/FPGA_0/SMC_IO0
- U2 pad 34: /TopSheet/SMC/RPi_SW3 -> /TopSheet/FPGA_0/SMC_IO1
- U2 pad 35: /TopSheet/SMC/RPi_SW4 -> /TopSheet/FPGA_1/SMC_IO2
- U2 pad 36: /TopSheet/SMC/RPi_SW5 -> /TopSheet/FPGA_1/SMC_IO3
- U20 pad AA18: /TopSheet/FPGA_0/FPGA_0_SPI_MCU_TX -> unconnected-(U20-PadAA18)
- U20 pad AA20: /TopSheet/FPGA_0/FPGA_0_MCU_IO8 -> /TopSheet/FPGA_0/FPGA_0_MCU_IO1
- U20 pad AA21: /TopSheet/FPGA_0/FPGA_0_MCU_IO9 -> /TopSheet/FPGA_0/FPGA_0_MCU_IO2
- U20 pad AB21: /TopSheet/FPGA_0/FPGA_0_MCU_IO12 -> /TopSheet/FPGA_0/FPGA_0_MCU_IO5
- U20 pad AB22: /TopSheet/FPGA_0/FPGA_0_MCU_IO13 -> /TopSheet/FPGA_0/FPGA_0_MCU_IO6
- U20 pad N17: /TopSheet/FPGA_0/FPGA_0_SW7 -> unconnected-(U20-PadN17)
- U20 pad P19: /TopSheet/FPGA_0/FPGA_0_MCU_IO3 -> unconnected-(U20-PadP19)
- U20 pad R14: /TopSheet/FPGA_0/FPGA_0_SW4 -> unconnected-(U20-PadR14)
- U20 pad R18: /TopSheet/FPGA_0/FPGA_0_SW5 -> unconnected-(U20-PadR18)
- U20 pad R19: /TopSheet/FPGA_0/FPGA_0_MCU_IO4 -> unconnected-(U20-PadR19)
- U20 pad T18: /TopSheet/FPGA_0/FPGA_0_SW6 -> unconnected-(U20-PadT18)
- U20 pad T20: /TopSheet/FPGA_0/FPGA_0_MCU_IO5 -> unconnected-(U20-PadT20)
- U20 pad T21: /TopSheet/FPGA_0/FPGA_0_MCU_IO1 -> /TopSheet/FPGA_0/SMC_IO0
- U20 pad U20: /TopSheet/FPGA_0/FPGA_0_MCU_IO14 -> /TopSheet/FPGA_0/FPGA_0_MCU_IO7
- U20 pad U21: /TopSheet/FPGA_0/FPGA_0_MCU_IO2 -> /TopSheet/FPGA_0/SMC_IO1
- U20 pad V17: /TopSheet/FPGA_0/FPGA_0_SPI_MCU_CS -> unconnected-(U20-PadV17)
- U20 pad V20: /TopSheet/FPGA_0/FPGA_0_MCU_IO15 -> /TopSheet/FPGA_0/FPGA_0_MCU_IO8
- U20 pad V22: /TopSheet/FPGA_0/FPGA_0_MCU_IO0 -> unconnected-(U20-PadV22)
- U20 pad W17: /TopSheet/FPGA_0/FPGA_0_SPI_MCU_RX -> unconnected-(U20-PadW17)
- U20 pad W21: /TopSheet/FPGA_0/FPGA_0_MCU_IO6 -> unconnected-(U20-PadW21)
- U20 pad W22: /TopSheet/FPGA_0/FPGA_0_MCU_IO7 -> /TopSheet/FPGA_0/FPGA_0_MCU_IO0
- U20 pad Y19: /TopSheet/FPGA_0/FPGA_0_SPI_MCU_SCLK -> unconnected-(U20-PadY19)
- U20 pad Y21: /TopSheet/FPGA_0/FPGA_0_MCU_IO10 -> /TopSheet/FPGA_0/FPGA_0_MCU_IO3
- U20 pad Y22: /TopSheet/FPGA_0/FPGA_0_MCU_IO11 -> /TopSheet/FPGA_0/FPGA_0_MCU_IO4
- U3 pad 1: GND -> /TopSheet/RP2040 MCU/QSPI2_CS
- U3 pad 2: /TopSheet/FPGA_1/FPGA_1_SPI_MCU_CS -> /TopSheet/RP2040 MCU/QSPI2_SD1
- U3 pad 3: /TopSheet/FPGA_1/FPGA_1_SPI_MCU_TX -> /TopSheet/RP2040 MCU/QSPI2_SD2
- U3 pad 4: /TopSheet/FPGA_1/FPGA_1_MCU_IO0 -> GND
- U3 pad 5: /TopSheet/FPGA_1/FPGA_1_MCU_IO1 -> /TopSheet/RP2040 MCU/QSPI2_SD0
- U3 pad 6: /TopSheet/FPGA_1/FPGA_1_MCU_IO2 -> /TopSheet/RP2040 MCU/QSPI2_SCLK
- U3 pad 7: /TopSheet/FPGA_1/FPGA_1_MCU_IO3 -> /TopSheet/RP2040 MCU/QSPI2_SD3
- U3 pad 8: /TopSheet/FPGA_1/FPGA_1_MCU_IO4 -> /TopSheet/RP2040 MCU/+3V3_RPi2_AUX
- U3 pad 9: /TopSheet/FPGA_1/FPGA_1_MCU_IO5 -> unconnected-(U3-Pad9)
- U5 pad 1: Net-(C34-Pad1) -> +1V8
- U5 pad 12: Net-(C34-Pad1) -> +1V8
- U5 pad 14: +1V8 -> Net-(C34-Pad1)
- U5 pad 15: +1V8 -> Net-(C34-Pad1)
- U5 pad 16: +1V8 -> Net-(C34-Pad1)
- U5 pad 2: Net-(C34-Pad1) -> +1V8
- U5 pad 3: Net-(C34-Pad1) -> +1V8
- U8 pad 1: Net-(C52-Pad1) -> +1V0
- U8 pad 12: Net-(C52-Pad1) -> +1V0
- U8 pad 14: +1V0 -> Net-(C56-Pad1)
- U8 pad 15: +1V0 -> Net-(C56-Pad1)
- U8 pad 16: +1V0 -> Net-(C56-Pad1)
- U8 pad 2: Net-(C52-Pad1) -> +1V0
- U8 pad 3: Net-(C52-Pad1) -> +1V0
- Y1 pad 3: GND -> /TopSheet/SMC/XO_RPi
- Y1 pad 4: /TopSheet/SMC/XO_RPi -> GND
- Y2 pad 1: Net-(C226-Pad2) -> /TopSheet/RP2040 MCU/XI_RPi2
- Y2 pad 2: Net-(C225-Pad2) -> GND
Other:
- board text removed: "MCU COMPONENTS"

Commit message: Layout Update
Parts:
- removed H5: MountingHole, MountingHole:MountingHole_3.5mm
- Q5, R111: moved to B.Cu
- moved R76 470.4 mm to (186.2, 173.0), turned to 90 degrees
- moved R68 457.3 mm to (191.8, 172.5)
- moved R74 450.1 mm to (170.9, 173.0), turned to 90 degrees
- moved R77 443.0 mm to (193.8, 173.0), turned to 90 degrees
- moved R65 429.1 mm to (168.9, 172.5)
- moved C165 408.6 mm to (184.2, 173.5), turned to 180 degrees
- moved SW11 408.0 mm to (176.5, 179.6), turned to 90 degrees
- moved C163 399.0 mm to (168.9, 173.5), turned to 180 degrees
- moved R91 393.9 mm to (262.9, 172.5)
- moved C190 389.1 mm to (262.9, 173.5), turned to 180 degrees
- moved R67 385.9 mm to (184.2, 172.5)
- moved R90 385.1 mm to (255.3, 172.5)
- moved SW10 381.1 mm to (168.9, 179.6), turned to 90 degrees
- moved R98 377.6 mm to (257.3, 173.0), turned to 90 degrees
- moved SW13 377.3 mm to (191.8, 179.6), turned to 90 degrees
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Connections:
- SW18 pad 1: Net-(SW18-Pad1) -> GND
- SW19 pad 1: Net-(SW18-Pad1) -> GND
- SW20 pad 1: Net-(SW18-Pad1) -> GND
- SW21 pad 1: Net-(SW18-Pad1) -> GND

Commit message: Layout Update
Parts:
- removed C180, C181, C182, C183, C184, C195, C198, C199, C200: 100nF, Capacitor_SMD:C_0402_1005Metric
- removed R100, R101, R102, R103, R107, R84, R86, R87: 100K, Resistor_SMD:R_0402_1005Metric
- removed R105, R106, R109, R110, R83: 1Meg, Resistor_SMD:R_0402_1005Metric
- removed R108: 0R, Resistor_SMD:R_0402_1005Metric
- removed R85: 1K, Resistor_SMD:R_0402_1005Metric
- removed R92, R93, R94, R95: 3K3, Resistor_SMD:R_0402_1005Metric
- removed SW14, SW15, SW16, SW17, SW22, SW23, SW24, SW25: SW_Push, Button_Switch_SMD:SW_SPST_EVQQ2
- added C38: 100nF, Capacitor_SMD:C_0402_1005Metric, F.Cu at (290.1, 98.0)
- added C39: 100nF, Capacitor_SMD:C_0402_1005Metric, F.Cu at (281.0, 98.0)
- added C40: 100nF, Capacitor_SMD:C_0402_1005Metric, F.Cu at (285.0, 98.0)
- added C41: 100nF, Capacitor_SMD:C_0402_1005Metric, F.Cu at (288.1, 98.0)
- added C51: 100nF, Capacitor_SMD:C_0402_1005Metric, F.Cu at (279.9, 98.0)
- added C52: 100nF, Capacitor_SMD:C_0402_1005Metric, F.Cu at (284.0, 98.0)
- added C53: 100nF, Capacitor_SMD:C_0402_1005Metric, F.Cu at (291.6, 95.0)
- added C54: 100nF, Capacitor_SMD:C_0402_1005Metric, F.Cu at (282.0, 98.0)
- added R26: 1Meg, Resistor_SMD:R_0402_1005Metric, B.Cu at (287.0, 95.8)
- added R27: 1Meg, Resistor_SMD:R_0402_1005Metric, B.Cu at (288.0, 95.8)
- added R28: 100K, Resistor_SMD:R_0402_1005Metric, F.Cu at (291.6, 97.5)
- Q10, Q11, Q12, Q13, Q14, Q15, Q16, Q17, Q18, Q19, Q20, Q6, Q7, Q8, Q9, R112, R115, R116, R124, R125, R128, R129, R136, R137, R140, R141, R144, R145, R148, R149, R81: moved to B.Cu
- R69: value 3K3 -> 100K
- R70: value 3K3 -> 1K; moved to B.Cu
- R71: value 3K3 -> 100K; moved to B.Cu
- R73: value 3K3 -> 1Meg; moved to B.Cu
- R78: value 100K -> 1Meg; moved to B.Cu
- R79, R80: value 100K -> 1Meg
- R82: value 1Meg -> 0R; moved to B.Cu
- moved TP16 698.0 mm to (68.6, 242.3)
- moved TP15 662.8 mm to (79.8, 235.7)
- moved C243 645.7 mm to (124.1, 241.3)
- moved C245 645.7 mm to (129.0, 254.2)
- moved C247 645.7 mm to (118.5, 244.3)
- moved C249 645.7 mm to (142.2, 239.2)
- moved C250 645.7 mm to (129.6, 236.5)
- moved C251 645.7 mm to (147.8, 232.6)
- moved C252 645.7 mm to (133.1, 243.5)
- moved C253 645.7 mm to (106.2, 258.4)
- moved C254 645.7 mm to (111.7, 267.3)
- moved C255 645.7 mm to (131.8, 249.4)
- moved C256 645.7 mm to (116.3, 264.1)
- moved C257 645.7 mm to (119.1, 240.7)
- moved C258 645.7 mm to (123.2, 254.8)
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Connections:
- C166 pad 1: /TopSheet/UserIO/DP_TX_C_LANE0_N -> /TopSheet/FPGA_1/FPGA_1_DP_RXL3_P
- C166 pad 2: /TopSheet/FPGA_1/FPGA_1_DP_TXL0_N -> /TopSheet/UserIO/DP_TX_C_LANE3_P
- C168 pad 1: /TopSheet/UserIO/DP_TX_C_LANE2_N -> /TopSheet/UserIO/DP_TX_C_LANE3_N
- C168 pad 2: /TopSheet/FPGA_1/FPGA_1_DP_TXL2_N -> /TopSheet/FPGA_1/FPGA_1_DP_TXL3_N
- C169 pad 1: /TopSheet/FPGA_1/FPGA_1_DP_TXL0_P -> /TopSheet/UserIO/DP_RX_C_AUX_N
- C169 pad 2: /TopSheet/UserIO/DP_TX_C_LANE0_P -> /TopSheet/FPGA_1/FPGA_1_DP_RX_AUX_N
- C170 pad 1: /TopSheet/FPGA_1/FPGA_1_DP_TXL1_P -> /TopSheet/FPGA_1/FPGA_1_DP_RX_AUX_P
- C170 pad 2: /TopSheet/UserIO/DP_TX_C_LANE1_P -> /TopSheet/UserIO/DP_RX_C_AUX_P
- C171 pad 1: /TopSheet/FPGA_1/FPGA_1_DP_TXL2_P -> /TopSheet/UserIO/DP_RX_PWR
- C171 pad 2: /TopSheet/UserIO/DP_TX_C_LANE2_P -> GND
- J10 pad 1: GND -> /TopSheet/FPGA_1/FPGA_1_DP_RXL3_N
- J10 pad 11: /TopSheet/FPGA_1/FPGA_1_DP_RXL2_P -> GND
- J10 pad 13: GND -> /TopSheet/UserIO/DP_RX_CFG1
- J10 pad 14: GND -> /TopSheet/UserIO/DP_RX_CFG2
- J10 pad 15: /TopSheet/FPGA_1/FPGA_1_DP_RXL1_N -> /TopSheet/UserIO/DP_RX_C_AUX_P
- J10 pad 16: /TopSheet/UserIO/DP_RX_C_AUX_P -> GND
- J10 pad 17: /TopSheet/FPGA_1/FPGA_1_DP_RXL1_P -> /TopSheet/UserIO/DP_RX_C_AUX_N
- J10 pad 18: /TopSheet/UserIO/DP_RX_C_AUX_N -> /TopSheet/UserIO/DP_RX_C_HPD
- J10 pad 2: /TopSheet/UserIO/DP_RX_C_HPD -> GND
- J10 pad 3: /TopSheet/FPGA_1/FPGA_1_DP_RXL3_N -> /TopSheet/FPGA_1/FPGA_1_DP_TXL3_P
- J10 pad 4: /TopSheet/UserIO/DP_RX_CFG1 -> /TopSheet/FPGA_1/FPGA_1_DP_RXL2_N
- J10 pad 5: /TopSheet/FPGA_1/FPGA_1_DP_TXL3_P -> GND
- J10 pad 6: /TopSheet/UserIO/DP_RX_CFG2 -> /TopSheet/FPGA_1/FPGA_1_DP_RXL2_P
- J10 pad 7: GND -> /TopSheet/FPGA_1/FPGA_1_DP_RXL1_N
- J10 pad 9: /TopSheet/FPGA_1/FPGA_1_DP_RXL2_N -> /TopSheet/FPGA_1/FPGA_1_DP_RXL1_P
- J7 pad 1: GND -> /TopSheet/UserIO/DP_TX_C_LANE0_P
- J7 pad 11: /TopSheet/UserIO/DP_TX_C_LANE1_N -> GND
- J7 pad 13: GND -> /TopSheet/UserIO/DP_TX_CFG1
- J7 pad 14: GND -> /TopSheet/UserIO/DP_TX_CFG2
- J7 pad 15: /TopSheet/UserIO/DP_TX_C_LANE2_P -> /TopSheet/UserIO/DP_TX_C_AUX_P
- J7 pad 16: /TopSheet/UserIO/DP_TX_C_AUX_P -> GND
- J7 pad 17: /TopSheet/UserIO/DP_TX_C_LANE2_N -> /TopSheet/UserIO/DP_TX_C_AUX_N
- J7 pad 18: /TopSheet/UserIO/DP_TX_C_AUX_N -> Net-(J7-Pad18)
- J7 pad 2: /TopSheet/UserIO/DP_TX_C_HPD -> GND
- J7 pad 3: /TopSheet/UserIO/DP_TX_C_LANE0_P -> /TopSheet/UserIO/DP_TX_C_LANE0_N
- J7 pad 4: /TopSheet/UserIO/DP_TX_CFG1 -> /TopSheet/UserIO/DP_TX_C_LANE1_P
- J7 pad 5: /TopSheet/UserIO/DP_TX_C_LANE0_N -> GND
- J7 pad 6: /TopSheet/UserIO/DP_TX_CFG2 -> /TopSheet/UserIO/DP_TX_C_LANE1_N
- J7 pad 7: GND -> /TopSheet/UserIO/DP_TX_C_LANE2_P
- J7 pad 9: /TopSheet/UserIO/DP_TX_C_LANE1_P -> /TopSheet/UserIO/DP_TX_C_LANE2_N
- R69 pad 1: +3V3 -> GND
- R69 pad 2: /TopSheet/UserIO/FPGA_1_SW4_R -> /TopSheet/UserIO/DP_TX_C_AUX_P
- R70 pad 1: +3V3 -> Net-(J7-Pad18)
- R70 pad 2: /TopSheet/UserIO/FPGA_1_SW5_R -> /TopSheet/FPGA_1/FPGA_1_DP_TX_HPD
- R71 pad 1: +3V3 -> Net-(J7-Pad18)
- R71 pad 2: /TopSheet/UserIO/FPGA_1_SW6_R -> GND
- R73 pad 1: +3V3 -> GND
- R73 pad 2: /TopSheet/UserIO/FPGA_1_SW7_R -> /TopSheet/UserIO/DP_RX_CFG1
- R78 pad 1: /TopSheet/UserIO/FPGA_1_SW4_R -> GND
- R78 pad 2: /TopSheet/FPGA_0/FPGA_0_SW4 -> /TopSheet/UserIO/DP_RX_CFG2
- R79 pad 1: /TopSheet/UserIO/FPGA_1_SW5_R -> /TopSheet/UserIO/DP_RX_C_AUX_N
- R79 pad 2: /TopSheet/FPGA_0/FPGA_0_SW5 -> +3V3
- R80 pad 1: /TopSheet/UserIO/FPGA_1_SW6_R -> /TopSheet/UserIO/DP_RX_C_AUX_P
- R80 pad 2: /TopSheet/FPGA_0/FPGA_0_SW6 -> GND
- R81 pad 1: /TopSheet/UserIO/FPGA_1_SW7_R -> GND
- R81 pad 2: /TopSheet/FPGA_0/FPGA_0_SW7 -> /TopSheet/UserIO/DP_RX_C_HPD
- R82 pad 1: GND -> /TopSheet/UserIO/DP_RX_C_HPD
- R82 pad 2: /TopSheet/UserIO/DP_TX_CFG1 -> /TopSheet/FPGA_1/FPGA_1_DP_RX_HPD
Routing:
- net GND: track 0.00 -> 116.5 mm, vias 0 -> 157
- net +3V3: track 0.00 -> 65.7 mm, vias 0 -> 68
- net +1V0: track 0.00 -> 31.2 mm, vias 0 -> 44
- net +1V8: track 0.00 -> 21.4 mm, vias 0 -> 22
- net +1V2: track 0.00 -> 8.52 mm, vias 0 -> 12
- net /TopSheet/FPGA_0/FPGA_0_PMOD2_LV_IO6: track 0.00 -> 6.49 mm, vias 0 -> 3
- net /TopSheet/FPGA_0/FPGA_0_USER_IO2: track 0.00 -> 6.48 mm, vias 0 -> 3
- net /TopSheet/FPGA_0/FPGA_0_USER_IO1: track 0.00 -> 6.48 mm, vias 0 -> 3
- net /TopSheet/FPGA_0/FPGA_0_PMOD1_LV_IO5: track 0.00 -> 6.48 mm, vias 0 -> 3
- net /TopSheet/FPGA_0/FPGA_0_PMOD1_LV_IO4: track 0.00 -> 6.48 mm, vias 0 -> 3
- net /TopSheet/FPGA_0/FPGA_0_PMOD0_LV_IO0: track 0.00 -> 6.48 mm, vias 0 -> 3
- net /TopSheet/FPGA_0/FPGA_0_LINK_IO70: track 0.00 -> 4.32 mm, vias 0 -> 2
- net /TopSheet/FPGA_0/FPGA_0_LINK_IO69: track 0.00 -> 4.32 mm, vias 0 -> 2
- net /TopSheet/FPGA_0/FPGA_0_LINK_IO30: track 0.00 -> 4.32 mm, vias 0 -> 2
- net /TopSheet/FPGA_0/FPGA_0_LINK_IO29: track 0.00 -> 4.32 mm, vias 0 -> 2
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