File: DSN/PMU.kicad_sch (KiCad schematic)
At the start: 56 parts, among them U4 INA260, U5 INA260, U6 LTC3370, U7 INA260, U8 INA260

Commit message: Layout Update
Connections:
- net at R47.2, R48.1: now also U6.25 (FB4); no longer U6.24 (VIN_H)
Changed lines of the file:
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@@
     (pin "22")
     (pin "23")
-    (pin "24")
+    (pin "25")
     (pin "24")
     (pin "26")
