File: DSN/USB-UART-JTAG.kicad_sch (KiCad schematic)
At the start: 91 parts, among them J27 USB_C_Receptacle_USB2.0, J28 Conn_02x07_Odd_Even, J29 Conn_01x03_Male, J30 Conn_01x03_Male, J31 Conn_02x07_Odd_Even, Q21 AON6411, U15 93LCxxB, U16 74HC595, U17 FT4232H, U18 ADG794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

Commit message: Layout Update
Connections:
- net FTDI_TMS_CH0: now also U18.14 (S4A); no longer U18.15 (S4A)
- net FTDI_TMS_CH1: now also U19.14 (S4A); no longer U19.15 (S4A)
Changed lines of the file:
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@@
     (pin "2")
   )
-  (symbol (lib_id "Analog:ADG794") (at 444.5 203.2 0) (unit 1)
+  (symbol (lib_name "ADG794_1") (lib_id "Analog:ADG794") (at 444.5 203.2 0) (unit 1)
     (in_bom yes) (on_board yes) (fields_autoplaced)
     (property "Reference" "U18" (id 0) (at 454.025 163.83 0))
@@
     (pin "12")
     (pin "13")
-    (pin "15")
+    (pin "14")
     (pin "15")
     (pin "16")
@@
     (pin "13")
     (pin "15")
-    (pin "15")
+    (pin "14")
     (pin "16")
     (pin "2")
